File: src/HardwareDesign/Relay-Board_Rack-PDU.brd (EAGLE design)
At the start: 147 x 95 mm, 70 parts, among them IC1 ULN2803, IC3 TS432ILT, T1 750370228

Commit message: first order send to JLCPCB
Parts:
- C14: value 100nF 275V -> MP2104K27C3R6LC 100nF 275V
- C15, C17: value 15uF 400V -> KM150M400G160A 15uF 400V
- D1: value MBRA340T3 -> MBRA340T3G
- IC1: value ULN2803 -> ULN2803A
Changed lines of the file:
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@@
 <drawing>
 <settings>
-<setting alwaysvectorfont="yes"/>
+<setting alwaysvectorfont="no"/>
 <setting verticaltext="up"/>
 </settings>
@@
 </autorouter>
 <elements>
-<element name="D1" library="diode" library_urn="urn:adsk.eagle:library:210" package="SMA" package3d_urn="urn:adsk.eagle:package:43460/3" value="MBRA340T3" x="19.09" y="39.72" smashed="yes" rot="R180">
+<element name="D1" library="diode" library_urn="urn:adsk.eagle:library:210" package="SMA" package3d_urn="urn:adsk.eagle:package:43460/3" value="MBRA340T3G" x="19.09" y="39.72" smashed="yes" rot="R180">
 <attribute name="NAME" x="21.84" y="37.72" size="1.27" layer="25" ratio="10" rot="R180"/>
 <attribute name="VALUE" x="21.84" y="43.22" size="1.27" layer="27" ratio="10" rot="R180"/>
@@
 <attribute name="WMAX" value="4.8J" x="15.4" y="67.17" size="1.778" layer="27" rot="R270" display="off"/>
 </element>
-<element name="C14" library="ds_passive" package="103-275V" package3d_urn="urn:adsk.eagle:package:46766481/2" value="100nF 275V" x="21.93" y="79.38" smashed="yes">
+<element name="C14" library="ds_passive" package="103-275V" package3d_urn="urn:adsk.eagle:package:46766481/2" value="MP2104K27C3R6LC 100nF 275V" x="21.93" y="79.38" smashed="yes">
 <attribute name="NAME" x="13.53" y="74.98" size="1.016" layer="25"/>
 <attribute name="VALUE" x="13.43" y="75.38" size="1.016" layer="27"/>
@@
 <attribute name="VALUE" x="11.898" y="67.31" size="1.27" layer="27" rot="R90"/>
 </element>
-<element name="C15" library="Capacitor" library_urn="urn:adsk.eagle:library:16290819" package="CAPPRD550W110D1250H2500B" package3d_urn="urn:adsk.eagle:package:16290890/3" value="15uF 400V" x="24.94" y="56.35" smashed="yes" rot="R180">
+<element name="C15" library="Capacitor" library_urn="urn:adsk.eagle:library:16290819" package="CAPPRD550W110D1250H2500B" package3d_urn="urn:adsk.eagle:package:16290890/3" value="KM150M400G160A 15uF 400V" x="24.94" y="56.35" smashed="yes" rot="R180">
 <attribute name="CATEGORY" value="Capacitor" x="24.94" y="56.35" size="1.778" layer="27" rot="R180" display="off"/>
 <attribute name="DATASHEET" value="" x="24.94" y="56.35" size="1.778" layer="27" rot="R180" display="off"/>
@@
 <attribute name="VALUE" x="26.15" y="93.95" size="1.27" layer="27" rot="R180"/>
 </element>
-<element name="C17" library="Capacitor" library_urn="urn:adsk.eagle:library:16290819" package="CAPPRD550W110D1250H2500B" package3d_urn="urn:adsk.eagle:package:16290890/3" value="15uF 400V" x="24.94" y="69.42" smashed="yes" rot="R180">
+<element name="C17" library="Capacitor" library_urn="urn:adsk.eagle:library:16290819" package="CAPPRD550W110D1250H2500B" package3d_urn="urn:adsk.eagle:package:16290890/3" value="KM150M400G160A 15uF 400V" x="24.94" y="69.42" smashed="yes" rot="R180">
 <attribute name="CATEGORY" value="Capacitor" x="24.94" y="69.42" size="1.778" layer="27" rot="R180" display="off"/>
 <attribute name="DATASHEET" value="" x="24.94" y="69.42" size="1.778" layer="27" rot="R180" display="off"/>
@@
 <attribute name="VALUE" x="94.05" y="55.22" size="1.016" layer="27" rot="R270"/>
 </element>
-<element name="IC1" library="ds_ic_peripherals" package="SO18" package3d_urn="urn:adsk.eagle:package:46683893/2" value="ULN2803" x="119.4" y="56.3" smashed="yes" rot="R90">
+<element name="IC1" library="ds_ic_peripherals" package="SO18" package3d_urn="urn:adsk.eagle:package:46683893/2" value="ULN2803A" x="119.4" y="56.3" smashed="yes" rot="R90">
 <attribute name="NAME" x="122.02" y="48.77" size="1.27" layer="25"/>
 </element>
