File: src/HardwareDesign/Display-Board_Rack-PDU_2.0.brd (EAGLE design)
At the start: 135 x 65 mm, 43 parts, among them IC2 MCP23017-E/ML, J1 68714014022, J2 68714014022, T1 BSS138

Commit message: working on Rev2.0
Parts:
- removed J2: 68714014022, Wurth_Connectors_WR-FPC:68714014022
- added DISPBOARD: 687320124422, Wurth_Connectors_WR-FPC:687320124422
Connections:
- removed net EXP_RST: IC2.14, J2.23
- removed net N$10: J2.38
- removed net N$11: J2.37
- new net MCP_DSP_RST: DISPBOARD.20, IC2.14
- net +3V3: now also DISPBOARD.1, DISPBOARD.2, IC2.11; no longer J2.1, J2.2
- net +5V: now also DISPBOARD.3, DISPBOARD.4; no longer J2.3, J2.4
- net DSP_RES: now also DISPBOARD.9; no longer J2.9
- net GND: now also DISPBOARD.14, DISPBOARD.19, DISPBOARD.5, DISPBOARD.8, DISPBOARD.Z1, DISPBOARD.Z2, DISPBOARD.Z3, DISPBOARD.Z4; no longer IC2.11, J2.10, J2.12, J2.17, J2.22, J2.5, J2.8, J2.Z1, J2.Z2
- net I2C_SCL: now also DISPBOARD.7; no longer J2.7
- net I2C_SDA: now also DISPBOARD.6; no longer J2.6
- net KEY_0: now also DISPBOARD.10; no longer J2.13
- net KEY_1: now also DISPBOARD.11; no longer J2.14
- net KEY_2: now also DISPBOARD.12; no longer J2.15
- net KEY_3: now also DISPBOARD.13; no longer J2.16
- net SPI_CS: now also DISPBOARD.18; no longer J2.21
- net SPI_MISO: now also DISPBOARD.16; no longer J2.19
- net SPI_MOSI: now also DISPBOARD.15; no longer J2.18
- net SPI_SCLK: now also DISPBOARD.17; no longer J2.20
Routing:
- net I2C_SCL: track 100.6 -> 0.00 mm, vias 2 -> 0
- net I2C_SDA: track 99.8 -> 0.00 mm, vias 2 -> 0
- net EXP_RST: track 83.5 -> 0.00 mm, vias 2 -> 0
- net BCKL: track 81.1 -> 0.00 mm, vias 4 -> 0
- net KEY_0: track 74.0 -> 0.00 mm, vias 2 -> 0
- net GND: track 417.8 -> 350.7 mm, vias 25 -> 17
- net KEY_1: track 54.5 -> 0.00 mm, vias 2 -> 0
- net KEY_2: track 52.7 -> 0.00 mm, vias 2 -> 0
- net KEY_3: track 64.1 -> 12.6 mm, vias 2 -> 1
- net SPI_SCLK: track 44.5 -> 2.19 mm, vias 2 -> 1
- net SPI_CS: track 44.5 -> 2.47 mm, vias 2 -> 1
- net SPI_MOSI: track 43.1 -> 2.39 mm, vias 2 -> 1
- net SPI_MISO: track 43.7 -> 3.59 mm, vias 2 -> 1
- net DSP_RES: track 32.3 -> 1.61 mm, vias 2 -> 1
- net +3V3: track 202.5 -> 181.5 mm
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
Commit message: finished with design update for 2.0
Parts:
- removed J1: 68714014022, Wurth_Connectors_WR-FPC:68714014022
- removed R17: 10K, ds_passive:0402
- added 3V3, 5V, BL, CS, DC, GND, I2C_SCL, I2C_SDA, KEY0, KEY1, KEY2, KEY3, LCD_RES, MCP_RES, MISO, MOSI, SCK: TP, ds_passive:TP
- added R4: 10K, ds_passive:0402
- added TFT: FPC40-HD, ds_con:FPC40_3.5TFT
- DISPBOARD: value 687320124422 -> FPC20-H; device Wurth_Connectors_WR-FPC:687320124422 -> ds_con:FPC20
- R1, R2, R3: value 330R -> 56R
- moved DISPBOARD 1.56 mm to (74.8, 9.00), turned to 180 degrees
Connections:
- removed net BCKL: IC2.28, T1.1
- removed net DSP_RES: DISPBOARD.9, J1.15
- removed net N$1: J1.10, R17.2
- removed net SPI_CS: DISPBOARD.18, J1.9
- removed net SPI_MISO: DISPBOARD.16, J1.14
- removed net SPI_MOSI: DISPBOARD.15, J1.13
- removed net SPI_SCLK: DISPBOARD.17, J1.11
- new net LCD_BL: BL.TP, DISPBOARD.13, R4.1, T1.1
- new net LCD_CS: CS.TP, DISPBOARD.19, TFT.9
- new net LCD_DC: DC.TP, DISPBOARD.18, TFT.10
- new net LCD_MISO: DISPBOARD.15, MISO.TP, TFT.14
- new net LCD_MOSI: DISPBOARD.16, MOSI.TP, TFT.13
- new net LCD_RES: DISPBOARD.14, LCD_RES.TP, TFT.15
- new net LCD_SCLK: DISPBOARD.17, SCK.TP, TFT.11
- net +3V3: now also 3V3.TP, TFT.12, TFT.38, TFT.39, TFT.40, TFT.6, TFT.7; no longer J1.12, J1.38, J1.39, J1.40, J1.6, J1.7
- net +5V: now also 5V.TP, TFT.33; no longer J1.33
- net GND: now also GND.TP, R4.2, TFT.16, TFT.17, TFT.18, TFT.19, TFT.20, TFT.21, TFT.22, TFT.23, TFT.24, TFT.25, TFT.26, TFT.27, TFT.28, TFT.29, TFT.30, TFT.31, TFT.32, TFT.37, TFT.5, TFT.Z1, TFT.Z2; no longer DISPBOARD.14, DISPBOARD.19, J1.16, J1.17, J1.18, J1.19, J1.20, J1.21, J1.22, J1.23, J1.24, J1.25, J1.26, J1.27, J1.28, J1.29, J1.30, J1.31, J1.32, J1.37, J1.5, J1.Z1, J1.Z2, R17.1
- net I2C_SCL: now also I2C_SCL.TP
- net I2C_SDA: now also I2C_SDA.TP
- net KEY_0: now also DISPBOARD.12, KEY0.TP; no longer DISPBOARD.10
- net KEY_1: now also KEY1.TP
- net KEY_2: now also DISPBOARD.10, KEY2.TP; no longer DISPBOARD.12
- net KEY_3: now also DISPBOARD.9, KEY3.TP; no longer DISPBOARD.13
- net MCP_DSP_RST: now also MCP_RES.TP
- net N$2: now also TFT.35; no longer J1.35
- net N$3: now also TFT.36; no longer J1.36
- net N$5: now also TFT.34; no longer J1.34
Routing:
- net GND: track 350.7 -> 475.4 mm, vias 17 -> 23
- net KEY_1: track 0.00 -> 93.5 mm, vias 0 -> 2
- net I2C_SDA: track 0.00 -> 92.8 mm, vias 0 -> 4
- net I2C_SCL: track 0.00 -> 89.4 mm, vias 0 -> 4
- net MCP_DSP_RST: track 0.00 -> 88.0 mm, vias 0 -> 4
- net KEY_0: track 0.00 -> 83.4 mm, vias 0 -> 2
- net KEY_2: track 0.00 -> 72.6 mm, vias 0 -> 2
- net LCD_BL: track 0.00 -> 67.6 mm, vias 0 -> 1
- net KEY_3: track 12.6 -> 79.5 mm, vias 1 -> 2
- net LCD_DC: track 0.00 -> 63.4 mm, vias 0 -> 1
- net LCD_CS: track 0.00 -> 62.5 mm, vias 0 -> 1
- net LCD_RES: track 0.00 -> 62.0 mm, vias 0 -> 1
- net LCD_MOSI: track 0.00 -> 59.7 mm, vias 0 -> 1
- net LCD_MISO: track 0.00 -> 57.7 mm, vias 0 -> 1
- net LCD_SCLK: track 0.00 -> 57.3 mm, vias 0 -> 1
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Other:
- board text added: "o"
