File: src/HardwareDesign/Controller-Board_Rack-PDU_2.0.brd (EAGLE design)
At the start: 90 x 85 mm, 104 parts, among them IC1 W5500, IC2 RP2040, IC3 MCP6001AIDBVRG, IC4 W25Q128JVPIQ, IC5 MIC5504-3.3YM5-TR, IC6 CAT24C256HU4IGT3, J2 68714014022, X1 XC53M4-25.000-F18NJDTL, X2 K5A1200015304P

Commit message: working on Rev2.0
Parts:
- removed 12VFB: TP, ds_passive:TP
- removed J2: 68714014022, Wurth_Connectors_WR-FPC:68714014022
- removed R46, R47: 0R, ds_passive:0402
- removed R48: 100K, ds_passive:0402
- removed R49: 10K, ds_passive:0402
- added DISPBOARD, RELAYBOARD: 687320124422, Wurth_Connectors_WR-FPC:687320124422
- IC3: value MCP6001AIDBVRG -> MCP6001R
- moved IC5 19.7 mm to (-7.30, -23.6)
- moved C40 15.6 mm to (-21.0, -23.8)
- moved C41 13.9 mm to (-15.4, -8.80)
- moved C36 11.9 mm to (-20.5, -8.80)
- moved U$1 8.60 mm to (25.0, 2.00)
- moved C42 6.89 mm to (-15.6, -23.8)
- moved R25 4.22 mm to (68.8, 11.2)
- moved C26 4.22 mm to (69.3, 6.71)
- moved C27 4.22 mm to (68.8, 9.75)
- moved USBC 4.22 mm to (74.1, -0.66)
- moved ESD1 4.22 mm to (73.6, 8.23)
- moved R26 4.22 mm to (66.7, 10.5)
- moved R39 4.22 mm to (78.4, 5.94)
- moved C54 4.22 mm to (78.4, 7.21)
- moved R20 4.22 mm to (68.8, 8.48)
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Connections:
- removed net +12V: R48.2
- removed net DIO_RESET: IC2.9
- removed net EXP_RST: IC2.35, J2.23
- removed net I_MEA/TX: IC2.40, R46.1
- removed net N$8: IC1.31, R12.2
- removed net N$9: IC1.30, R13.2
- removed net PWR_DETECT: 12VFB.TP, IC2.41, R48.1, R49.2
- removed net V_MEA/RX: IC2.39, R47.1
- new net +12V_MEA: IC2.41, RELAYBOARD.13
- new net MCP_DSP_RST: DISPBOARD.20, IC2.9
- new net MCP_REL_RST: IC2.35, RELAYBOARD.15
- new net XO: IC1.31, R12.2, R13.2
- net !SPI1_CS_S: now also DISPBOARD.18; no longer J2.21
- net +3V3: now also DISPBOARD.1, DISPBOARD.2, RELAYBOARD.4, RELAYBOARD.5, RELAYBOARD.6; no longer J2.1, J2.2
- net +5V: now also DISPBOARD.3, DISPBOARD.4, RELAYBOARD.1, RELAYBOARD.2, RELAYBOARD.3; no longer J2.3, J2.4
- net DSP_RES: now also DISPBOARD.9; no longer J2.9
- net GND: now also DISPBOARD.14, DISPBOARD.19, DISPBOARD.5, DISPBOARD.8, DISPBOARD.Z1, DISPBOARD.Z2, DISPBOARD.Z3, DISPBOARD.Z4, RELAYBOARD.12, RELAYBOARD.14, RELAYBOARD.16, RELAYBOARD.9, RELAYBOARD.Z1, RELAYBOARD.Z2, RELAYBOARD.Z3, RELAYBOARD.Z4; no longer J2.10, J2.12, J2.17, J2.22, J2.5, J2.8, J2.Z1, J2.Z2, R49.1
- net I2C0_SCL: now also DISPBOARD.7; no longer J2.7
- net I2C0_SDA: now also DISPBOARD.6; no longer J2.6
- net I2C1_SCL: now also RELAYBOARD.8
- net I2C1_SDA: now also RELAYBOARD.7
- net KEY_0: now also DISPBOARD.10; no longer J2.13
- net KEY_1: now also DISPBOARD.11; no longer J2.14
- net KEY_2: now also DISPBOARD.12; no longer J2.15
- net KEY_3: now also DISPBOARD.13; no longer J2.16
- net N$7: now also IC1.30
- net SPI1_MISO: now also DISPBOARD.16; no longer J2.19
- net SPI1_MOSI: now also DISPBOARD.15; no longer J2.18
- net SPI1_SCK: now also DISPBOARD.17; no longer J2.20
- net UART0_RX: now also RELAYBOARD.10; no longer J2.25, R47.2
- net UART0_TX: now also RELAYBOARD.11; no longer J2.26, R46.2
Routing:
- net N$7: track 0.00 -> 15.1 mm
- net XO: track 0.00 -> 7.94 mm
- net N$6: track 0.00 -> 2.20 mm
Other:
- board size 90 x 85 mm -> 66 x 83 mm

Commit message: finished with design update for 2.0
Parts:
- moved DISPBOARD 2.24 mm to (30.7, 9.80)
Connections:
- net !SPI1_CS_S renamed LCD_DC
- net SPI1_SCK renamed LCD_SCLK
- removed net !SPI1_CS: IC2.12
- removed net DSP_RES: DISPBOARD.9, IC2.34
- removed net SPI1_MISO: DISPBOARD.16, IC2.11
- removed net SPI1_MOSI: DISPBOARD.15, IC2.14
- new net LCD_BL: DISPBOARD.13, IC2.9
- new net LCD_CS: DISPBOARD.19, IC2.12
- new net LCD_MISO: DISPBOARD.15, IC2.11
- new net LCD_MOSI: DISPBOARD.16, IC2.14
- new net LCD_RES: DISPBOARD.14, IC2.34
- net GND: no longer DISPBOARD.14, DISPBOARD.19
- net KEY_0: now also DISPBOARD.12; no longer DISPBOARD.10
- net KEY_2: now also DISPBOARD.10; no longer DISPBOARD.12
- net KEY_3: now also DISPBOARD.9; no longer DISPBOARD.13
- net MCP_DSP_RST: now also IC2.36; no longer IC2.9

Commit message: finished Rev2
Parts:
- removed R12: 0R, ds_passive:0402
- removed USB_BOOT: B3U-1000P-B, 52101-101-REV-A_v16:SWITCH-OMRON_B3U-1000P
- added BOOT: 430182043816, Wurth_Switch_WS-TASV:430182043816
- RESET: value B3U-1000P-B -> 430182043816; device 52101-101-REV-A_v16:SWITCH-OMRON_B3U-1000P -> Wurth_Switch_WS-TASV:430182043816
- moved C40 73.8 mm to (40.8, 16.5)
- moved C42 72.9 mm to (40.8, 22.4)
- moved DBG1 69.8 mm to (3.93, 72.4), turned to 180 degrees
- moved C36 65.8 mm to (40.9, 14.9)
- moved C41 65.8 mm to (43.4, 20.6), turned to 90 degrees
- moved IC5 64.6 mm to (40.8, 19.5)
- moved RESET 52.4 mm to (16.0, 73.5), turned to 180 degrees
- moved DBG2 48.8 mm to (3.87, 60.5), turned to 180 degrees
- moved R50 45.9 mm to (16.1, 69.1), turned to 180 degrees
- moved R28 45.7 mm to (25.9, 71.2), turned to 90 degrees
- moved R15 43.1 mm to (11.5, 60.7), turned to 270 degrees
- moved IC6 42.6 mm to (28.5, 71.3), turned to 0 degrees
- moved R27 40.8 mm to (28.4, 73.2), turned to 0 degrees
- moved C25 40.6 mm to (40.1, 60.4)
- moved R18 40.6 mm to (40.1, 63.7)
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Connections:
- removed net N$6: C8.1, R12.1, X1.1
- net GND: now also BOOT.3, BOOT.4, RESET.1; no longer USB_BOOT.2
- net N$17: now also RESET.3, RESET.4; no longer RESET.1
- net USB_BOOT: now also BOOT.1, BOOT.2; no longer USB_BOOT.1
- net XO: now also C8.1, X1.1; no longer R12.2
Routing:
- net +3V3: track 0.00 -> 321.2 mm, vias 0 -> 10
- net GND: track 0.00 -> 182.0 mm, vias 0 -> 96
- net I2C1_SDA: track 0.00 -> 84.4 mm, vias 0 -> 5
- net I2C1_SCL: track 0.00 -> 84.3 mm, vias 0 -> 5
- net LCD_MISO: track 0.00 -> 83.1 mm, vias 0 -> 2
- net LCD_DC: track 0.00 -> 82.6 mm, vias 0 -> 2
- net LCD_CS: track 0.00 -> 79.0 mm, vias 0 -> 2
- net I2C0_SCL: track 0.00 -> 78.5 mm, vias 0 -> 2
- net LCD_SCLK: track 0.00 -> 77.2 mm, vias 0 -> 2
- net LCD_BL: track 0.00 -> 76.2 mm, vias 0 -> 2
- net UART0_RX: track 0.00 -> 75.7 mm, vias 0 -> 4
- net I2C0_SDA: track 0.00 -> 74.0 mm, vias 0 -> 2
- net LCD_MOSI: track 0.00 -> 73.8 mm, vias 0 -> 2
- net UART0_TX: track 0.00 -> 73.3 mm, vias 0 -> 2
- net KEY_1: track 0.00 -> 68.0 mm, vias 0 -> 2
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Other:
- board size 66 x 83 mm -> 47 x 83 mm
- board text added: "R4"
- board text added: "R7"

Commit message: update readme
Other:
- outline, holes or cut-outs redrawn

Commit message: update repo to Rev2.0
Parts:
- IC6: value CAT24C256HU4IGT3 -> CAT24C512HU5IGT3
Changed lines of the file:
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@@
 <drawing>
 <settings>
-<setting alwaysvectorfont="yes"/>
+<setting alwaysvectorfont="no"/>
 <setting verticaltext="up"/>
 </settings>
@@
 <layer number="37" name="tTest" color="7" fill="1" visible="no" active="yes"/>
 <layer number="38" name="bTest" color="7" fill="1" visible="no" active="yes"/>
-<layer number="39" name="tKeepout" color="4" fill="11" visible="yes" active="yes"/>
-<layer number="40" name="bKeepout" color="1" fill="11" visible="yes" active="yes"/>
-<layer number="41" name="tRestrict" color="4" fill="10" visible="yes" active="yes"/>
-<layer number="42" name="bRestrict" color="1" fill="10" visible="yes" active="yes"/>
+<layer number="39" name="tKeepout" color="4" fill="11" visible="no" active="yes"/>
+<layer number="40" name="bKeepout" color="1" fill="11" visible="no" active="yes"/>
+<layer number="41" name="tRestrict" color="4" fill="10" visible="no" active="yes"/>
+<layer number="42" name="bRestrict" color="1" fill="10" visible="no" active="yes"/>
 <layer number="43" name="vRestrict" color="2" fill="10" visible="no" active="yes"/>
 <layer number="44" name="Drills" color="7" fill="1" visible="no" active="yes"/>
@@
 <attribute name="VALUE" x="33.415" y="63.92" size="1.27" layer="27" rot="R270" align="top-center"/>
 </element>
-<element name="IC6" library="ds_ic_memory" package="SON50P300X200X50-9T130X140N" package3d_urn="urn:adsk.eagle:package:45817778/1" value="CAT24C256HU4IGT3" x="28.486" y="71.328" smashed="yes">
+<element name="IC6" library="ds_ic_memory" package="SON50P300X200X50-9T130X140N" package3d_urn="urn:adsk.eagle:package:45817778/1" value="CAT24C512HU5IGT3" x="28.486" y="71.328" smashed="yes">
 <attribute name="NAME" x="28.0344" y="68.6266" size="1.27" layer="25" align="bottom-center"/>
 <attribute name="VALUE" x="28.486" y="69.494" size="1.27" layer="27" align="top-center"/>
