File: src/HardwareDesign/Controller-Board_Rack-PDU_2.0.sch (EAGLE design)
At the start: 144 parts, among them IC1 W5500, IC2 RP2040, IC3 MCP6001AIDBVRG, IC4 W25Q128JVPIQ, IC5 MP2315S, IC6 CAT24C256HU4IGT3, IC7 MP2315GJ-Z, IC8 MCP23S18-E/MJ, SW3 TP, SW5 TP, X1 XC53M4-25.000-F18NJDTL, X2 K5A1200015304P

Commit message: working on Rev2.0
Parts:
- removed 3V3DC, 5VDC, GND, GND-3, GND-5, SW3, SW5, VFB3, VFB5: TP, ds_passive:TP
- removed C43, C52: 33pF, ds_passive:C0402
- removed C44, C45: CL31A226KAHNNNE - 22uF 25V, ds_passive:C-1206
- removed C46, C47, C53, C57: CL31A226KPHNNNE - 22uF - 10V, ds_passive:C-1206
- removed C48, C49, C51: 100nF, ds_passive:C0402
- removed C55, C56: 100nF, ds_passive:C-0402
- removed IC7: MP2315GJ-Z, ds_ic_vreg:MP2315TSOT23-8
- removed IC8: MCP23S18-E/MJ, ds_ic_peripherals:MCP23S18
- removed J1, J3: (no value), ds_con:CON-2X7
- removed L2: 4.9uH, ds_passive:L
- removed L3: 4.2uH, ds_passive:L
- removed R29, R45: 100K, ds_passive:R0402
- removed R30, R31: 499K, ds_passive:R0402
- removed R32, R37: 7.5K, ds_passive:R0402
- removed R33: 9.09K, ds_passive:R0402
- removed R34, R41: 10R, ds_passive:R0402
- removed R35: 20K, ds_passive:R0402
- removed R36, R43: 40.2K, ds_passive:R0402
- removed R42: 33K, ds_passive:R0402
- removed R44: 12.7K, ds_passive:R0402
- added C41: 10uF, ds_passive:C0805
- C36: value 100nF -> 10uF; device ds_passive:C0402 -> ds_passive:C0805
- IC5: value MP2315S -> MIC5504-3.3YM5-TR; device ds_ic_vreg:MP2315TSOT23-8 -> ds_ic_vreg:MIC5504-3.3YM5-TR
- J2: value (none) -> 68714014022; device ds_con:CON-2X7 -> Wurth_Connectors_WR-FPC:6871XX14022_68714014022
Connections:
- removed net N$11: IC5.BST, R41.2
- removed net N$12: IC5.AAM, R32.1, R45.2
- removed net N$13: IC7.AAM, R29.2, R33.1
- removed net N$15: IC7.EN, R31.2
- removed net N$16: C49.1, IC7.VCC, R29.1
- removed net N$20: IC5.FB, R42.1
- removed net N$21: C42.2, IC5.SW, L3.1, SW3.P$1
- removed net N$22: C42.1, R41.1
- removed net N$24: C43.2, R42.2, R43.2, R44.1, VFB3.P$1
- removed net N$26: IC5.EN, R30.2
- removed net N$31: C40.1, IC5.VCC, R45.1
- removed net N$33: IC7.BST, R34.2
- removed net N$34: IC7.FB, R35.1
- removed net N$35: C51.2, IC7.SW, L2.1, SW5.P$1
- removed net N$36: C51.1, R34.1
- removed net N$37: C52.2, R35.2, R36.2, R37.1, VFB5.P$1
- removed net REL_0: IC8.GPA0, J1.12
- removed net REL_1: IC8.GPA1, J1.11
- removed net REL_2: IC8.GPA2, J1.10
- removed net REL_3: IC8.GPA3, J1.9
- removed net REL_4: IC8.GPA4, J1.8
- removed net REL_5: IC8.GPA5, J1.7
- removed net REL_6: IC8.GPA6, J1.6
- removed net REL_7: IC8.GPA7, J1.5
- net !SPI1_CS: no longer IC8.!CS
- net !SPI1_CS_S: now also J2.21; no longer J2.11
- net +12V: no longer C36.1, C44.1, C45.1, C48.1, IC5.IN, IC7.IN, J1.14, R30.1, R31.1
- net +3V3: now also C41.1, C42.1, IC5.VOUT, J2.1, J2.2; no longer 3V3DC.P$1, C43.1, C47.1, C55.1, C56.1, C57.1, IC8.VDD, J1.1, J2.3, J3.3, L3.2, R43.1
- net +5V: now also J2.3; no longer 5VDC.P$1, C46.1, C52.1, C53.1, J1.2, J3.4, L2.2, R36.1
- net DIO_RESET: no longer IC8.!RESET
- net DSP_RES: now also J2.9; no longer J3.9
- net EXP_RST: now also J2.23; no longer J3.11
- net GND: now also C41.2, C42.2, J2.10, J2.12, J2.17, J2.22, J2.5, J2.8, J2.Z1, J2.Z2; no longer C44.2, C45.2, C46.2, C47.2, C48.2, C49.2, C53.2, C55.2, C56.2, C57.2, GND-3.P$1, GND-5.P$1, GND.P$1, IC7.GND, IC8.VSS, J1.13, J2.1, J2.13, J2.14, J2.2, J3.1, J3.13, J3.14, J3.2, R32.2, R33.2, R37.2, R44.2
- net I2C0_SCL: now also J2.7; no longer J3.7
- net I2C0_SDA: now also J2.6; no longer J3.5
- net I_MEA/TX: no longer J1.4
- net KEY_0: now also J2.13; no longer J3.6
- net KEY_1: now also J2.14; no longer J3.8
- net KEY_2: now also J2.15; no longer J3.10
- net KEY_3: now also J2.16; no longer J3.12
- net SPI1_MISO: now also J2.19; no longer IC8.SO, J2.7
- net SPI1_MOSI: now also J2.18; no longer IC8.SI, J2.5
- net SPI1_SCK: now also J2.20; no longer IC8.SCK, J2.9
- net UART0_RX: now also J2.25
- net UART0_TX: now also J2.26
- net VBUS: now also C36.1, C40.1, IC5.EN, IC5.VIN
- net V_MEA/RX: no longer J1.3
Other:
- note added: "BOARD CONNECTOR"
- note removed: "3.3V DC-DC CONVERTER"
- note removed: "5V DC-DC CONVERTER"
- note removed: "OUTPUT INTERFACES"
- note removed: "RELAY DRIVER - PORT EXPANDER"
- moved on the sheet: C1, C10, C11, C12, C13, C14, C15, C16, C17, C18, C2, C3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

Commit message: working on Rev2.0
Parts:
- removed 12VFB: TP, ds_passive:TP
- removed J2: 68714014022, Wurth_Connectors_WR-FPC:6871XX14022_68714014022
- removed R46, R47: 0R, ds_passive:R0402
- removed R48: 100K, ds_passive:R0402
- removed R49: 10K, ds_passive:R0402
- added DISPBOARD, RELAYBOARD: 687320124422, Wurth_Connectors_WR-FPC:6873XX124422_687320124422
- IC3: value MCP6001AIDBVRG -> MCP6001R
Connections:
- removed net +12V: R48.2
- removed net DIO_RESET: IC2.GPIO7
- removed net EXP_RST: IC2.GPIO23, J2.23
- removed net I_MEA/TX: IC2.GPIO28/ADC2, R46.1
- removed net N$8: IC1.XO, R12.2
- removed net N$9: IC1.XI, R13.2
- removed net PWR_DETECT: 12VFB.P$1, IC2.GPIO29/ADC3, R48.1, R49.2
- removed net V_MEA/RX: IC2.GPIO27/ADC1, R47.1
- new net +12V_MEA: IC2.GPIO29/ADC3, RELAYBOARD.13
- new net MCP_DSP_RST: DISPBOARD.20, IC2.GPIO7
- new net MCP_REL_RST: IC2.GPIO23, RELAYBOARD.15
- new net XO: IC1.XO, R12.2, R13.2
- net !SPI1_CS_S: now also DISPBOARD.18; no longer J2.21
- net +3V3: now also DISPBOARD.1, DISPBOARD.2, RELAYBOARD.4, RELAYBOARD.5, RELAYBOARD.6; no longer J2.1, J2.2
- net +5V: now also DISPBOARD.3, DISPBOARD.4, RELAYBOARD.1, RELAYBOARD.2, RELAYBOARD.3; no longer J2.3, J2.4
- net DSP_RES: now also DISPBOARD.9; no longer J2.9
- net GND: now also DISPBOARD.14, DISPBOARD.19, DISPBOARD.5, DISPBOARD.8, DISPBOARD.Z1, DISPBOARD.Z2, DISPBOARD.Z3, DISPBOARD.Z4, RELAYBOARD.12, RELAYBOARD.14, RELAYBOARD.16, RELAYBOARD.9, RELAYBOARD.Z1, RELAYBOARD.Z2, RELAYBOARD.Z3, RELAYBOARD.Z4; no longer J2.10, J2.12, J2.17, J2.22, J2.5, J2.8, J2.Z1, J2.Z2, R49.1
- net I2C0_SCL: now also DISPBOARD.7; no longer J2.7
- net I2C0_SDA: now also DISPBOARD.6; no longer J2.6
- net I2C1_SCL: now also RELAYBOARD.8
- net I2C1_SDA: now also RELAYBOARD.7
- net KEY_0: now also DISPBOARD.10; no longer J2.13
- net KEY_1: now also DISPBOARD.11; no longer J2.14
- net KEY_2: now also DISPBOARD.12; no longer J2.15
- net KEY_3: now also DISPBOARD.13; no longer J2.16
- net N$7: now also IC1.XI
- net SPI1_MISO: now also DISPBOARD.16; no longer J2.19
- net SPI1_MOSI: now also DISPBOARD.15; no longer J2.18
- net SPI1_SCK: now also DISPBOARD.17; no longer J2.20
- net UART0_RX: now also RELAYBOARD.10; no longer J2.25, R47.2
- net UART0_TX: now also RELAYBOARD.11; no longer J2.26, R46.2
Other:
- note added: "3.3 VBUS-LDO"
- note added: "DISPALY SPI"
- note added: "DSP I2C"
- note added: "NETWORK SPI"
- note added: "PUSHBUTTONS"
- note added: "REL I2C"
- note added: "Rev 2.0"
- note removed: "Rev 1.0"

Commit message: finished with design update for 2.0
Connections:
- net !SPI1_CS_S renamed LCD_DC
- net SPI1_SCK renamed LCD_SCLK
- removed net !SPI1_CS: IC2.GPIO9
- removed net DSP_RES: DISPBOARD.9, IC2.GPIO22
- removed net SPI1_MISO: DISPBOARD.16, IC2.GPIO8
- removed net SPI1_MOSI: DISPBOARD.15, IC2.GPIO11
- new net LCD_BL: DISPBOARD.13, IC2.GPIO7
- new net LCD_CS: DISPBOARD.19, IC2.GPIO9
- new net LCD_MISO: DISPBOARD.15, IC2.GPIO8
- new net LCD_MOSI: DISPBOARD.16, IC2.GPIO11
- new net LCD_RES: DISPBOARD.14, IC2.GPIO22
- net GND: no longer DISPBOARD.14, DISPBOARD.19
- net KEY_0: now also DISPBOARD.12; no longer DISPBOARD.10
- net KEY_2: now also DISPBOARD.10; no longer DISPBOARD.12
- net KEY_3: now also DISPBOARD.9; no longer DISPBOARD.13
- net MCP_DSP_RST: now also IC2.GPIO24; no longer IC2.GPIO7

Commit message: finished Rev2
Parts:
- removed R12: 0R, ds_passive:R0402
- removed USB_BOOT: B3U-1000P-B, 52101-101-REV-A_v16:SWITCH-OMRON_B3U-1000P
- added BOOT: 430182043816, Wurth_Switch_WS-TASV:430182043816
- RESET: value B3U-1000P-B -> 430182043816; device 52101-101-REV-A_v16:SWITCH-OMRON_B3U-1000P -> Wurth_Switch_WS-TASV:430182043816
Connections:
- removed net N$6: C8.1, R12.1, X1.CON
- net GND: now also BOOT.3, BOOT.4, RESET.1, RESET.2; no longer RESET.S, USB_BOOT.S
- net N$17: now also RESET.3, RESET.4; no longer RESET.P
- net USB_BOOT: now also BOOT.1, BOOT.2; no longer USB_BOOT.P
- net XO: now also C8.1, X1.CON; no longer R12.2
Changed lines of the file:
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@@
 <part name="GND8" library="ds_passive" deviceset="GND" device=""/>
 <part name="GND9" library="ds_passive" deviceset="GND" device=""/>
-<part name="R12" library="ds_passive" deviceset="R" device="0402" package3d_urn="urn:adsk.eagle:package:46683744/2" value="0R"/>
 <part name="R13" library="ds_passive" deviceset="R" device="0402" package3d_urn="urn:adsk.eagle:package:46683744/2" value="1M"/>
 <part name="R14" library="ds_passive" deviceset="R" device="0402" package3d_urn="urn:adsk.eagle:package:46683744/2" value="4.7K"/>
@@
 <part name="GND30" library="ds_passive" deviceset="GND" device=""/>
 <part name="GND31" library="ds_passive" deviceset="GND" device=""/>
-<part name="USB_BOOT" library="52101-101-REV-A_v16" library_urn="urn:adsk.eagle:library:21899384" deviceset="SWITCH-OMRON_B3U-1000P" device="" package3d_urn="urn:adsk.eagle:package:15662278/2" value="B3U-1000P-B"/>
 <part name="GND37" library="ds_passive" deviceset="GND" device=""/>
 <part name="DBG2" library="ds_con" deviceset="CON-1X4" device="" package3d_urn="urn:adsk.eagle:package:46684991/2"/>
@@
 <part name="GND67" library="ds_passive" library_urn="urn:adsk.eagle:library:46685041" deviceset="GND" device=""/>
 <part name="R40" library="ds_passive" deviceset="R" device="0402" package3d_urn="urn:adsk.eagle:package:46683744/2" value="470R"/>
-<part name="RESET" library="52101-101-REV-A_v16" library_urn="urn:adsk.eagle:library:21899384" deviceset="SWITCH-OMRON_B3U-1000P" device="" package3d_urn="urn:adsk.eagle:package:15662278/2" value="B3U-1000P-B"/>
 <part name="GND50" library="ds_passive" deviceset="GND" device=""/>
 <part name="R50" library="ds_passive" library_urn="urn:adsk.eagle:library:46685041" deviceset="R" device="0402" package3d_urn="urn:adsk.eagle:package:46683744/2" value="10K"/>
@@
 <part name="NC20" library="ds_passive" deviceset="NC" device=""/>
 <part name="DISPBOARD" library="Wurth_Connectors_WR-FPC" library_urn="urn:adsk.eagle:library:15778639" deviceset="6873XX124422_687320124422" device="" package3d_urn="urn:adsk.eagle:package:15743882/4" value="687320124422"/>
+<part name="BOOT" library="Wurth_Switch_WS-TASV" library_urn="urn:adsk.eagle:library:18304196" deviceset="430182043816" device="" package3d_urn="urn:adsk.eagle:package:18304300/2" value="430182043816"/>
+<part name="RESET" library="Wurth_Switch_WS-TASV" library_urn="urn:adsk.eagle:library:18304196" deviceset="430182043816" device="" package3d_urn="urn:adsk.eagle:package:18304300/2" value="430182043816"/>
 </parts>
 <sheets>
@@
 <attribute name="VALUE" x="330.2" y="200.66" size="1.778" layer="96" align="top-center"/>
 </instance>
-<instance part="USB_BOOT" gate="G$1" x="81.28" y="124.46" smashed="yes" rot="R270">
-<attribute name="NAME" x="79.375" y="130.81" size="1.778" layer="95"/>
-<attribute name="VALUE" x="84.455" y="128.27" size="1.778" layer="96"/>
-</instance>
 <instance part="GND37" gate="1" x="91.44" y="119.38" smashed="yes">
 <attribute name="VALUE" x="91.44" y="116.84" size="1.778" layer="96" align="top-center"/>
@@
 <attribute name="VALUE" x="198.12" y="27.94" size="1.778" layer="96" align="top-center"/>
 </instance>
-<instance part="RESET" gate="G$1" x="109.22" y="213.36" smashed="yes" rot="MR270">
-<attribute name="NAME" x="111.125" y="219.71" size="1.778" layer="95" rot="MR0"/>
-<attribute name="VALUE" x="106.045" y="217.17" size="1.778" layer="96" rot="MR0"/>
-</instance>
 <instance part="GND50" gate="1" x="99.06" y="208.28" smashed="yes" rot="MR0">
 <attribute name="VALUE" x="99.06" y="205.74" size="1.778" layer="96" rot="MR0" align="top-center"/>
@@
 <instance part="NC21" gate="G$1" x="187.96" y="137.16" smashed="yes"/>
 <instance part="NC22" gate="G$1" x="187.96" y="134.62" smashed="yes"/>
+<instance part="BOOT" gate="G$1" x="83.82" y="127" smashed="yes">
+<attribute name="NAME" x="83.82" y="132.842" size="1.778" layer="95" align="bottom-center"/>
+<attribute name="VALUE" x="81.28" y="121.92" size="1.778" layer="96" align="bottom-center"/>
+</instance>
+<instance part="RESET" gate="G$1" x="109.22" y="215.9" smashed="yes">
+<attribute name="NAME" x="109.22" y="221.742" size="1.778" layer="95" align="bottom-center"/>
+<attribute name="VALUE" x="109.22" y="210.82" size="1.778" layer="96" align="bottom-center"/>
+</instance>
 </instances>
 <busses>
@@
 </segment>
 <segment>
-<pinref part="USB_BOOT" gate="G$1" pin="S"/>
-<wire x1="86.36" y1="124.46" x2="91.44" y2="124.46" width="0.1524" layer="91"/>
+<wire x1="88.9" y1="124.46" x2="91.44" y2="124.46" width="0.1524" layer="91"/>
 <wire x1="91.44" y1="124.46" x2="91.44" y2="121.92" width="0.1524" layer="91"/>
 <pinref part="GND37" gate="1" pin="GND"/>
+<pinref part="BOOT" gate="G$1" pin="4"/>
+<pinref part="BOOT" gate="G$1" pin="3"/>
+<wire x1="88.9" y1="132.08" x2="91.44" y2="132.08" width="0.1524" layer="91"/>
+<wire x1="91.44" y1="132.08" x2="91.44" y2="124.46" width="0.1524" layer="91"/>
+<junction x="91.44" y="124.46"/>
 </segment>
 <segment>
@@
 </segment>
 <segment>
-<pinref part="RESET" gate="G$1" pin="S"/>
 <wire x1="104.14" y1="213.36" x2="99.06" y2="213.36" width="0.1524" layer="91"/>
 <wire x1="99.06" y1="213.36" x2="99.06" y2="210.82" width="0.1524" layer="91"/>
 <pinref part="GND50" gate="1" pin="GND"/>
+<pinref part="RESET" gate="G$1" pin="2"/>
+<pinref part="RESET" gate="G$1" pin="1"/>
+<wire x1="104.14" y1="220.98" x2="99.06" y2="220.98" width="0.1524" layer="91"/>
+<wire x1="99.06" y1="220.98" x2="99.06" y2="213.36" width="0.1524" layer="91"/>
+<junction x="99.06" y="213.36"/>
 </segment>
 </net>
@@
 </segment>
 <segment>
-<pinref part="USB_BOOT" gate="G$1" pin="P"/>
-<wire x1="76.2" y1="124.46" x2="68.58" y2="124.46" width="0.1524" layer="91"/>
+<wire x1="78.74" y1="124.46" x2="73.66" y2="124.46" width="0.1524" layer="91"/>
 <label x="68.58" y="124.46" size="1.27" layer="95" rot="R180" xref="yes"/>
+<pinref part="BOOT" gate="G$1" pin="2"/>
+<pinref part="BOOT" gate="G$1" pin="1"/>
+<wire x1="73.66" y1="124.46" x2="68.58" y2="124.46" width="0.1524" layer="91"/>
+<wire x1="78.74" y1="132.08" x2="73.66" y2="132.08" width="0.1524" layer="91"/>
+<wire x1="73.66" y1="132.08" x2="73.66" y2="124.46" width="0.1524" layer="91"/>
+<junction x="73.66" y="124.46"/>
 </segment>
 </net>
@@
 <net name="N$17" class="0">
 <segment>
-<pinref part="RESET" gate="G$1" pin="P"/>
 <pinref part="IC2" gate="G$1" pin="RUN"/>
-<wire x1="114.3" y1="213.36" x2="121.92" y2="213.36" width="0.1524" layer="91"/>
+<wire x1="114.3" y1="213.36" x2="116.84" y2="213.36" width="0.1524" layer="91"/>
+<wire x1="116.84" y1="213.36" x2="121.92" y2="213.36" width="0.1524" layer="91"/>
 <wire x1="121.92" y1="213.36" x2="137.16" y2="213.36" width="0.1524" layer="91"/>
 <wire x1="121.92" y1="213.36" x2="121.92" y2="215.9" width="0.1524" layer="91"/>
 <junction x="121.92" y="213.36"/>
 <pinref part="R50" gate="G$1" pin="2"/>
+<pinref part="RESET" gate="G$1" pin="4"/>
+<pinref part="RESET" gate="G$1" pin="3"/>
+<wire x1="114.3" y1="220.98" x2="116.84" y2="220.98" width="0.1524" layer="91"/>
+<wire x1="116.84" y1="220.98" x2="116.84" y2="213.36" width="0.1524" layer="91"/>
+<junction x="116.84" y="213.36"/>
 </segment>
 </net>
@@
 <instance part="GND9" gate="1" x="81.28" y="165.1" smashed="yes">
 <attribute name="VALUE" x="81.28" y="162.56" size="1.778" layer="96" align="top-center"/>
-</instance>
-<instance part="R12" gate="G$1" x="66.04" y="200.66" smashed="yes" rot="R90">
-<attribute name="NAME" x="60.325" y="202.1586" size="1.778" layer="95"/>
-<attribute name="VALUE" x="66.675" y="202.1586" size="1.778" layer="96"/>
 </instance>
 <instance part="R13" gate="G$1" x="81.28" y="193.04" smashed="yes" rot="MR180">
@@
 </segment>
 </net>
-<net name="N$6" class="0">
-<segment>
-<pinref part="X1" gate="G$1" pin="CON"/>
-<pinref part="C8" gate="G$1" pin="1"/>
-<wire x1="55.88" y1="185.42" x2="50.8" y2="185.42" width="0.1524" layer="91"/>
-<wire x1="50.8" y1="185.42" x2="50.8" y2="182.88" width="0.1524" layer="91"/>
-<pinref part="R12" gate="G$1" pin="1"/>
-<wire x1="60.96" y1="200.66" x2="50.8" y2="200.66" width="0.1524" layer="91"/>
-<wire x1="50.8" y1="200.66" x2="50.8" y2="185.42" width="0.1524" layer="91"/>
-<junction x="50.8" y="185.42"/>
-</segment>
-</net>
 <net name="N$7" class="0">
 <segment>
@@
 <net name="XO" class="0">
 <segment>
-<pinref part="R12" gate="G$1" pin="2"/>
 <pinref part="IC1" gate="G$1" pin="XO"/>
-<wire x1="71.12" y1="200.66" x2="81.28" y2="200.66" width="0.1524" layer="91"/>
 <pinref part="R13" gate="G$1" pin="2"/>
 <wire x1="81.28" y1="200.66" x2="124.46" y2="200.66" width="0.1524" layer="91"/>
 <wire x1="81.28" y1="200.66" x2="81.28" y2="198.12" width="0.1524" layer="91"/>
 <junction x="81.28" y="200.66"/>
-</segment>
-</net>
+<pinref part="X1" gate="G$1" pin="CON"/>
+<pinref part="C8" gate="G$1" pin="1"/>
+<wire x1="55.88" y1="185.42" x2="50.8" y2="185.42" width="0.1524" layer="91"/>
+<wire x1="50.8" y1="185.42" x2="50.8" y2="182.88" width="0.1524" layer="91"/>
+<wire x1="50.8" y1="200.66" x2="50.8" y2="185.42" width="0.1524" layer="91"/>
+<junction x="50.8" y="185.42"/>
+<wire x1="50.8" y1="200.66" x2="81.28" y2="200.66" width="0.1524" layer="91"/>
+</segment>
+</net>

Commit message: update repo to Rev2.0
Parts:
- IC6: value CAT24C256HU4IGT3 -> CAT24C512HU5IGT3
Changed lines of the file:
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@@
 <part name="GND39" library="ds_passive" library_urn="urn:adsk.eagle:library:46685041" deviceset="GND" device=""/>
 <part name="NC17" library="ds_passive" deviceset="NC" device=""/>
-<part name="IC6" library="ds_ic_memory" deviceset="CAT24C256" device="-HU4" package3d_urn="urn:adsk.eagle:package:45817778/1" value="CAT24C256HU4IGT3"/>
+<part name="IC6" library="ds_ic_memory" deviceset="CAT24C256" device="-HU4" package3d_urn="urn:adsk.eagle:package:45817778/1" value="CAT24C512HU5IGT3"/>
 <part name="R27" library="ds_passive" deviceset="R" device="0402" package3d_urn="urn:adsk.eagle:package:46683744/2" value="4.7K"/>
 <part name="R28" library="ds_passive" deviceset="R" device="0402" package3d_urn="urn:adsk.eagle:package:46683744/2" value="4.7K"/>
