File: src/HardwareDesign/Display-Board_Rack-PDU_2.0.sch (EAGLE design)
At the start: 41 parts, among them CON1 3.5IN_TFTLCD, IC1 MCP23S18-E/MJ, T1 BSS138

Commit message: working on Rev2.0
Parts:
- removed CON1: 3.5IN_TFTLCD, ds_displays:3.5IN_TFTLCD
- removed CON3, CON4: (no value), ds_con:CON-2X72
- removed IC1: MCP23S18-E/MJ, ds_ic_peripherals:MCP23S18
- added IC2: MCP23017-E/ML, ds_ic_peripherals:MCP23017-E/ML
- added J1, J2: 68714014022, Wurth_Connectors_WR-FPC:6871XX14022_68714014022
- added R2, R3: 330R, ds_passive:R0402
- R1: value 10K -> 330R
Connections:
- removed net CS: CON1.CS/SPI_CS
- removed net MISO: CON1.SPI_SDO
- removed net MOSI: CON1.SPI_SDA
- removed net N$42: CON4.6
- removed net N$43: CON4.8
- removed net N$44: CON4.10
- removed net N$45: CON4.12
- removed net RES: CON1.RESET
- removed net SCLK: CON1.WR/SPI_AO
- removed net SPI_SCK: CON4.9, IC1.SCK
- new net BCKL: IC2.IO2.3, T1.G
- new net N$10: J2.38
- new net N$11: J2.37
- new net N$4: R1.1, R2.1, R3.1, T1.D
- new net SPI_SCLK: J1.11, J2.20
- net +3V3: now also IC2.VDD, J1.12, J1.38, J1.39, J1.40, J1.6, J1.7, J2.1, J2.2; no longer CON1.A, CON1.IM0, CON1.IM1, CON1.IM2, CON1.RD, CON1.VCC(3V3)@1, CON1.VCC(3V3)@2, CON3.3, CON4.3, IC1.VDD
- net +5V: now also J1.33, J2.3, J2.4; no longer CON3.4, CON4.4
- net DSP_RES: now also J1.15, J2.9; no longer CON3.9
- net EXP_RST: now also IC2.!RESET, J2.23; no longer CON3.11, IC1.!RESET
- net GND: now also IC2.A0, IC2.A1, IC2.A2, IC2.VSS, J1.16, J1.17, J1.18, J1.19, J1.20, J1.21, J1.22, J1.23, J1.24, J1.25, J1.26, J1.27, J1.28, J1.29, J1.30, J1.31, J1.32, J1.37, J1.5, J1.Z1, J1.Z2, J2.10, J2.12, J2.17, J2.22, J2.5, J2.8, J2.Z1, J2.Z2, T1.S; no longer CON1.DB0, CON1.DB1, CON1.DB10, CON1.DB11, CON1.DB12, CON1.DB13, CON1.DB14, CON1.DB15, CON1.DB2, CON1.DB3, CON1.DB4, CON1.DB5, CON1.DB6, CON1.DB7, CON1.DB8, CON1.DB9, CON1.GND@1, CON1.GND@2, CON1.GND@3, CON3.1, CON3.13, CON3.14, CON3.2, CON4.1, CON4.13, CON4.14, CON4.2, IC1.VSS
- net I2C_SCL: now also IC2.SCL, J2.7; no longer CON3.7
- net I2C_SDA: now also IC2.SDA, J2.6; no longer CON3.5
- net KEY_0: now also J2.13; no longer CON3.6
- net KEY_1: now also J2.14; no longer CON3.8
- net KEY_2: now also J2.15; no longer CON3.10
- net KEY_3: now also J2.16; no longer CON3.12
- net N$1: now also J1.10; no longer CON1.RS/SPI_SCL
- net N$2: now also J1.35, R2.2; no longer CON1.K2
- net N$3: now also J1.36, R3.2; no longer CON1.K3
- net N$46: now also IC2.IO2.1; no longer IC1.GPB1
- net N$47: now also IC2.IO2.2; no longer IC1.GPB2
- net N$48: now also IC2.IO2.0; no longer IC1.GPB0
- net N$5: now also J1.34; no longer CON1.K1
- net N$50: now also IC2.IO1.0; no longer IC1.GPA0
- net N$51: now also IC2.IO1.1; no longer IC1.GPA1
- net N$52: now also IC2.IO1.2; no longer IC1.GPA2
- net N$53: now also IC2.IO1.3; no longer IC1.GPA3
- net N$54: now also IC2.IO1.4; no longer IC1.GPA4
- net N$55: now also IC2.IO1.5; no longer IC1.GPA5
- net N$56: now also IC2.IO1.6; no longer IC1.GPA6
- net N$57: now also IC2.IO1.7; no longer IC1.GPA7
- net SPI_CS: now also J1.9, J2.21; no longer CON4.11, IC1.!CS
- net SPI_MISO: now also J1.14, J2.19; no longer CON4.7, IC1.SO
- net SPI_MOSI: now also J1.13, J2.18; no longer CON4.5, IC1.SI
Other:
- note added: "3.5-IN LCD"
- note added: "BOARD CONNECTOR"
- note added: "IO DRIVER"
- note added: "Rev 2.0"
- note removed: "128x64 OLED"
- note removed: "BOARD CONNECTORS"
- note removed: "Rev 1.0"
- note removed: "STATUS LED DRIVER"
- moved on the sheet: BUT+1, BUT-1, BUT_PWR1, BUT_SET1, C1, C15, C16, C17, C18, C19, C2, C20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

Commit message: working on Rev2.0
Parts:
- removed J2: 68714014022, Wurth_Connectors_WR-FPC:6871XX14022_68714014022
- added DISPBOARD: 687320124422, Wurth_Connectors_WR-FPC:6873XX124422_687320124422
Connections:
- removed net EXP_RST: IC2.!RESET, J2.23
- removed net N$10: J2.38
- removed net N$11: J2.37
- new net MCP_DSP_RST: DISPBOARD.20, IC2.!RESET
- net +3V3: now also DISPBOARD.1, DISPBOARD.2, IC2.A0; no longer J2.1, J2.2
- net +5V: now also DISPBOARD.3, DISPBOARD.4; no longer J2.3, J2.4
- net DSP_RES: now also DISPBOARD.9; no longer J2.9
- net GND: now also DISPBOARD.14, DISPBOARD.19, DISPBOARD.5, DISPBOARD.8, DISPBOARD.Z1, DISPBOARD.Z2, DISPBOARD.Z3, DISPBOARD.Z4; no longer IC2.A0, J2.10, J2.12, J2.17, J2.22, J2.5, J2.8, J2.Z1, J2.Z2
- net I2C_SCL: now also DISPBOARD.7; no longer J2.7
- net I2C_SDA: now also DISPBOARD.6; no longer J2.6
- net KEY_0: now also DISPBOARD.10; no longer J2.13
- net KEY_1: now also DISPBOARD.11; no longer J2.14
- net KEY_2: now also DISPBOARD.12; no longer J2.15
- net KEY_3: now also DISPBOARD.13; no longer J2.16
- net SPI_CS: now also DISPBOARD.18; no longer J2.21
- net SPI_MISO: now also DISPBOARD.16; no longer J2.19
- net SPI_MOSI: now also DISPBOARD.15; no longer J2.18
- net SPI_SCLK: now also DISPBOARD.17; no longer J2.20
Other:
- moved on the sheet: C1, C15, C16, C2, J1, R1, R17, R2, R3, T1

Commit message: finished with design update for 2.0
Parts:
- removed J1: 68714014022, Wurth_Connectors_WR-FPC:6871XX14022_68714014022
- removed R17: 10K, ds_passive:R0402
- added 3V3, 5V, BL, CS, DC, GND, I2C_SCL, I2C_SDA, KEY0, KEY1, KEY2, KEY3, LCD_RES, MCP_RES, MISO, MOSI, SCK: TP, ds_passive:TP
- added R4: 10K, ds_passive:R0402
- added TFT: FPC40-HD, ds_con:FPC40-HD
- DISPBOARD: value 687320124422 -> FPC20-H; device Wurth_Connectors_WR-FPC:6873XX124422_687320124422 -> ds_con:FPC20-H
- R1, R2, R3: value 330R -> 56R
Connections:
- removed net BCKL: IC2.IO2.3, T1.G
- removed net DSP_RES: DISPBOARD.9, J1.15
- removed net N$1: J1.10, R17.2
- removed net SPI_CS: DISPBOARD.18, J1.9
- removed net SPI_MISO: DISPBOARD.16, J1.14
- removed net SPI_MOSI: DISPBOARD.15, J1.13
- removed net SPI_SCLK: DISPBOARD.17, J1.11
- new net LCD_BL: BL.P$1, DISPBOARD.13, R4.1, T1.G
- new net LCD_CS: CS.P$1, DISPBOARD.19, TFT.9
- new net LCD_DC: DC.P$1, DISPBOARD.18, TFT.10
- new net LCD_MISO: DISPBOARD.15, MISO.P$1, TFT.14
- new net LCD_MOSI: DISPBOARD.16, MOSI.P$1, TFT.13
- new net LCD_RES: DISPBOARD.14, LCD_RES.P$1, TFT.15
- new net LCD_SCLK: DISPBOARD.17, SCK.P$1, TFT.11
- net +3V3: now also 3V3.P$1, TFT.12, TFT.38, TFT.39, TFT.40, TFT.6, TFT.7; no longer J1.12, J1.38, J1.39, J1.40, J1.6, J1.7
- net +5V: now also 5V.P$1, TFT.33; no longer J1.33
- net GND: now also GND.P$1, R4.2, TFT.16, TFT.17, TFT.18, TFT.19, TFT.20, TFT.21, TFT.22, TFT.23, TFT.24, TFT.25, TFT.26, TFT.27, TFT.28, TFT.29, TFT.30, TFT.31, TFT.32, TFT.37, TFT.5, TFT.Z1, TFT.Z2; no longer DISPBOARD.14, DISPBOARD.19, J1.16, J1.17, J1.18, J1.19, J1.20, J1.21, J1.22, J1.23, J1.24, J1.25, J1.26, J1.27, J1.28, J1.29, J1.30, J1.31, J1.32, J1.37, J1.5, J1.Z1, J1.Z2, R17.1
- net I2C_SCL: now also I2C_SCL.P$1
- net I2C_SDA: now also I2C_SDA.P$1
- net KEY_0: now also DISPBOARD.12, KEY0.P$1; no longer DISPBOARD.10
- net KEY_1: now also KEY1.P$1
- net KEY_2: now also DISPBOARD.10, KEY2.P$1; no longer DISPBOARD.12
- net KEY_3: now also DISPBOARD.9, KEY3.P$1; no longer DISPBOARD.13
- net MCP_DSP_RST: now also MCP_RES.P$1
- net N$2: now also TFT.35; no longer J1.35
- net N$3: now also TFT.36; no longer J1.36
- net N$5: now also TFT.34; no longer J1.34
Other:
- note added: "TESTPOINTS"
- moved on the sheet: C1, C15, C16, C2, DISPBOARD, R1, R2, R3, T1

Commit message: update repo to Rev2.0
Changed lines of the file:
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@@
 <instance part="NC5" gate="G$1" x="233.68" y="205.74" smashed="yes" rot="R180"/>
 <instance part="DISPBOARD" gate="G$1" x="124.46" y="198.12" smashed="yes">
-<attribute name="NAME" x="123.19" y="201.168" size="1.27" layer="95" align="bottom-center"/>
+<attribute name="NAME" x="123.952" y="201.93" size="1.27" layer="95" rot="R90" align="bottom-center"/>
 </instance>
 <instance part="NC6" gate="G$1" x="33.02" y="203.2" smashed="yes" rot="MR180"/>
