File: src/HardwareDesign/Relay-Board_Rack-PDU_2.0.brd (EAGLE design)
At the start: 147 x 95 mm, 70 parts, among them IC1 ULN2803A, IC3 TS432ILT, T1 750370228

Commit message: working on Rev2.0
Parts:
- removed CON1: (no value), ds_con:2X7
- added 3V3DC, 5VDC, GND, GND-3, GND-5, SW3, SW5, VFB3, VFB5: TP, ds_passive:TP
- added C1, C2: 100nF, ds_passive:C0402
- added C36, C40, C42, C48, C49, C51: 100nF, ds_passive:0402
- added C43, C52: 33pF, ds_passive:0402
- added C44, C45: 22uF 25V, ds_passive:C1206
- added C46, C47, C53, C57: 22uF - 10V, ds_passive:C1206
- added IC2: MCP23017-E/ML, ds_ic_peripherals:QFN28[6X6]ML
- added IC5: MP2315S, ds_ic_vreg:SOT65P280X110-8N
- added IC7: MP2315GJ-Z, ds_ic_vreg:SOT65P280X110-8N
- added L1: 4.9uH, ds_passive:SRR5228A
- added L3: 4.2uH, ds_passive:SRR5228A
- added R29, R45: 100K, ds_passive:0402
- added R30, R31: 499K, ds_passive:0402
- added R32, R37: 7.5K, ds_passive:0402
- added R33: 9.09K, ds_passive:0402
- added R34, R41: 10R, ds_passive:0402
- added R35: 20K, ds_passive:0402
- added R36, R43: 40.2K, ds_passive:0402
- added R42: 33K, ds_passive:0402
- added R44: 12.7K, ds_passive:0402
- moved R1 61.3 mm to (18.9, 43.1), turned to 180 degrees
- moved R2 48.2 mm to (35.4, 42.5), turned to 180 degrees
- moved R3 35.6 mm to (51.4, 42.5), turned to 180 degrees
- moved R8 33.5 mm to (130.9, 42.6), turned to 180 degrees
- moved IC1 29.3 mm to (90.1, 56.6)
- moved R4 23.5 mm to (67.3, 42.6), turned to 180 degrees
- moved R7 22.1 mm to (115.5, 42.6), turned to 180 degrees
- moved R5 13.7 mm to (83.2, 42.5), turned to 180 degrees
- moved R6 12.6 mm to (99.2, 42.6), turned to 180 degrees
Connections:
- removed net I_MEA/TX: CON1.4
- removed net VMEA/RX: CON1.3
- new net EXP_RST: IC2.14
- new net I2C_SCL: IC2.8
- new net I2C_SDA: IC2.9
- new net N$14: IC7.5, R34.2
- new net N$16: IC7.8, R35.1
- new net N$17: C51.2, IC7.3, L1.1, SW5.TP
- new net N$18: C51.1, R34.1
- new net N$19: IC7.6, R31.2
- new net N$21: C49.1, IC7.7, R29.1
- new net N$37: C52.2, R35.2, R36.2, R37.1, VFB5.TP
- new net N$38: IC5.5, R41.2
- new net N$39: IC5.8, R42.1
- new net N$40: C42.2, IC5.3, L3.1, SW3.TP
- new net N$41: C42.1, R41.1
- new net N$42: C43.2, R42.2, R43.2, R44.1, VFB3.TP
- new net N$43: IC5.6, R30.2
- new net N$44: C40.1, IC5.7, R45.1
- new net N$45: IC7.1, R29.2, R33.1
- new net N$46: IC5.1, R32.1, R45.2
- net +12V: now also C36.1, C44.1, C45.1, C48.1, IC5.2, IC7.2, R30.1, R31.1; no longer CON1.14
- net +3V3: now also 3V3DC.TP, C1.1, C2.1, C43.1, C47.1, C57.1, IC2.5, L3.2, R43.1; no longer CON1.1
- net +5V: now also 5VDC.TP, C46.1, C52.1, C53.1, L1.2, R36.1; no longer CON1.2
- net GND: now also C1.2, C2.2, C36.2, C40.2, C44.2, C45.2, C46.2, C47.2, C48.2, C49.2, C53.2, C57.2, GND-3.TP, GND-5.TP, GND.TP, IC2.11, IC2.12, IC2.13, IC2.6, IC2.PAD, IC5.4, IC7.4, R32.2, R33.2, R37.2, R44.2; no longer CON1.13
- net REL_0: now also IC2.17; no longer CON1.12
- net REL_1: now also IC2.18; no longer CON1.11
- net REL_2: now also IC2.19; no longer CON1.10
- net REL_3: now also IC2.20; no longer CON1.9
- net REL_4: now also IC2.21; no longer CON1.8
- net REL_5: now also IC2.22; no longer CON1.7
- net REL_6: now also IC2.23; no longer CON1.6
- net REL_7: now also IC2.24; no longer CON1.5
Routing:
- net +12V: track 411.9 -> 45.5 mm, vias 4 -> 0
- net GND: track 321.2 -> 193.0 mm, vias 41 -> 27
- net RELAY_1: track 74.6 -> 6.02 mm
- net RELAY_2: track 65.1 -> 5.70 mm
- net N$6: track 54.6 -> 0.00 mm, vias 2 -> 0
- net RELAY_3: track 52.8 -> 0.00 mm
- net N$7: track 50.5 -> 0.00 mm, vias 2 -> 0
- net N$8: track 45.5 -> 0.00 mm, vias 2 -> 0
- net N$9: track 40.6 -> 0.00 mm, vias 2 -> 0
- net RELAY_8: track 44.9 -> 5.63 mm
- net N$10: track 36.0 -> 0.00 mm, vias 2 -> 0
- net RELAY_4: track 39.4 -> 5.65 mm
- net N$11: track 31.0 -> 0.00 mm, vias 2 -> 0
- net N$13: track 26.3 -> 0.00 mm, vias 2 -> 0
- net RELAY_7: track 31.7 -> 5.86 mm
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
Commit message: working on Rev2.0
Parts:
- removed 3V3DC, SW5, VFB3, VFB5: TP, ds_passive:TP
- removed BR1: DBLS207G, ds_active:DIOB_DBLS207G
- removed C45: 22uF 25V, ds_passive:C1206
- removed C46, C47, C53, C57: 22uF - 10V, ds_passive:C1206
- removed C51: 100nF, ds_passive:0402
- removed C52: 33pF, ds_passive:0402
- removed CM1: 20mH CM CHOKE, ds_trafo:WE-CMB_XS_744821120
- removed D15: MRA4007T3G, Diodes:SMA
- removed D16: STPS5H100B, ds_active:DPAK_STM
- removed D17, D18, D19: BAT41ZFILM, diode:SOD-123_MINI-SMA
- removed D20: MMSZ5248B-V-GS08, Diodes-2:DO214AC
- removed F2: 696101000002, Wurth_Connectors_WR-FSH:696101000002
- removed L3: 4.2uH, ds_passive:SRR5228A
- removed REL1, REL2, REL3, REL4, REL5, REL6, REL7, REL8: G2RL-1A-E_DC12, ds_passive:RELAY_G2RL-1A-E_DC5_OMR
- removed RV1: B72210S0321K101, Wurth_EMC Components_WE-VD:WE-VD_10MM_820412001
- removed T1: 750370228, ds_trafo:WE-OLSTM_EE20_L22.2W25H16
- added 12VDC, 3VDC, 3VFB, 5VFB, SW: TP, ds_passive:TP
- added AC/DC1: (no value), ds_trafo:IRM_10_12
- added AC_L, AC_N: (no value), con-wago-500:W237-102
- added C10, C13: 100uF, ds_passive:100UF-16V
- added C11, C12: 33pF, ds_passive:0402
- added C27, C28, C29, C30, C31, C32, C37, C38, C39, C41, C50, C54, C55, C56: 33nF, ds_passive:C1206
- added C3, C4, C6, C7, C8, C9: 100nF, ds_passive:0402
- added C33, C34: 100nF, ds_passive:C0402
- added C5: 10uF 16V, ds_passive:C1206
- added D10, D9: S1M, diode:SMA
- added D11: 9.1V 1W, diode:SMB
- added IC10, IC11, IC12, IC14, IC16, IC6, IC8: HLW8032, ds_ic_peripherals:SO8
- added IC9: SN74HC151PWR, ds_ic_logic:TSSOP16
- added J1: 687320124422, Wurth_Connectors_WR-FPC:687320124422
- added K1, K2, K3, K4, K5, K6, K7, K8: G2RL-1A-E_DC12, ds_passive:RELAY_G2RL-1A-E_DC5_OMR
- added OPT1: TLP291-4, ds_ic_peripherals:SO16
- added R100, R101, R102, R103, R116, R117, R118, R119, R38, R39, R46, R47, R52, R53, R54, R55, R68, R69, R70, R71, R76, R77, R78, R79, R84, R85, R86, R87: 470K, ds_passive:1206
- added R104, R113, R114, R120, R40, R48, R49, R50, R56, R65, R66, R72, R73, R74, R80, R81, R82, R88, R97, R98: 1K 1%, ds_passive:1206
- added R11: 40.2K, ds_passive:0402
- added R115, R25, R26, R27, R28, R51, R67, R75, R83, R99: 0.002R 1%, ds_passive:2512
- added R12: 7.5K, ds_passive:0402
- added R57, R58, R59: JP, ds_passive:0402
- added R60: 470K 1W, ds_passive:2512
- added R61, R62: 100R 1W, ds_passive:2512
- added R63, R64, R89, R90: 4x1K 1206, Resistor Array:742C083103JP
- added R91, R92: 0R, ds_passive:0402
- added R93: 4x10K 1206, Resistor Array:742C083103JP
- added R94: 100K, ds_passive:0402
- added R95: 10K, ds_passive:0402
- added U$3: (no value), ds_passive:2-LAYER
- added Z1: SMAJ15A, 52101-101-REV-A_v16:SUPRESSOR_SMAJ
- C1, C2: value 100nF -> 22uF 25V; device ds_passive:C0402 -> ds_passive:C1206
- C14: value MP2104K27C3R6LC 100nF 275V -> 22uF - 10V; device ds_passive:103-275V -> ds_passive:C1206
- C15, C17: value KM150M400G160A 15uF 400V -> 22uF - 10V; device Capacitor:CAPPRD550W110D1250H2500B -> ds_passive:C1206
- C16: value 1nF 630V -> 100uF; device ds_passive:C1206 -> ds_passive:100UF-16V
- C18: value 470uF 25V -> 22uF - 10V; device Capacitor:CAPPRD508W65D1000H1100B -> ds_passive:C1206
- C19: value 100uF 25V -> 100nF; device Capacitor:CAPPRD508W65D1000H1100B -> ds_passive:C0402
- C20: value 1uF 25V -> 100nF; device ds_passive:C0805 -> ds_passive:C0402
- C21: value 10nF 50V -> 470nF 630V; device ds_passive:C0805 -> ds_passive:2225
- C22: value 2.2nF 50V -> 470uF 25V; device ds_passive:C0603 -> ds_passive:100UF-16V
- C23: value 33nF 16V -> 10uF 16V; device ds_passive:C0603 -> ds_passive:C1206
- C24: value 220pF -> 33nF; device ds_passive:C0805 -> ds_passive:C1206
- C25: value 33uF 35V -> 33nF; device Capacitor:CAPPRD508W65D1000H1100B -> ds_passive:C1206
- C26: value 2.2nF 250VAC -> 33nF; device ds_passive:AR21AC103K4R -> ds_passive:C1206
- C36, C40, C42, C48, C49: value 100nF -> 33nF; device ds_passive:0402 -> ds_passive:C1206
- C43: value 33pF -> 33nF; device ds_passive:0402 -> ds_passive:C1206
- C44: value 22uF 25V -> 33nF
- IC1: value ULN2803A -> MP2315GJ-Z; device ds_ic_peripherals:SO18 -> ds_ic_vreg:SOT65P280X110-8N
- IC2: value MCP23017-E/ML -> MP2315S; device ds_ic_peripherals:QFN28[6X6]ML -> ds_ic_vreg:SOT65P280X110-8N
- IC3: value TS432ILT -> ULN2803A; device ds_ic_vreg:SOT23 -> ds_ic_peripherals:SO18
- IC4: value (none) -> MCP23017-E/ML; device ds_ic_peripherals:VIPER35HD -> ds_ic_peripherals:QFN28[6X6]ML
- IC5: value MP2315S -> BA50BC0FP-E2; device ds_ic_vreg:SOT65P280X110-8N -> ds_ic_vreg:DPAK
- IC7: value MP2315GJ-Z -> HLW8032; device ds_ic_vreg:SOT65P280X110-8N -> ds_ic_peripherals:SO8
- L2: value 3.3uH SD43-332ML -> 4.2uH; device 52101-101-REV-A_v16:INDUCTOR-BOURNS_SRN8040 -> ds_passive:SRR5228A
- OPT2: value SFH6106-2T -> TLP291-4; device ds_ic_peripherals:SMD-4_SFH610X_VIS-M -> ds_ic_peripherals:SO16
- R1, R2: value 330R 1W -> 499K; device ds_passive:1206 -> ds_passive:0402
- R10: value 0R -> 33K; device ds_passive:0805 -> ds_passive:0402
- R13: value 220K 5% 0.33W 200V -> 40.2K; device ds_passive:1206 -> ds_passive:0402
- R14: value 1K -> 12.7K; device ds_passive:0603 -> ds_passive:0402
- R15: value 12K -> 0R; device ds_passive:0603 -> ds_passive:0805
- R16: value 82K -> 0R; device ds_passive:0603 -> ds_passive:0805
- R17: value 130K 1% -> 330R 1W; device ds_passive:0603 -> ds_passive:1206
- R18: value 15K 1% -> 330R 1W; device ds_passive:0603 -> ds_passive:1206
- R19: value 4.7R 1% -> 330R 1W; device ds_passive:0603 -> ds_passive:1206
- R20: value 330K 1% -> 330R 1W; device ds_passive:0603 -> ds_passive:1206
- R21: value 133K 1% -> 330R 1W; device ds_passive:0603 -> ds_passive:1206
- R22: value 30K 1% -> 330R 1W; device ds_passive:0603 -> ds_passive:1206
- R23: value 47K 1% -> 330R 1W; device ds_passive:0603 -> ds_passive:1206
- R24: value 220R -> 330R 1W; device ds_passive:0805 -> ds_passive:1206
- R29: value 100K -> 0.002R 1%; device ds_passive:0402 -> ds_passive:2512
- R3, R5: value 330R 1W -> 100K; device ds_passive:1206 -> ds_passive:0402
- R30, R31: value 499K -> 0.002R 1%; device ds_passive:0402 -> ds_passive:2512
- R32: value 7.5K -> 0.002R 1%; device ds_passive:0402 -> ds_passive:2512
- R33: value 9.09K -> 1K 1%; device ds_passive:0402 -> ds_passive:1206
- R34, R41: value 10R -> 1K 1%; device ds_passive:0402 -> ds_passive:1206
- R35: value 20K -> 0.002R 1%; device ds_passive:0402 -> ds_passive:2512
- R36: value 40.2K -> 470K; device ds_passive:0402 -> ds_passive:1206
- R37: value 7.5K -> 470K; device ds_passive:0402 -> ds_passive:1206
- R4: value 330R 1W -> 9.09K; device ds_passive:1206 -> ds_passive:0402
- R42: value 33K -> 1K 1%; device ds_passive:0402 -> ds_passive:1206
- R43: value 40.2K -> 0.002R 1%; device ds_passive:0402 -> ds_passive:2512
- R44: value 12.7K -> 470K; device ds_passive:0402 -> ds_passive:1206
- R45: value 100K -> 470K; device ds_passive:0402 -> ds_passive:1206
- R6: value 330R 1W -> 7.5K; device ds_passive:1206 -> ds_passive:0402
- R7: value 330R 1W -> 10R; device ds_passive:1206 -> ds_passive:0402
- R8: value 330R 1W -> 20K; device ds_passive:1206 -> ds_passive:0402
- R9: value 0R -> 10R; device ds_passive:0805 -> ds_passive:0402
- moved R30 196.1 mm to (105.4, 114.1), flipped to the bottom, turned to 90 degrees
- moved SW3 195.9 mm to (148.5, 87.7), turned to 180 degrees
- moved GND-5 193.1 mm to (143.0, 96.2)
- moved 5VDC 192.4 mm to (153.1, 93.1), turned to 180 degrees
- moved L1 182.3 mm to (148.5, 103.3)
- moved C43 181.9 mm to (92.0, 113.0), turned to 180 degrees
- moved GND-3 181.4 mm to (143.2, 73.9), turned to 180 degrees
- moved R31 180.7 mm to (77.6, 114.0), flipped to the bottom, turned to 90 degrees
- moved R32 167.6 mm to (50.3, 113.9), flipped to the bottom, turned to 90 degrees
- moved C42 166.6 mm to (92.0, 115.2), turned to 180 degrees
- moved R35 165.9 mm to (22.2, 113.7), turned to 90 degrees
- moved C44 165.9 mm to (99.6, 97.8), turned to 180 degrees
- moved R34 164.8 mm to (16.6, 112.5), turned to 180 degrees
- moved R33 161.7 mm to (16.6, 114.7), turned to 180 degrees
- moved C36 161.5 mm to (64.2, 115.1), turned to 180 degrees
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Connections:
- removed net AC_LINE: F2.1, REL1.3, REL1.6, REL2.3, REL2.6, REL3.3, REL3.6, REL4.3, REL4.6, REL5.3, REL5.6, REL6.3, REL6.6, REL7.3, REL7.6, REL8.3, REL8.6
- removed net AC_LINE2: C14.2, CM1.1, RV1.2
- removed net DC_RAW: BR1.+, C15.1, C16.1, C17.1, R13.2, T1.6
- removed net EXP_RST: IC2.14
- removed net FB: C22.1, C23.1, IC4.7, OPT2.3
- new net +12V_MEA: J1.13, R94.1, R95.2
- new net +5V_MEA: C23.1, C5.1, IC10.1, IC11.1, IC12.1, IC14.1, IC16.1, IC5.3, IC6.1, IC7.1, IC8.1, R63.1, R63.2, R63.3, R63.4, R64.1, R64.2, R64.3, R64.4
- new net 5VFB: 5VFB.TP, C11.2, R11.2, R12.1, R8.2
- new net AC_L: AC/DC1.AC_L, AC_L.1, AC_L.2, C21.1, K1.3, K1.6, K2.3, K2.6, K3.3, K3.6, K4.3, K4.6, K5.3, K5.6, K6.3, K6.6, K7.3, K7.6, K8.3, K8.6, R60.1
- new net AC_N: AC/DC1.AC_N, AC_N.1, AC_N.2, R57.1, R58.1, R59.1
- new net C13_IN1: R25.2, R33.1, R35.2
- new net C13_IN2: R32.2, R49.1, R51.2
- new net C13_IN3: R31.2, R65.1, R67.2
- new net C13_IN4: R30.2, R81.1, R83.2
- new net C13_IN5: R26.2, R41.1, R43.2
- new net C13_IN6: R27.2, R73.1, R75.2
- new net C13_IN7: R28.2, R97.1, R99.2
- new net C13_IN8: R113.1, R115.2, R29.2
- new net MCP_REL_RST: IC4.14, J1.15
- new net MUX_A: IC4.25, IC9.11, R93.4
- new net MUX_B: IC4.26, IC9.10, R93.3
- new net MUX_C: IC4.27, IC9.9, R93.2
- new net MUX_EN: IC4.28, IC9.7, R93.1
- new net N$1: IC9.5, R91.1
- new net N$100: C56.1, IC16.4, R119.2, R120.1
- new net N$3: C21.2, R60.2, R61.1
- new net N$4: IC3.14, R21.1
- new net N$47: C30.1, IC8.2, R49.2
- new net N$48: C31.1, IC8.3, R50.2
- new net N$49: R52.2, R53.1
- new net N$50: R53.2, R54.1
- new net N$51: R54.2, R55.1
- new net N$52: C32.1, IC8.4, R55.2, R56.1
- new net N$53: OPT2.5, R64.6
- new net N$54: OPT2.7, R64.5
- new net N$59: C36.1, IC10.2, R65.2
- new net N$60: C37.1, IC10.3, R66.2
- new net N$61: R68.2, R69.1
- new net N$62: R69.2, R70.1
- new net N$63: R70.2, R71.1
- new net N$64: C38.1, IC10.4, R71.2, R72.1
- new net N$65: C39.1, IC11.2, R73.2
- new net N$66: C40.1, IC11.3, R74.2
- new net N$67: R76.2, R77.1
- new net N$68: R77.2, R78.1
- new net N$69: R78.2, R79.1
- new net N$70: C41.1, IC11.4, R79.2, R80.1
- new net N$71: C42.1, IC12.2, R81.2
- new net N$72: C43.1, IC12.3, R82.2
- new net N$73: R84.2, R85.1
- new net N$74: R85.2, R86.1
- new net N$75: R86.2, R87.1
- new net N$76: C44.1, IC12.4, R87.2, R88.1
- new net N$83: C48.1, IC14.2, R97.2
- new net N$84: C49.1, IC14.3, R98.2
- new net N$85: R100.2, R101.1
- new net N$86: R101.2, R102.1
- new net N$87: R102.2, R103.1
- new net N$88: C50.1, IC14.4, R103.2, R104.1
- new net N$95: C54.1, IC16.2, R113.2
- new net N$96: C55.1, IC16.3, R114.2
- new net N$97: R116.2, R117.1
- new net N$98: R117.2, R118.1
- new net N$99: R118.2, R119.1
- new net RX_CH1: IC6.8
- new net RX_CH2: IC8.8
- new net RX_CH3: IC10.8
- new net RX_CH4: IC12.8
- new net RX_CH5: IC7.8
- new net RX_CH6: IC11.8
- new net RX_CH7: IC14.8
- new net RX_CH8: IC16.8
- new net SW3: C9.2, IC2.3, L2.1, SW3.TP
- new net SW5: C8.2, IC1.3, L1.1, SW.TP
- new net TX_CH1: IC6.6, OPT1.2
- new net TX_CH2: IC8.6, OPT1.4
- new net TX_CH3: IC10.6, OPT1.6
- new net TX_CH4: IC12.6, OPT1.8
- new net TX_CH5: IC7.6, OPT2.2
- new net TX_CH6: IC11.6, OPT2.4
- new net TX_CH7: IC14.6, OPT2.6
- new net TX_CH8: IC16.6, OPT2.8
- new net TX_MUX1: IC9.4, OPT1.16, R89.1
- new net TX_MUX2: IC9.3, OPT1.14, R89.2
- new net TX_MUX3: IC9.2, OPT1.12, R89.3
- new net TX_MUX4: IC9.1, OPT1.10, R89.4
- new net TX_MUX5: IC9.15, OPT2.16, R90.1
- new net TX_MUX6: IC9.14, OPT2.14, R90.2
- new net TX_MUX7: IC9.13, OPT2.12, R90.3
- new net TX_MUX8: IC9.12, OPT2.10, R90.4
- new net UART0_RX: J1.10
- new net UART0_TX: J1.11, R91.2, R92.2
- net +12V: now also C1.1, C2.1, C3.1, C4.1, IC1.2, IC2.2, IC3.10, K1.8, K2.8, K3.8, K4.8, K5.8, K6.8, K7.8, K8.8, R1.1, R15.1, R16.1, R2.1, R94.2; no longer C36.1, C44.1, C45.1, C48.1, IC1.10, IC5.2, IC7.2, R10.1, R30.1, R31.1, R9.1, REL1.8, REL2.8, REL3.8, REL4.8, REL5.8, REL6.8, REL7.8, REL8.8
- net +3V3: now also 3VDC.TP, C12.1, C15.1, C18.1, C19.1, C20.1, C33.1, C34.1, IC4.5, IC9.16, J1.4, J1.5, J1.6, L2.2, R13.1, R89.5, R89.6, R89.7, R89.8, R90.5, R90.6, R90.7, R90.8, R93.5, R93.6, R93.7, R93.8; no longer 3V3DC.TP, C1.1, C2.1, C43.1, C47.1, C57.1, IC2.5, L3.2, R43.1
- net +5V: now also C11.1, C14.1, C17.1, J1.1, J1.2, J1.3, R11.1; no longer C46.1, C52.1, C53.1, R36.1
- net AGND: now also C23.2, C26.2, C27.2, C28.2, C29.2, C30.2, C31.2, C32.2, C36.2, C37.2, C38.2, C39.2, C40.2, C41.2, C42.2, C43.2, C44.2, C48.2, C49.2, C5.2, C50.2, C54.2, C55.2, C56.2, D10.A, D11.A, IC10.5, IC11.5, IC12.5, IC14.5, IC16.5, IC5.4, IC6.5, IC7.5, IC8.5, R104.2, R120.2, R40.2, R48.2, R56.2, R57.2, R58.2, R59.2, R72.2, R80.2, R88.2; no longer BR1.-, C15.2, C17.2, C26.1, D17.A, D20.A, IC4.1, IC4.2, IC4.3, IC4.4, IC4.8, OPT2.4, R22.2, R23.2, T1.3
- net GND: now also AC/DC1.-V, C10.2, C13.2, C14.2, C15.2, C16.2, C17.2, C3.2, C33.2, C34.2, C4.2, C6.2, C7.2, IC1.4, IC2.4, IC3.9, IC4.11, IC4.12, IC4.13, IC4.6, IC4.PAD, IC9.8, J1.12, J1.14, J1.16, J1.9, J1.Z1, J1.Z2, J1.Z3, J1.Z4, OPT1.11, OPT1.13, OPT1.15, OPT1.9, OPT2.11, OPT2.13, OPT2.15, OPT2.9, R12.2, R14.2, R4.2, R6.2, R95.1, Z1.A; no longer C26.2, C36.2, C40.2, C44.2, C45.2, C46.2, C47.2, C48.2, C49.2, C53.2, C57.2, IC1.9, IC2.11, IC2.12, IC2.13, IC2.6, IC2.PAD, IC3.3, IC5.4, IC7.4, R18.2, R32.2, R33.2, R37.2, R44.2, T1.10
- net I2C_SCL: now also IC4.8, J1.8; no longer IC2.8
- net I2C_SDA: now also IC4.9, J1.7; no longer IC2.9
- net N$10: now also IC3.15, R20.1; no longer IC1.14, R5.1
- net N$11: now also IC3.16, R19.1; no longer IC1.13, R6.1
- net N$12: now also C24.1, IC6.2, R33.2; no longer BR1.AC2, CM1.3
- net N$13: now also IC3.17, R18.1; no longer IC1.12, R7.1
- net N$14: now also IC1.5, R7.2; no longer IC7.5, R34.2
- net N$15: now also IC3.18, R17.1; no longer IC1.11, R8.1
- net N$16: now also IC1.8, R8.1; no longer IC7.8, R35.1
- net N$17: now also OPT1.5, R63.6; no longer C51.2, IC7.3, L1.1, SW5.TP
- net N$18: now also C8.1, R7.1; no longer C51.1, R34.1
- net N$19: now also IC1.6, R1.2; no longer IC7.6, R31.2
- net N$2: now also 12VDC.TP, AC/DC1.+V, C10.1, C13.1, C16.1, R15.2, R16.2, Z1.C; no longer C19.1, C20.1, L2.2, R10.2, R17.1, R9.2
- net N$20: now also D10.C, D9.A, R61.2; no longer C14.1, CM1.2, F2.2, RV1.1
- net N$21: now also C6.1, IC1.7, R3.1; no longer C49.1, IC7.7, R29.1
- net N$22: now also C25.1, IC6.3, R34.2; no longer C16.2, D15.C, R13.1
- net N$23: now also OPT1.7, R63.5; no longer D15.A, IC4.13, IC4.14, IC4.15, IC4.16, T1.4
- net N$24: now also IC9.6, R92.1; no longer D16.2, T1.8
- net N$25: now also C22.1, IC5.1, R62.2; no longer C18.1, D16.3, L2.1, R14.1
- net N$26: now also D11.C, D9.C, R62.1; no longer IC3.2, OPT2.1, R14.2, R15.1
- net N$27: now also R36.2, R37.1; no longer OPT2.2, R15.2, R16.1
- net N$28: now also R37.2, R38.1; no longer C21.1, R16.2
- net N$29: now also R38.2, R39.1; no longer C21.2, IC3.1, R17.2, R18.1
- net N$30: now also C26.1, IC6.4, R39.2, R40.1; no longer C24.1, C25.1, D19.C, IC4.5, R24.1
- net N$31: now also C27.1, IC7.2, R41.2; no longer D19.A, R19.2
- net N$32: now also C28.1, IC7.3, R42.2; no longer D18.A, R19.1, R20.1, T1.1
- net N$33: now also R44.2, R45.1; no longer D17.C, D18.C, R21.1
- net N$34: now also R45.2, R46.1; no longer IC4.6, R20.2, R21.2, R22.1
- net N$35: now also R46.2, R47.1; no longer C23.2, R23.1
- net N$36: now also C29.1, IC7.4, R47.2, R48.1; no longer D20.C, R24.2
- net N$37: now also OPT2.1, R64.8; no longer C52.2, R35.2, R36.2, R37.1, VFB5.TP
- net N$38: now also IC2.5, R9.2; no longer IC5.5, R41.2
- net N$39: now also IC2.8, R10.1; no longer IC5.8, R42.1
- net N$40: now also OPT2.3, R64.7; no longer C42.2, IC5.3, L3.1, SW3.TP
- net N$41: now also C9.1, R9.1; no longer C42.1, R41.1
- net N$42: now also 3VFB.TP, C12.2, R10.2, R13.2, R14.1; no longer C43.2, R42.2, R43.2, R44.1, VFB3.TP
- net N$43: now also IC2.6, R2.2; no longer IC5.6, R30.2
- net N$44: now also C7.1, IC2.7, R5.1; no longer C40.1, IC5.7, R45.1
- net N$45: now also IC1.1, R3.2, R4.1; no longer IC7.1, R29.2, R33.1
- net N$46: now also IC2.1, R5.2, R6.1; no longer IC5.1, R32.1, R45.2
- net N$5: now also OPT1.1, R63.8; no longer BR1.AC1, CM1.4
- net N$6: now also IC3.11, R24.1; no longer IC1.18, R1.1
- net N$7: now also IC3.12, R23.1; no longer IC1.17, R2.1
- net N$8: now also IC3.13, R22.1; no longer IC1.16, R3.1
- net N$9: now also OPT1.3, R63.7; no longer IC1.15, R4.1
- net OUT_1: now also K1.4, K1.5, R25.1, R34.1, R35.1, R36.1; no longer REL1.4, REL1.5
- net OUT_2: now also K2.4, K2.5, R32.1, R50.1, R51.1, R52.1; no longer REL2.4, REL2.5
- net OUT_3: now also K3.4, K3.5, R31.1, R66.1, R67.1, R68.1; no longer REL3.4, REL3.5
- net OUT_4: now also K4.4, K4.5, R30.1, R82.1, R83.1, R84.1; no longer REL4.4, REL4.5
- net OUT_5: now also K5.4, K5.5, R26.1, R42.1, R43.1, R44.1; no longer REL5.4, REL5.5
- net OUT_6: now also K6.4, K6.5, R27.1, R74.1, R75.1, R76.1; no longer REL6.4, REL6.5
- net OUT_7: now also K7.4, K7.5, R100.1, R28.1, R98.1, R99.1; no longer REL7.4, REL7.5
- net OUT_8: now also K8.4, K8.5, R114.1, R115.1, R116.1, R29.1; no longer REL8.4, REL8.5
- net RELAY_1: now also K1.1, R24.2; no longer R1.2, REL1.1
- net RELAY_2: now also K2.1, R23.2; no longer R2.2, REL2.1
- net RELAY_3: now also K3.1, R22.2; no longer R3.2, REL3.1
- net RELAY_4: now also K4.1, R21.2; no longer R4.2, REL4.1
- net RELAY_5: now also K5.1, R20.2; no longer R5.2, REL5.1
- net RELAY_6: now also K6.1, R19.2; no longer R6.2, REL6.1
- net RELAY_7: now also K7.1, R18.2; no longer R7.2, REL7.1
- net RELAY_8: now also K8.1, R17.2; no longer R8.2, REL8.1
- net REL_0: now also IC3.8, IC4.17; no longer IC1.1, IC2.17
- net REL_1: now also IC3.7, IC4.18; no longer IC1.2, IC2.18
- net REL_2: now also IC3.6, IC4.19; no longer IC1.3, IC2.19
- net REL_3: now also IC3.5, IC4.20; no longer IC1.4, IC2.20
- net REL_4: now also IC3.4, IC4.21; no longer IC1.5, IC2.21
- net REL_5: now also IC3.3, IC4.22; no longer IC1.6, IC2.22
- net REL_6: now also IC3.2, IC4.23; no longer IC1.7, IC2.23
- net REL_7: now also IC3.1, IC4.24; no longer IC1.8, IC2.24
Routing:
- net AC_L: track 0.00 -> 630.6 mm, vias 0 -> 20
- net +12V: track 45.5 -> 489.6 mm, vias 0 -> 7
- net +5V_MEA: track 0.00 -> 430.6 mm, vias 0 -> 17
- net AGND: track 155.8 -> 530.5 mm, vias 1 -> 22
- net N$25: track 221.5 -> 21.2 mm, vias 22 -> 0
- net +3V3: track 0.00 -> 169.6 mm, vias 0 -> 6
- net GND: track 193.0 -> 348.6 mm, vias 27 -> 32
- net +5V: track 0.00 -> 145.1 mm, vias 0 -> 4
- net TX_CH1: track 0.00 -> 134.5 mm, vias 0 -> 2
- net TX_CH2: track 0.00 -> 106.6 mm, vias 0 -> 2
- net N$6: track 0.00 -> 93.2 mm
- net TX_CH5: track 0.00 -> 90.0 mm
- net N$10: track 0.00 -> 84.9 mm
- net N$11: track 0.00 -> 81.9 mm
- net N$2: track 126.7 -> 47.6 mm, vias 3 -> 0
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- added copper zone on layer 1, net AC_L
- added copper zone on layer 16, net AC_L
- added copper zone on layer 16, net AGND
- added copper zone on layer 1, net N$2
- removed copper zone on layer 1, net AC_LINE
- removed copper zone on layer 16, net AC_LINE
- removed copper zone on layer 1, net OUT_1
- removed copper zone on layer 16, net OUT_1
- removed copper zone on layer 1, net OUT_2
- removed copper zone on layer 16, net OUT_2
- removed copper zone on layer 1, net OUT_3
- removed copper zone on layer 16, net OUT_3
- removed copper zone on layer 1, net OUT_4
- removed copper zone on layer 16, net OUT_4
- removed copper zone on layer 1, net OUT_5
- removed copper zone on layer 16, net OUT_5
- removed copper zone on layer 1, net OUT_6
- removed copper zone on layer 16, net OUT_6
- removed copper zone on layer 1, net OUT_7
- removed copper zone on layer 16, net OUT_7
- removed copper zone on layer 1, net OUT_8
- removed copper zone on layer 16, net OUT_8
Other:
- board size 147 x 95 mm -> 156.1 x 120 mm
- board text removed: "L"
- board text removed: "L N"

Commit message: finished with design update for 2.0
Parts:
- J1: value 687320124422 -> FPC20-H; device Wurth_Connectors_WR-FPC:687320124422 -> ds_con:FPC20
- moved J1 0.20 mm to (145.9, 21.2)
Routing:
- net GND: track 348.6 -> 356.0 mm

Commit message: add datasheets for Rev2.0
Parts:
- AC/DC1: value (none) -> IRM_10_12
Changed lines of the file:
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@@
 <drawing>
 <settings>
-<setting alwaysvectorfont="yes"/>
+<setting alwaysvectorfont="no"/>
 <setting verticaltext="up"/>
 </settings>
@@
 <attribute name="VALUE" x="153.345" y="-50.075" size="1.27" layer="27" rot="R90"/>
 </element>
-<element name="AC/DC1" library="ds_trafo" package="IRM_10_12" package3d_urn="urn:adsk.eagle:package:47075710/2" value="" x="54.5" y="59.3" smashed="yes">
+<element name="AC/DC1" library="ds_trafo" package="IRM_10_12" package3d_urn="urn:adsk.eagle:package:47075710/2" value="IRM_10_12" x="54.5" y="59.3" smashed="yes">
 <attribute name="NAME" x="32" y="46.02" size="1.27" layer="25"/>
 <attribute name="VALUE" x="31.4" y="46.62" size="1.27" layer="27" align="top-left"/>

Commit message: update repo to Rev2.0
Changed lines of the file:
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@@
 <wire x1="-1" y1="3.41420625" x2="2.41420625" y2="0" width="0" layer="20" curve="90"/>
 <circle x="3" y="4" radius="3" width="1" layer="29"/>
-<circle x="141" y="4" radius="3" width="1" layer="29"/>
 <circle x="3" y="115.9" radius="2.828425" width="1" layer="29"/>
 <text x="153.98" y="8.39" size="1.4224" layer="25" font="vector" ratio="13" rot="R90">github.com/DvidMakesThings/HW_10-In-Rack_PDU
@@
 </element>
 <element name="C10" library="ds_passive" package="100UF-16V" package3d_urn="urn:adsk.eagle:package:46684204/2" value="100uF" x="84" y="69" smashed="yes">
-<attribute name="NAME" x="84.9144" y="73.3688" size="1.27" layer="25" align="center"/>
+<attribute name="NAME" x="89.5144" y="66.8688" size="1.27" layer="25" align="center"/>
 <attribute name="VALUE" x="84.4572" y="64.6566" size="1.27" layer="27" align="center"/>
 </element>
 <element name="C13" library="ds_passive" package="100UF-16V" package3d_urn="urn:adsk.eagle:package:46684204/2" value="100uF" x="84" y="61.3" smashed="yes">
-<attribute name="NAME" x="84.9144" y="65.6688" size="1.27" layer="25" align="center"/>
+<attribute name="NAME" x="89.4144" y="59.0688" size="1.27" layer="25" align="center"/>
 <attribute name="VALUE" x="84.4572" y="56.9566" size="1.27" layer="27" align="center"/>
 </element>
 <element name="C16" library="ds_passive" package="100UF-16V" package3d_urn="urn:adsk.eagle:package:46684204/2" value="100uF" x="84" y="53.7" smashed="yes">
-<attribute name="NAME" x="84.9144" y="58.0688" size="1.27" layer="25" align="center"/>
+<attribute name="NAME" x="89.3856" y="55.9312" size="1.27" layer="25" rot="R180" align="center"/>
 <attribute name="VALUE" x="84.4572" y="49.3566" size="1.27" layer="27" align="center"/>
 </element>
