File: src/HardwareDesign/_Display-Board/Rev3.0/Display-Board_Rack-PDU_3.0.brd (EAGLE design)
At the start: 124 x 42 mm, 57 parts, among them IC2 MCP23017-E/ML, T1 BSS138

Commit message: Creating HW release version ENERGIS Rev1.0.0 from CB1.0.21, DB1.0.30, RB1.0.21
Parts:
- removed C15: 10uF, ds_passive:C0402
- removed C16: 100nF, ds_passive:C0402
- removed KEY3: TP, ds_passive:TP
- added C3: 10uF, ds_passive:C0402
- added C4: 100nF, ds_passive:C0402
- moved C1 12.7 mm to (53.7, 23.1), turned to 90 degrees
- moved C2 2.48 mm to (55.0, 32.3)
- moved U$1 0.57 mm to (127.8, 24.1)
- renumbered 3V3 to TP1, 5V to TP2, BL to TP3, BUT+1 to S1, BUT-1 to S2, BUT_SET1 to S3, C17 to C7, C18 to C8, C19 to C9, C21 to C5, C22 to C6, CS to TP5, DC to TP4, DISPBOARD to CON2, ETH to LED2, FAULT to LED3, GND to TP16, I2C_SCL to TP15, I2C_SDA to TP14, IC2 to IC1, KEY0 to TP9, KEY1 to TP10, KEY2 to TP11, LCD_RES to TP13, MCP_RES to TP12, MISO to TP7, MOSI to TP8, OUT-1 to LED4, OUT-2 to LED5, OUT-3 to LED6, OUT-4 to LED7, OUT-5 to LED8, OUT-6 to LED9, OUT-7 to LED10, OUT-8 to LED11, PWR to LED1, R21 to R5, R22 to R6, R23 to R12, R26 to R8, R27 to R9, R28 to R10, R29 to R11, R30 to R7, SCK to TP6, TFT to CON1
Connections:
- net +3V3: now also C3.1, C4.1; no longer C15.1, C16.1
- net GND: now also C3.2, C4.2; no longer C15.2, C16.2
- net KEY_3: no longer KEY3.TP
Routing:
- net +3V3: track 0.00 -> 162.3 mm, vias 0 -> 12
- net GND: track 0.00 -> 155.7 mm, vias 0 -> 59
- net N$68: track 0.00 -> 63.7 mm, vias 0 -> 2
- net KEY_1: track 0.00 -> 56.7 mm, vias 0 -> 2
- net N$67: track 0.00 -> 53.1 mm, vias 0 -> 2
- net N$58: track 0.00 -> 52.0 mm
- net KEY_0: track 0.00 -> 51.3 mm, vias 0 -> 1
- net LCD_BL: track 0.00 -> 48.9 mm, vias 0 -> 2
- net N$66: track 0.00 -> 48.1 mm, vias 0 -> 2
- net LCD_RES: track 0.00 -> 48.1 mm, vias 0 -> 2
- net N$59: track 0.00 -> 47.0 mm, vias 0 -> 2
- net LCD_DC: track 0.00 -> 44.3 mm, vias 0 -> 2
- net LCD_CS: track 0.00 -> 43.9 mm, vias 0 -> 2
- net MCP_LCD_RST: track 0.00 -> 43.3 mm, vias 0 -> 2
- net I2C0_SCL: track 0.00 -> 43.2 mm, vias 0 -> 2
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Other:
- board text removed: "Display Board REV3.0"
