File: src/HardwareDesign/ENERGIS/Rev1.0.0/ENERGIS_Rack-PDU_1.0.0.brd (EAGLE design)
At the start: 210 x 100 mm, 361 parts, among them IC1 MP2315GJ-Z, IC10 HLW8032, IC11 HLW8032, IC12 HLW8032, IC13 MP150GJ, IC14 HLW8032, IC15 RP2040, IC16 HLW8032, IC17 MCP6001R, IC18 W25Q128JVPIQ, IC19 CAT24C512HU5IGT3, IC2 MP2315S, IC20 W5500, IC21 MIC5504-3.3YM5-TR, IC22 FT232RNQ, IC3 ULN2803A, IC4 MCP23017-E/ML, IC5 MP150GJ, IC6 HLW8032, IC7 HLW8032, IC8 HLW8032, IC9 SN74HC151PWR, J1 0R-JUMPA, J10 0R, J7 JP, J8 0R, J9 0R, K1 G2RL-1A-E_DC12, K2 G2RL-1A-E_DC12, K3 G2RL-1A-E_DC12, K4 G2RL-1A-E_DC12, K5 G2RL-1A-E_DC12, K6 G2RL-1A-E_DC12, K7 G2RL-1A-E_DC12, K8 G2RL-1A-E_DC12, SW3 TP, X1 12MHz, X2 25MHz

Commit message: update schematics
Parts:
- removed D16: CHIP-FLAT-B_0603-0.35MM, LED:LEDC1608X35N_FLAT-B
- removed D17: CHIP-FLAT-G_0603-0.35MM, LED:LEDC1608X35N_FLAT-G
- removed DISPBOARD: FPC20-H, ds_con:FPC20
- removed U$7: (no value), holes:3,2
- added CON1: AFC11-S20ICC-00, ds_con:FPC20
- added PWR, RX: CHIP-FLAT-G_0603-0.35MM, LED:LEDC1608X35N_FLAT-G
- added R122, R123: DNI, ds_passive:R0201
- added R151: 1K, ds_passive:0402
- added TX: CHIP-FLAT-B_0603-0.35MM, LED:LEDC1608X35N_FLAT-B
- moved USBC 3.25 mm to (175.2, -0.60)
- moved R124 3.08 mm to (177.0, 6.08)
- moved R125 2.36 mm to (173.7, 6.54), turned to 90 degrees
- moved R121 2.00 mm to (178.1, 6.98)
- moved R131 2.00 mm to (169.2, 4.75)
- moved C78 1.98 mm to (168.0, 4.77)
Connections:
- new net N$112: PWR.C, R151.2
- net +3V3: now also CON1.1, CON1.2; no longer DISPBOARD.1, DISPBOARD.2
- net +3V3_MCU: now also PWR.A
- net +5V: now also CON1.3, CON1.4; no longer DISPBOARD.3, DISPBOARD.4
- net DP_N: now also R123.1
- net DP_P: now also R122.1
- net GND: now also CON1.5, CON1.8, CON1.Z0, CON1.Z1, CON1.Z2, CON1.Z3, CON1.Z4, CON1.Z5, R151.1; no longer DISPBOARD.5, DISPBOARD.8, DISPBOARD.Z0, DISPBOARD.Z1, DISPBOARD.Z2, DISPBOARD.Z3, DISPBOARD.Z4, DISPBOARD.Z5
- net I2C0_SCL: now also CON1.7; no longer DISPBOARD.7
- net I2C0_SDA: now also CON1.6; no longer DISPBOARD.6
- net KEY_0: now also CON1.12; no longer DISPBOARD.12
- net KEY_1: now also CON1.11; no longer DISPBOARD.11
- net KEY_2: now also CON1.10; no longer DISPBOARD.10
- net KEY_3: now also CON1.9; no longer DISPBOARD.9
- net LCD_BL: now also CON1.13; no longer DISPBOARD.13
- net LCD_CS: now also CON1.19; no longer DISPBOARD.19
- net LCD_DC: now also CON1.18; no longer DISPBOARD.18
- net LCD_MISO: now also CON1.15; no longer DISPBOARD.15
- net LCD_MOSI: now also CON1.16; no longer DISPBOARD.16
- net LCD_RES: now also CON1.14; no longer DISPBOARD.14
- net LCD_SCLK: now also CON1.17; no longer DISPBOARD.17
- net MCP_DSP_RST: now also CON1.20; no longer DISPBOARD.20
- net N$110: now also TX.C; no longer D16.C
- net N$111: now also RX.C; no longer D17.C
- net USBRP_DP_N: now also R123.2
- net USBRP_DP_P: now also R122.2
- net VBUS: now also RX.A, TX.A; no longer D16.A, D17.A
Routing:
- net GND: track 262.2 -> 286.0 mm, vias 146 -> 144
- net +3V3_MCU: track 170.5 -> 189.6 mm, vias 16 -> 17
- net DP_P: track 28.8 -> 40.5 mm, vias 2 -> 4
- net DP_N: track 28.8 -> 39.2 mm, vias 2 -> 4
- net VBUS: track 165.6 -> 175.9 mm
- net N$111: track 52.9 -> 59.5 mm
- net RUN: track 106.7 -> 111.3 mm, vias 2 -> 4
- net USB_SHIELD: track 24.2 -> 21.6 mm
- net USBRP_DP_P: track 16.4 -> 18.7 mm
- net N$110: track 41.8 -> 43.8 mm
- net N$112: track 0.00 -> 1.53 mm
- net !W5500_CS: track 32.4 -> 34.0 mm
- net W5500_SCK: track 30.1 -> 31.5 mm
- net USBRP_DP_N: track 16.4 -> 17.8 mm
- net W5500_MISO: track 34.0 -> 35.1 mm
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Other:
- board size 210 x 100 mm -> 210 x 102 mm

Commit message: update main board
Parts:
- added R152: DNI, ds_passive:0402
Connections:
- net +3V3_MCU: now also R152.1
- net USB_SEL: now also R152.2
Routing:
- net +3V3_MCU: track 189.6 -> 192.8 mm, vias 17 -> 18
- net USB_SEL: track 20.8 -> 22.2 mm
Changed lines of the file:
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@@
 <drawing>
 <settings>
-<setting alwaysvectorfont="yes"/>
+<setting alwaysvectorfont="no"/>
 <setting verticaltext="up"/>
 </settings>
-<grid distance="0.5" unitdist="mm" unit="mm" style="lines" multiple="1" display="yes" altdistance="5" altunitdist="mil" altunit="mm"/>
+<grid distance="0.01" unitdist="mm" unit="mm" style="lines" multiple="1" display="yes" altdistance="5" altunitdist="mil" altunit="mm"/>
 <layers>
 <layer number="1" name="SIG_HS" color="4" fill="1" visible="yes" active="yes"/>
@@
 </element>
 <element name="C65" library="ds_passive" library_urn="urn:adsk.eagle:library:46685041" package="0805" package3d_urn="urn:adsk.eagle:package:46683742/2" value="10uF" x="171.2886" y="10.0278" smashed="yes" rot="R180">
-<attribute name="NAME" x="169.1552" y="10.4672" size="0.8128" layer="25" rot="R180"/>
+<attribute name="NAME" x="172.1552" y="8.9672" size="0.8128" layer="25" rot="R180"/>
 </element>
 <element name="C66" library="ds_passive" library_urn="urn:adsk.eagle:library:46685041" package="0402" package3d_urn="urn:adsk.eagle:package:46683744/2" value="100nF" x="171.7822" y="11.6528" smashed="yes" rot="R180">
@@
 </element>
 <element name="R127" library="ds_passive" package="R0201" package3d_urn="urn:adsk.eagle:package:47403529/2" value="10K" x="169.7322" y="11.7758" smashed="yes" rot="R270">
-<attribute name="NAME" x="169.1412" y="12.2894" size="0.8128" layer="25" rot="R180"/>
+<attribute name="NAME" x="168.4906" y="12.4112" size="0.8128" layer="25" rot="R270"/>
 </element>
 <element name="IC19" library="ds_ic_memory" package="SON50P300X200X50-9T130X140N" package3d_urn="urn:adsk.eagle:package:45817778/1" value="CAT24C512HU5IGT3" x="157.4152" y="22.9804" smashed="yes" rot="R270">
@@
 <attribute name="VALUE" x="143.653" y="32.6651" size="1.27" layer="27" align="top-center"/>
 </element>
+<element name="R152" library="ds_passive" package="0402" package3d_urn="urn:adsk.eagle:package:46683744/2" value="DNI" x="167.75" y="11" smashed="yes" rot="R90">
+<attribute name="NAME" x="166.245" y="12.115" size="0.8128" layer="25" rot="R270"/>
+<attribute name="VALUE" x="169.655" y="10.365" size="1.27" layer="27" rot="R90"/>
+</element>
 </elements>
 <signals>
@@
 <contactref element="IC15" pad="38"/>
 <wire x1="159.917084375" y1="12.564415625" x2="162.1115" y2="10.37" width="0.2032" layer="1"/>
-<wire x1="167.2908" y1="12.0508" x2="169.68" y2="12.0508" width="0.2032" layer="1"/>
+<wire x1="166.2508" y1="11.0108" x2="168.38" y2="11.0108" width="0.2032" layer="1"/>
+<wire x1="169.42" y1="12.0508" x2="169.68" y2="12.0508" width="0.2032" layer="1"/>
 <wire x1="169.68" y1="12.0508" x2="169.7322" y2="12.0508" width="0.2032" layer="1"/>
 <wire x1="162.1115" y1="10.37" x2="165.61" y2="10.37" width="0.2032" layer="1"/>
-<wire x1="165.61" y1="10.37" x2="167.2908" y2="12.0508" width="0.2032" layer="1"/>
+<wire x1="165.61" y1="10.37" x2="166.2508" y2="11.0108" width="0.2032" layer="1"/>
 <wire x1="169.7422" y1="12.8052" x2="169.7422" y2="12.113" width="0.2032" layer="1"/>
 <wire x1="169.7422" y1="12.113" x2="169.68" y2="12.0508" width="0.2032" layer="1"/>
+<wire x1="169.42" y1="12.0508" x2="168.38" y2="11.0108" width="0.2032" layer="1"/>
 </signal>
 <signal name="I2C0_SDA">
@@
 <wire x1="150.83" y1="24.12" x2="150.58" y2="24.37" width="0.2" layer="15"/>
 <wire x1="152.22" y1="36.03" x2="152.22" y2="27.08" width="0.2" layer="15"/>
+<contactref element="R152" pad="1"/>
+<wire x1="166.95" y1="9.47" x2="166.95" y2="10.18" width="0.2" layer="1"/>
+<via x="166.95" y="9.47" extent="1-16" drill="0.2"/>
+<wire x1="166.95" y1="9.47" x2="166.95" y2="10.08" width="0.2" layer="15"/>
+<wire x1="166.95" y1="10.08" x2="166.6" y2="10.43" width="0.2" layer="15"/>
+<wire x1="166.6" y1="10.43" x2="166.6" y2="10.9" width="0.2" layer="15"/>
+<wire x1="167.12" y1="10.35" x2="167.75" y2="10.35" width="0.2" layer="1"/>
+<wire x1="166.95" y1="10.18" x2="167.12" y2="10.35" width="0.2" layer="1"/>
 </signal>
 <signal name="VCCIO">
@@
 <wire x1="172.21425" y1="13.93425" x2="172.5236875" y2="14.2436875" width="0.2" layer="1"/>
 <wire x1="172.5236875" y1="14.2436875" x2="172.5236875" y2="16.3663125" width="0.2" layer="1"/>
-<wire x1="166.58" y1="11.87655625" x2="166.58" y2="14.06" width="0.2" layer="1"/>
+<wire x1="166.58" y1="11.87655625" x2="166.58" y2="11.9" width="0.2" layer="1"/>
+<wire x1="166.58" y1="11.9" x2="166.58" y2="14.06" width="0.2" layer="1"/>
 <wire x1="171.61" y1="16.885" x2="171.61" y2="17.11" width="0.2" layer="1"/>
 <wire x1="171.61" y1="17.11" x2="171.695" y2="17.195" width="0.2" layer="1"/>
+<contactref element="R152" pad="2"/>
+<wire x1="167.74" y1="11.9" x2="166.58" y2="11.9" width="0.2" layer="1"/>
+<wire x1="167.75" y1="11.65" x2="167.74" y2="11.66" width="0.2" layer="1"/>
+<wire x1="167.74" y1="11.66" x2="167.74" y2="11.9" width="0.2" layer="1"/>
 </signal>
 <signal name="N$112">

Commit message: update BOM
Parts:
- IC23: value (none) -> PI3USB102JXUCEX
Changed lines of the file:
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@@
 <attribute name="VALUE" x="193.165" y="22.985" size="1.27" layer="27" rot="R270"/>
 </element>
-<element name="IC23" library="ds_ic_peripherals" package="QFN40P120X140X35-10N" package3d_urn="urn:adsk.eagle:package:48463072/1" value="" x="170.62" y="18.48" smashed="yes" rot="R180">
+<element name="IC23" library="ds_ic_peripherals" package="QFN40P120X140X35-10N" package3d_urn="urn:adsk.eagle:package:48463072/1" value="PI3USB102JXUCEX" x="170.62" y="18.48" smashed="yes" rot="R180">
 <attribute name="NAME" x="173.1351" y="18.41" size="0.8128" layer="25" rot="R90" align="bottom-center"/>
 <attribute name="VALUE" x="170.62" y="20.0709" size="1.27" layer="27" rot="R180" align="top-center"/>
