File: src/HardwareDesign/ENERGIS/Rev1.0.0/ENERGIS_Rack-PDU_1.0.0.brd (EAGLE design)
At the start: 210 x 108 mm, 393 parts, among them IC1 MP2315GJ-Z, IC10 HLW8032, IC11 HLW8032, IC12 HLW8032, IC13 MP150GJ, IC14 HLW8032, IC15 RP2040, IC16 HLW8032, IC17 MCP6001R, IC18 W25Q128JVPIQ, IC19 CAT24C512HU5IGT3, IC2 MP2315S, IC20 W5500, IC21 MIC5504-3.3YM5-TR, IC22 MCP6001R, IC3 ULN2803A, IC4 MCP23017-E/ML, IC5 MP150GJ, IC6 HLW8032, IC7 HLW8032, IC8 HLW8032, IC9 SN74HC151PWR, J10 0R, J2 JP, J7 JP, J8 0R, J9 0R, K1 G2RL-1A-E_DC12, K2 G2RL-1A-E_DC12, K3 G2RL-1A-E_DC12, K4 G2RL-1A-E_DC12, K5 G2RL-1A-E_DC12, K6 G2RL-1A-E_DC12, K7 G2RL-1A-E_DC12, K8 G2RL-1A-E_DC12, P12ON LEDC1608X35N_FLAT-G, P3ON LEDC1608X35N_FLAT-G, P5ON LEDC1608X35N_FLAT-G, SW3 TP, X1 12MHz, X2 25MHz

Commit message: update documentation
Parts:
- added U$5, U$7: (no value), ds_silkscreen:DMT

Commit message: starting with documentation
Parts:
- added C102, C104: 1uF, ds_passive:0201
- added R152: 10R, ds_passive:R0201
- added R161: DNI, ds_passive:0402
- added R162: 10K, ds_passive:0402
- R1: value 10K -> DNI
- moved R1 1.76 mm to (102.1, 6.30)
- moved C62 1.14 mm to (138.8, 21.0)
- moved C63 0.59 mm to (138.3, 19.7), turned to 90 degrees
Connections:
- new net 5V_EN: IC1.6, R1.1, R161.2, R162.1
- new net MCP_VIN: C102.1, C63.1, IC17.2, R152.2
- net +12V: now also R162.2
- net +3V3_MCU: now also C104.1, R152.1; no longer C63.1, IC17.2
- net BUCK_EN: no longer IC1.6
- net GND: now also C102.2, C104.2, R161.1; no longer R1.1
Routing:
- net BUCK_EN: track 135.8 -> 122.3 mm, vias 7 -> 5
- net 5V_EN: track 0.00 -> 13.3 mm, vias 0 -> 2
- net +3V3_MCU: track 114.0 -> 118.3 mm, vias 18 -> 19
- net MCP_VIN: track 0.00 -> 2.78 mm
- net +12V: track 368.3 -> 370.4 mm
- net GND: track 268.2 -> 269.3 mm, vias 172 -> 170

Commit message: update readme
Parts:
- C1, C2: device ds_passive:C1206 -> ds_capacitors:1206
- C10, C13, C16: value 100uF -> 100uF 25V; device ds_passive:100UF-16V -> ds_capacitors:6.3X7.7(DXL)
- C100, C101, C103, C61, C62, C63, C64, C67, C68, C69, C70, C71, C72, C73, C74, C75, C76, C77, C84, C88, C89, C90, C91, C92, C93, C94, C95, C96, C98: value 100nF -> 100nF 25V; device ds_passive:0201 -> ds_capacitors:0201
- C102: value 1uF -> 1uF 16V; device ds_passive:0201 -> ds_capacitors:0201
- C104: value 1uF -> 1uF 25V; device ds_passive:0201 -> ds_capacitors:0402
- C106, C107, C108, C109, C110, C111, C112, C113: value 1nF -> 1nF 25V; device ds_passive:0201 -> ds_capacitors:0201
- C11, C12: value 33pF -> 33pF 50V; device ds_passive:0402 -> ds_capacitors:0402
- C14, C15, C17, C18: value 22uF - 10V -> 22uF 25V; device ds_passive:C1206 -> ds_capacitors:1206
- C19, C20, C33, C34, C79: value 100nF -> 100nF 25V; device ds_passive:C0402 -> ds_capacitors:0402
- C21, C46: value 2.2uF 10V -> 2.2uF 50V; device ds_passive:C0603 -> ds_capacitors:0603
- C22, C52: value 220nF 16V -> 220nF 50V; device ds_passive:C0805 -> ds_capacitors:0805
- C23, C53: value 100uF 16V -> 100uF 50V; device Wurth_Capacitors_WCAP-PSHP:WCAP-PSHP_6.3X5.8(DXL) -> ds_capacitors:6.3X7.7(DXL)
- C24, C25, C26, C27, C28, C29, C30, C31, C32, C36, C37, C38, C39, C40, C41, C42, C43, C44, C48, C49, C50, C54, C55, C56: value 33nF -> 33nF 50V; device ds_passive:C0805 -> ds_capacitors:0805
- C3, C4, C6, C66, C7, C8, C9: value 100nF -> 100nF 25V; device ds_passive:0402 -> ds_capacitors:0402
- C35, C47: device Wurth_Capacitors_WCAP-HSAH:WCAP-HSAH_D6.3H7.7P2.2 -> ds_capacitors:6.3X7.7(DXL)
- C45, C57: device ds_passive:C0805 -> ds_capacitors:0805
- C5, C51: device ds_passive:C0603 -> ds_capacitors:0603
- C58, C59: value 15pF -> 15pF 50V; device ds_passive:0201 -> ds_capacitors:0201
- C60: value 1uF -> 1uF 25V; device ds_passive:C0402 -> ds_capacitors:0402
- C65, C97, C99: value 10uF -> 10uF 50V; device ds_passive:0805 -> ds_capacitors:0805
- C78: value 4.7nF -> 4.7nF 50V; device ds_passive:0402 -> ds_capacitors:0402
- C80: value 22nF -> 22nF 50V; device ds_passive:C0402 -> ds_capacitors:0402
- C81, C82: value 6.8nF -> 6.8nF 50V; device ds_passive:0201 -> ds_capacitors:0201
- C85: value 4.7uF -> 4.7uF 25V; device ds_passive:C0402 -> ds_capacitors:0402
- C86, C87: value 18pF -> 18pF 50V; device ds_passive:0201 -> ds_capacitors:0201
- DAT: value LEDC1608X35N_FLAT-B -> Blue; device LED:LEDC1608X35N_FLAT-B -> ds_LED:LED-0603
- IC15: device ds_ic_mcu:QFN40P700X700X100-57T510 -> ds_ic_mcu:QFN56
- IC21: value MIC5504-3.3YM5-TR -> MIC5504-3.3YM5
- J10, J8, J9: value 0R -> 0R 1%; device ds_passive:0805 -> ds_resistor:0805
- L3, L5: value FNR6028S102MT 1mH -> 1mH; device Wurth_Automotive_WE-HEPA:WE-HEPA_6030 -> ds_inductor:L-6.6X6.6
- P12ON, P3ON, P5ON, PWR: value LEDC1608X35N_FLAT-G -> Green; device LED:LEDC1608X35N_FLAT-G -> ds_LED:LED-0603
- R100, R101, R102, R103, R116, R117, R118, R119, R36, R37, R38, R39, R44, R45, R46, R47, R52, R53, R54, R55, R68, R69, R70, R71, R76, R77, R78, R79, R84, R85, R86, R87: value 470K -> 470K 1%; device ds_passive:0805 -> ds_resistor:0805
- R104, R113, R114, R120, R33, R34, R40, R41, R42, R48, R49, R50, R56, R65, R66, R72, R73, R74, R80, R81, R82, R88, R97, R98: device ds_passive:0805 -> ds_resistor:0805
- R105, R107, R60, R61: value 4.99K -> 4.99K 1%; device ds_passive:0603 -> ds_resistor:0603
- R106, R62: value 39R 2W -> 39R 1% 2W; device ds_passive:2512 -> ds_resistor:2512
- R108, R96: value 10K -> 10K 1%; device ds_passive:0805 -> ds_resistor:0805
- R109, R129, R145: value 4.7K -> 4.7K 1%; device ds_passive:R0201 -> ds_resistor:0201
- R11, R13: value 40.2K -> 40.2K 1%; device ds_passive:0402 -> ds_resistor:0402
- R110: value 4.99M -> 1M 1%; device ds_passive:1206 -> ds_resistor:1206
- R112, R122, R123, R151: value 1K -> 1K 1%; device ds_passive:0402 -> ds_resistor:0402
- R115, R25, R26, R27, R28, R29, R30, R31, R32, R35, R43, R51, R67, R75, R83, R99: device ds_passive:2512 -> ds_resistor:2512
- R12, R6: value 7.5K -> 7.5K 1%; device ds_passive:0402 -> ds_resistor:0402
- R121: device ds_passive:R0201 -> ds_resistor:0201
- R124, R125: value 5.1K -> 5.1K 1%; device ds_passive:R0201 -> ds_resistor:0201
- R126, R127: value 10K -> 10K 1%; device ds_passive:R0201 -> ds_resistor:0201
- R131: value 1M -> 1M 1%; device ds_passive:0402 -> ds_resistor:0402
- R132, R147, R162, R2, R95: value 10K -> 10K 1%; device ds_passive:0402 -> ds_resistor:0402
- R133, R134, R135, R136: value 3.3R -> 3.3R 1%; device ds_passive:R0201 -> ds_resistor:0201
- R137, R138, R139, R140: value 49.9R -> 49.9R 1%; device ds_passive:R0201 -> ds_resistor:0201
- R14: value 12.7K -> 12.7K 1%; device ds_passive:0402 -> ds_resistor:0402
- R141, R142, R146: value 470R -> 470R 1%; device ds_passive:0402 -> ds_resistor:0402
- R144: value 1M -> 1M 1%; device ds_passive:R0201 -> ds_resistor:0201
- R148: value 2.4 K -> 2.4K 1%; device ds_passive:0402 -> ds_resistor:0402
- R15, R160: value 27R -> 27R 1%; device ds_passive:R0201 -> ds_resistor:0201
- R150: value 8.2K -> 8.2K 1%; device ds_passive:0402 -> ds_resistor:0402
- R152: value 10R -> 10R 1%; device ds_passive:R0201 -> ds_resistor:0201
- R153, R154, R155, R156, R157, R158, R159, R16, R59: value 1K -> 1K 1%; device ds_passive:R0201 -> ds_resistor:0201
- R17, R18, R19, R20, R21, R22, R23, R24: value 330R 1W -> 330R 1% 1W; device ds_passive:2512 -> ds_resistor:2512
- R3, R5: value 100K -> 100K 1%; device ds_passive:0402 -> ds_resistor:0402
- R4: value 9.09K -> 9.09K 1%; device ds_passive:0402 -> ds_resistor:0402
- R57, R91: value 0R -> 0R 1%; device ds_passive:0402 -> ds_resistor:0402
- R7, R9: value 10R -> 10R 1%; device ds_passive:0402 -> ds_resistor:0402
- R8: value 20K -> 20K 1%; device ds_passive:0402 -> ds_resistor:0402
- R94: value 100K -> 10K 1%; device ds_passive:0402 -> ds_resistor:0402
- moved C104 1.61 mm to (135.1, 20.9)
- moved C23 1.10 mm to (17.3, 23.5)
- moved D9 1.00 mm to (32.7, 27.3)
- moved D13 0.71 mm to (55.1, 26.9)
- moved L5 0.30 mm to (48.5, 27.3)
- moved C10 0.28 mm to (120.7, 40.7), turned to 180 degrees
- moved C16 0.16 mm to (120.6, 25.6), turned to 180 degrees
- moved C13 0.16 mm to (120.6, 33.2), turned to 180 degrees
- moved L3 0.10 mm to (25.9, 27.6)
Connections:
- net AGND: now also C35.2, C47.2; no longer C35.1, C47.1
- net GND: now also IC15.PAD; no longer IC15.57
- net N$20: now also C35.1; no longer C35.2
- net N$77: now also C47.1; no longer C47.2
Routing:
- net N$78: track 0.00 -> 14.1 mm
- net N$25: track 0.00 -> 7.83 mm
- net +5V_MEA1: track 2.82 -> 7.84 mm
- net +5V_MEA2: track 2.00 -> 6.87 mm
- net +3V3_MCU: track 118.3 -> 119.8 mm
- net GND: track 269.3 -> 270.0 mm
- net AGND: track 353.4 -> 352.6 mm

Commit message: update design to final state
Parts:
- removed USBC: USB-TYPE-C-018, Wurth_Connectors_WR-USB:629722000214
- removed Z1: SMAJ15A, 52101-101-REV-A_v16:SUPRESSOR_SMAJ
- added D16: SMAJ15A, ds_diode:SMA/DO-214AC
- added PROC: Green, ds_LED:LED-0603
- added R163: 1K 1%, ds_resistor:0402
- added USB1: USB-TYPE-C-018, ds_con:USB-C
- AC/DC2: value (none) -> IRM-10-15
- BOOT, RESET: value RS032G05A3SM -> B3U-1000P; device BeagleBone_Blue_R3:TACTILE-SWITCH-1101NE -> ds_passive:B3U-1000P
- D1, D10, D12, D13, D9: device diode:SMA -> ds_diode:SMA/DO-214AC
- D11, D14: value US1J -> US1J-E3/61T; device diode:SMA -> ds_diode:SMA/DO-214AC
- D15: device Diodes:SMA -> ds_diode:SMA/DO-214AC
- D2, D3, D4, D5, D6, D7, D8: value MBRA340T3 -> MBRA340T3G; device diode:SMA -> ds_diode:SMA/DO-214AC
- DSP: value AFC11-S20ICC-00 -> AFC11-S20ICC-00
- ESD1: value SP0503BAHTG-ES -> SP0503BAHTG
- ETH1: value SI-60118-F -> J1B1211CCD; device ds_con:RJ45-CAT5 -> ds_con:J1B1211CCD
- IC1: value MP2315GJ-Z -> MP2315GJ-Z
- IC17, IC22: value MCP6001R -> MCP6001RT-I/OT
- IC19: value CAT24C512HU5IGT3 -> CAT24C256HU4IGT3
- IC2: value MP2315S -> MP2315GJ-Z
- IC3: value ULN2803A -> ULN2803AFWG
- IC4: value MCP23017-E/ML -> MCP23017T-E/ML
- K1, K2, K3, K4, K5, K6, K7, K8: value G2RL-1A-E_DC12 -> G2RL-1A-E DC12
- L4: device ds_passive:0603 -> ds_inductor:0603
- OPT1, OPT2: value ACPL-247 -> ACPL-247-500E
- R130, R149: value 4D03WGJ0332T5E -> 3.3K 1%; device Resistor Array:742C083103JP -> ds_resistor:_0603X4-1206
- R63, R64: value 4x1K 1206 -> 1K 1%; device Resistor Array:742C083103JP -> ds_resistor:_0603X4-1206
- R89, R90: value 4x1K 1206 -> 10K 1%; device Resistor Array:742C083103JP -> ds_resistor:_0603X4-1206
- R94: value 10K 1% -> 100K 1%
- REF1: value LM4040BXX -> LM4040B30FTA
- X1, X2: device Wurth_Quartz Crystals & Oscillators_WE-XTAL:WE-XTAL_CFPX-180 -> ds_passive:WE-XTAL_CFPX-180
- moved R142 12.1 mm to (185.7, 19.5)
- moved R141 11.9 mm to (197.5, 19.6)
- moved IOVDD 1.14 mm to (164.3, 3.26)
- moved D15 0.76 mm to (122.8, 8.47)
- moved ETH1 0.27 mm to (191.5, 6.92)
- moved X1 0.06 mm to (148.5, 5.38)
Connections:
- net N$20 renamed LREC1
- net N$25 renamed SRC1
- net N$26 renamed VNI1
- net N$55 renamed FB1
- net N$57 renamed FBIN1
- net N$77 renamed LREC2
- net N$78 renamed SRC2
- net N$79 renamed VNI2
- net N$80 renamed FB2
- net N$81 renamed FBIN2
- removed net USB_SEL: IC15.39
- new net N$17: IC15.40, R163.2
- new net N$19: PROC.A, R163.1
- net +3V3: now also ETH1.10, ETH1.12, R149.A1, R149.B1, R149.C1, R149.D1, R89.A2, R89.B2, R89.C2, R89.D2, R90.A2, R90.B2, R90.C2, R90.D2; no longer ETH1.11, ETH1.9, R149.1, R149.2, R149.3, R149.4, R89.5, R89.6, R89.7, R89.8, R90.5, R90.6, R90.7, R90.8
- net +3V3_MCU: now also R130.A2, R130.B2, R130.C2, R130.D2; no longer R130.5, R130.6, R130.7, R130.8
- net +5V_MEA: now also R63.A1, R63.B1, R63.C1, R63.D1, R64.A1, R64.B1, R64.C1, R64.D1; no longer R63.1, R63.2, R63.3, R63.4, R64.1, R64.2, R64.3, R64.4
- net 12VRAW: now also D16.C; no longer Z1.C
- net CC1: now also USB1.A5; no longer USBC.A5
- net CC2: now also USB1.B5; no longer USBC.B5
- net GND: now also D16.A, PROC.C, USB1.GND, USB1.GND2; no longer USBC.A1, USBC.A12, USBC.B1, USBC.B12, Z1.A
- net I2C0_SCL: now also R130.A1; no longer R130.1
- net I2C0_SDA: now also R130.B1; no longer R130.2
- net I2C1_SCL: now also R130.C1; no longer R130.3
- net I2C1_SDA: now also R130.D1; no longer R130.4
- net LCD_CS: now also R149.C2; no longer R149.6
- net LCD_MISO: now also R149.B2; no longer R149.7
- net LCD_RES: now also R149.A2; no longer R149.8
- net N$82: now also ETH1.11; no longer ETH1.10
- net N$91: now also ETH1.9; no longer ETH1.12
- net SH: now also ETH1.13, ETH1.14, USB1.SHLD1, USB1.SHLD2, USB1.SHLD3, USB1.SHLD4; no longer ETH1.S1, ETH1.S2, USBC.S1, USBC.S2, USBC.S3, USBC.S4
- net TX1_PU: now also R63.D2; no longer R63.5
- net TX2_PU: now also R63.C2; no longer R63.6
- net TX3_PU: now also R63.B2; no longer R63.7
- net TX4_PU: now also R63.A2; no longer R63.8
- net TX5_PU: now also R64.A2; no longer R64.8
- net TX6_PU: now also R64.B2; no longer R64.7
- net TX7_PU: now also R64.C2; no longer R64.6
- net TX8_PU: now also R64.D2; no longer R64.5
- net TX_MUX1: now also R89.D1; no longer R89.4
- net TX_MUX2: now also R89.C1; no longer R89.3
- net TX_MUX3: now also R89.B1; no longer R89.2
- net TX_MUX4: now also R89.A1; no longer R89.1
- net TX_MUX5: now also R90.A1; no longer R90.1
- net TX_MUX6: now also R90.B1; no longer R90.2
- net TX_MUX7: now also R90.C1; no longer R90.3
- net TX_MUX8: now also R90.D1; no longer R90.4
- net USB2_DP_N: now also USB1.A7, USB1.B7; no longer USBC.A7, USBC.B7
- net USB2_DP_P: now also USB1.A6, USB1.B6; no longer USBC.A6, USBC.B6
- net VBUS: now also USB1.VBUS1, USB1.VBUS2; no longer USBC.A4, USBC.A9, USBC.B4, USBC.B9
Routing:
- net !ACT: track 35.9 -> 23.7 mm
- net N$19: track 0.00 -> 11.3 mm
- net +3V3: track 75.7 -> 85.8 mm
- net !LINK: track 25.9 -> 34.2 mm
- net N$17: track 0.00 -> 7.71 mm
- net GND: track 270.0 -> 274.9 mm, vias 170 -> 151
- net VBUS: track 110.6 -> 106.7 mm, vias 10 -> 9
- net N$91: track 19.6 -> 17.2 mm
- net 12VRAW: track 48.7 -> 50.6 mm
- net RUN: track 82.1 -> 83.6 mm
- net USB_BOOT: track 2.35 -> 3.80 mm
- net AGND: track 352.6 -> 351.4 mm
- net +3V3_MCU: track 119.8 -> 120.9 mm
- net USB2_DP_N: track 39.4 -> 38.7 mm
- net BUCK_EN: track 122.3 -> 121.6 mm
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Other:
- outline, holes or cut-outs redrawn

Commit message: update software, bugfix
Parts:
- R93: value 4x10K 1206 -> 10K 1%; device Resistor Array:742C083103JP -> ds_resistor:_0603X4-1206
- X1: value 12MHz -> ABM8-272-T3 12MHz
- moved C19 0.07 mm to (152.1, 26.4)
- moved C20 0.05 mm to (152.9, 27.1)
Connections:
- net GND: now also R93.A2, R93.B2, R93.C2, R93.D2; no longer R93.5, R93.6, R93.7, R93.8
- net MUX_A: now also R93.D1; no longer R93.4
- net MUX_B: now also R93.C1; no longer R93.3
- net MUX_C: now also R93.B1; no longer R93.2
- net MUX_EN: now also R93.A1; no longer R93.1
Routing:
- net N$91: track 17.2 -> 19.5 mm
- net N$82: track 18.0 -> 18.8 mm
- net GND: vias 151 -> 155

Commit message: Baseline commit. Device is functioning as expected, software is working
Parts:
- added CS0, CS1, MISO0, MISO1, MOSI0, MOSI1, REL0, REL1, REL2, REL3, REL4, REL5, REL6, REL7, RX0, RX1, SCL0, SCL1, SCLK0, SCLK1, SDA0, SDA1: TP, ds_passive:TP
- added FAN: (no value), con-amp-quick:02P
- added R164: 10K 1%, ds_resistor:0402
- added R165: NC, ds_passive:R0201
- added T1: (no value), ds_active:SOT23
- moved 12VDC 0.89 mm to (128.4, 19.4)
- moved GND 0.58 mm to (128.3, 17.1)
Connections:
- new net FAN_CTRL: IC15.39, R164.1, R165.1, T1.1
- new net N$23: FAN.1, T1.3
- net !W5500_CS: now also CS1.TP
- net +12V: now also FAN.2
- net +3V3_MCU: now also R165.2
- net GND: now also R164.2, T1.2
- net I2C0_SCL: now also SCL0.TP
- net I2C0_SDA: now also SDA0.TP
- net I2C1_SCL: now also SCL1.TP
- net I2C1_SDA: now also SDA1.TP
- net LCD_CS: now also CS0.TP
- net LCD_MISO: now also MISO0.TP
- net LCD_MOSI: now also MOSI0.TP
- net LCD_SCLK: now also SCLK0.TP
- net REL_0: now also REL0.TP
- net REL_1: now also REL1.TP
- net REL_2: now also REL2.TP
- net REL_3: now also REL3.TP
- net REL_4: now also REL4.TP
- net REL_5: now also REL5.TP
- net REL_6: now also REL6.TP
- net REL_7: now also REL7.TP
- net UART0_RX: now also RX0.TP
- net UART0_TX: now also RX1.TP
- net W5500_MISO: now also MISO1.TP
- net W5500_MOSI: now also MOSI1.TP
- net W5500_SCK: now also SCLK1.TP
Routing:
- net FAN_CTRL: track 0.00 -> 50.1 mm, vias 0 -> 2
- net !W5500_CS: track 33.8 -> 61.5 mm, vias 2 -> 3
- net +12V: track 370.5 -> 395.1 mm
- net REL_7: track 7.27 -> 27.2 mm, vias 0 -> 1
- net W5500_SCK: track 33.9 -> 53.8 mm, vias 2 -> 3
- net W5500_MOSI: track 40.0 -> 57.4 mm, vias 2 -> 3
- net REL_6: track 6.47 -> 23.7 mm, vias 0 -> 1
- net LCD_MOSI: track 28.2 -> 44.4 mm
- net I2C0_SCL: track 43.0 -> 58.6 mm, vias 2 -> 5
- net W5500_MISO: track 39.7 -> 55.0 mm, vias 2 -> 3
- net REL_5: track 5.68 -> 19.6 mm, vias 0 -> 1
- net I2C1_SDA: track 21.4 -> 35.1 mm, vias 2 -> 4
- net REL_4: track 5.76 -> 16.6 mm, vias 0 -> 1
- net I2C1_SCL: track 22.1 -> 32.6 mm, vias 3 -> 5
- net I2C0_SDA: track 48.4 -> 58.4 mm, vias 2 -> 3
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