File: src/HardwareDesign/ENERGIS/Rev1.0.0/ENERGIS_Rack-PDU_1.0.0.sch (EAGLE design)
At the start: 353 parts, among them IC1 MP2315GJ-Z, IC10 HLW8032, IC11 HLW8032, IC12 HLW8032, IC13 MP150GJ, IC14 HLW8032, IC15 RP2040, IC16 HLW8032, IC17 MCP6001R, IC18 W25Q128JVPIQ, IC19 CAT24C512HU5IGT3, IC2 MP2315S, IC20 W5500, IC21 MIC5504-3.3YM5-TR, IC22 FT232RNQ, IC3 ULN2803A, IC4 MCP23017-E/ML, IC5 MP150GJ, IC6 HLW8032, IC7 HLW8032, IC8 HLW8032, IC9 SN74HC151PWR, J1 0R-JUMPA, J10 0R, J7 JP, J8 0R, J9 0R, K1 G2RL-1A-E_DC12, K2 G2RL-1A-E_DC12, K3 G2RL-1A-E_DC12, K4 G2RL-1A-E_DC12, K5 G2RL-1A-E_DC12, K6 G2RL-1A-E_DC12, K7 G2RL-1A-E_DC12, K8 G2RL-1A-E_DC12, SW3 TP, X1 12MHz, X2 25MHz

Commit message: update schematics
Parts:
- removed DISPBOARD: FPC20-H, ds_con:FPC20-H
- added CON1: AFC11-S20ICC-00, ds_con:AFC11-S20ICC-00
- added PWR: CHIP-FLAT-G_0603-0.35MM, LED:CHIP-FLAT-G_0603-0.35MM
- added R122, R123: DNI, ds_passive:R0201
- added R151: 1K, ds_passive:R0402
- renumbered D16 to TX, D17 to RX
Connections:
- new net N$112: PWR.C, R151.2
- net +3V3: now also CON1.1, CON1.2; no longer DISPBOARD.1, DISPBOARD.2
- net +3V3_MCU: now also PWR.A
- net +5V: now also CON1.3, CON1.4; no longer DISPBOARD.3, DISPBOARD.4
- net DP_N: now also R123.1
- net DP_P: now also R122.1
- net GND: now also CON1.5, CON1.8, CON1.Z1, CON1.Z2, CON1.Z3, CON1.Z4, R151.1; no longer DISPBOARD.5, DISPBOARD.8, DISPBOARD.Z1, DISPBOARD.Z2, DISPBOARD.Z3, DISPBOARD.Z4
- net I2C0_SCL: now also CON1.7; no longer DISPBOARD.7
- net I2C0_SDA: now also CON1.6; no longer DISPBOARD.6
- net KEY_0: now also CON1.12; no longer DISPBOARD.12
- net KEY_1: now also CON1.11; no longer DISPBOARD.11
- net KEY_2: now also CON1.10; no longer DISPBOARD.10
- net KEY_3: now also CON1.9; no longer DISPBOARD.9
- net LCD_BL: now also CON1.13; no longer DISPBOARD.13
- net LCD_CS: now also CON1.19; no longer DISPBOARD.19
- net LCD_DC: now also CON1.18; no longer DISPBOARD.18
- net LCD_MISO: now also CON1.15; no longer DISPBOARD.15
- net LCD_MOSI: now also CON1.16; no longer DISPBOARD.16
- net LCD_RES: now also CON1.14; no longer DISPBOARD.14
- net LCD_SCLK: now also CON1.17; no longer DISPBOARD.17
- net MCP_DSP_RST: now also CON1.20; no longer DISPBOARD.20
- net USBRP_DP_N: now also R123.2
- net USBRP_DP_P: now also R122.2

Commit message: update main board
Parts:
- added R152: DNI, ds_passive:R0402
Connections:
- net +3V3_MCU: now also R152.1
- net USB_SEL: now also R152.2
Changed lines of the file:
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@@
 <part name="PWR" library="LED" library_urn="urn:adsk.eagle:library:22900745" deviceset="CHIP-FLAT-G" device="_0603-0.35MM" package3d_urn="urn:adsk.eagle:package:24294786/2"/>
 <part name="GND84" library="ds_passive" library_urn="urn:adsk.eagle:library:46685041" deviceset="GND" device=""/>
+<part name="R152" library="ds_passive" deviceset="R" device="0402" package3d_urn="urn:adsk.eagle:package:46683744/2" value="DNI"/>
+<part name="+3V3_MCU13" library="ds_passive" deviceset="+3V3_MCU" device=""/>
 </parts>
 <sheets>
@@
 <attribute name="VALUE" x="203.835" y="80.2386" size="1.778" layer="96"/>
 </instance>
+<instance part="R152" gate="G$1" x="165.1" y="43.18" smashed="yes" rot="R180">
+<attribute name="NAME" x="160.655" y="44.2214" size="1.778" layer="95" rot="R180"/>
+<attribute name="VALUE" x="161.925" y="41.6814" size="1.778" layer="96" rot="R180"/>
+</instance>
+<instance part="+3V3_MCU13" gate="G$1" x="160.02" y="35.56" smashed="yes" rot="R90">
+<attribute name="VALUE" x="154.94" y="33.02" size="1.778" layer="96" align="top-center"/>
+</instance>
 </instances>
 <busses>
@@
 <wire x1="193.04" y1="50.8" x2="180.34" y2="50.8" width="0.1524" layer="91"/>
 <pinref part="R150" gate="G$1" pin="2"/>
-<wire x1="180.34" y1="50.8" x2="162.56" y2="50.8" width="0.1524" layer="91"/>
+<wire x1="180.34" y1="50.8" x2="165.1" y2="50.8" width="0.1524" layer="91"/>
+<wire x1="165.1" y1="50.8" x2="162.56" y2="50.8" width="0.1524" layer="91"/>
 <wire x1="180.34" y1="48.26" x2="180.34" y2="50.8" width="0.1524" layer="91"/>
 <junction x="180.34" y="50.8"/>
 <label x="162.56" y="50.8" size="1.27" layer="95" rot="R180" xref="yes"/>
+<pinref part="R152" gate="G$1" pin="2"/>
+<wire x1="165.1" y1="48.26" x2="165.1" y2="50.8" width="0.1524" layer="91"/>
+<junction x="165.1" y="50.8"/>
 </segment>
 </net>
@@
 <wire x1="254" y1="66.04" x2="254" y2="58.42" width="0.1524" layer="91"/>
 </segment>
-</net>
+<segment>
+<pinref part="R152" gate="G$1" pin="1"/>
+<wire x1="165.1" y1="38.1" x2="165.1" y2="35.56" width="0.1524" layer="91"/>
+<wire x1="165.1" y1="35.56" x2="160.02" y2="35.56" width="0.1524" layer="91"/>
+<pinref part="+3V3_MCU13" gate="G$1" pin="+3V3_MCU"/>
+</segment>
+</net>

Commit message: update BOM
Parts:
- IC23: value (none) -> PI3USB102JXUCEX
Changed lines of the file:
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@@
 <grid distance="0.1" unitdist="inch" unit="inch" style="lines" multiple="1" display="yes" altdistance="0.01" altunitdist="inch" altunit="inch"/>
 <layers>
-<layer number="1" name="Top" color="4" fill="1" visible="yes" active="no"/>
-<layer number="2" name="Route2" color="16" fill="1" visible="yes" active="no"/>
-<layer number="3" name="Route3" color="17" fill="1" visible="yes" active="no"/>
-<layer number="4" name="Route4" color="18" fill="1" visible="yes" active="no"/>
-<layer number="5" name="Route5" color="19" fill="1" visible="yes" active="no"/>
-<layer number="6" name="Route6" color="25" fill="1" visible="yes" active="no"/>
-<layer number="7" name="Route7" color="26" fill="1" visible="yes" active="no"/>
-<layer number="8" name="Route8" color="27" fill="1" visible="yes" active="no"/>
-<layer number="9" name="Route9" color="28" fill="1" visible="yes" active="no"/>
-<layer number="10" name="Route10" color="29" fill="1" visible="yes" active="no"/>
-<layer number="11" name="Route11" color="30" fill="1" visible="yes" active="no"/>
-<layer number="12" name="Route12" color="20" fill="1" visible="yes" active="no"/>
-<layer number="13" name="Route13" color="21" fill="1" visible="yes" active="no"/>
-<layer number="14" name="Route14" color="22" fill="1" visible="yes" active="no"/>
-<layer number="15" name="Route15" color="63" fill="1" visible="yes" active="no"/>
-<layer number="16" name="Bottom" color="1" fill="1" visible="yes" active="no"/>
-<layer number="17" name="Pads" color="2" fill="1" visible="yes" active="no"/>
-<layer number="18" name="Vias" color="2" fill="1" visible="yes" active="no"/>
-<layer number="19" name="Unrouted" color="6" fill="1" visible="yes" active="no"/>
-<layer number="20" name="Dimension" color="24" fill="1" visible="yes" active="no"/>
-<layer number="21" name="tPlace" color="7" fill="1" visible="yes" active="no"/>
-<layer number="22" name="bPlace" color="7" fill="1" visible="yes" active="no"/>
-<layer number="23" name="tOrigins" color="15" fill="1" visible="yes" active="no"/>
-<layer number="24" name="bOrigins" color="15" fill="1" visible="yes" active="no"/>
-<layer number="25" name="tNames" color="7" fill="1" visible="yes" active="no"/>
-<layer number="26" name="bNames" color="7" fill="1" visible="yes" active="no"/>
-<layer number="27" name="tValues" color="7" fill="1" visible="yes" active="no"/>
-<layer number="28" name="bValues" color="7" fill="1" visible="yes" active="no"/>
+<layer number="1" name="Top" color="4" fill="1" visible="no" active="no"/>
+<layer number="2" name="Route2" color="16" fill="1" visible="no" active="no"/>
+<layer number="3" name="Route3" color="17" fill="1" visible="no" active="no"/>
+<layer number="4" name="Route4" color="18" fill="1" visible="no" active="no"/>
+<layer number="5" name="Route5" color="19" fill="1" visible="no" active="no"/>
+<layer number="6" name="Route6" color="25" fill="1" visible="no" active="no"/>
+<layer number="7" name="Route7" color="26" fill="1" visible="no" active="no"/>
+<layer number="8" name="Route8" color="27" fill="1" visible="no" active="no"/>
+<layer number="9" name="Route9" color="28" fill="1" visible="no" active="no"/>
+<layer number="10" name="Route10" color="29" fill="1" visible="no" active="no"/>
+<layer number="11" name="Route11" color="30" fill="1" visible="no" active="no"/>
+<layer number="12" name="Route12" color="20" fill="1" visible="no" active="no"/>
+<layer number="13" name="Route13" color="21" fill="1" visible="no" active="no"/>
+<layer number="14" name="Route14" color="22" fill="1" visible="no" active="no"/>
+<layer number="15" name="Route15" color="63" fill="1" visible="no" active="no"/>
+<layer number="16" name="Bottom" color="1" fill="1" visible="no" active="no"/>
+<layer number="17" name="Pads" color="2" fill="1" visible="no" active="no"/>
+<layer number="18" name="Vias" color="2" fill="1" visible="no" active="no"/>
+<layer number="19" name="Unrouted" color="6" fill="1" visible="no" active="no"/>
+<layer number="20" name="Dimension" color="24" fill="1" visible="no" active="no"/>
+<layer number="21" name="tPlace" color="7" fill="1" visible="no" active="no"/>
+<layer number="22" name="bPlace" color="7" fill="1" visible="no" active="no"/>
+<layer number="23" name="tOrigins" color="15" fill="1" visible="no" active="no"/>
+<layer number="24" name="bOrigins" color="15" fill="1" visible="no" active="no"/>
+<layer number="25" name="tNames" color="7" fill="1" visible="no" active="no"/>
+<layer number="26" name="bNames" color="7" fill="1" visible="no" active="no"/>
+<layer number="27" name="tValues" color="7" fill="1" visible="no" active="no"/>
+<layer number="28" name="bValues" color="7" fill="1" visible="no" active="no"/>
 <layer number="29" name="tStop" color="7" fill="3" visible="no" active="no"/>
 <layer number="30" name="bStop" color="7" fill="6" visible="no" active="no"/>
@@
 <layer number="35" name="tGlue" color="7" fill="4" visible="no" active="no"/>
 <layer number="36" name="bGlue" color="7" fill="5" visible="no" active="no"/>
-<layer number="37" name="tTest" color="7" fill="1" visible="yes" active="no"/>
-<layer number="38" name="bTest" color="7" fill="1" visible="yes" active="no"/>
+<layer number="37" name="tTest" color="7" fill="1" visible="no" active="no"/>
+<layer number="38" name="bTest" color="7" fill="1" visible="no" active="no"/>
 <layer number="39" name="tKeepout" color="4" fill="11" visible="no" active="no"/>
 <layer number="40" name="bKeepout" color="1" fill="11" visible="no" active="no"/>
@@
 <layer number="44" name="Drills" color="7" fill="1" visible="no" active="no"/>
 <layer number="45" name="Holes" color="7" fill="1" visible="no" active="no"/>
-<layer number="46" name="Milling" color="3" fill="1" visible="yes" active="no"/>
-<layer number="47" name="Measures" color="7" fill="1" visible="yes" active="no"/>
-<layer number="48" name="Document" color="7" fill="1" visible="yes" active="no"/>
-<layer number="49" name="Reference" color="7" fill="1" visible="yes" active="no"/>
-<layer number="50" name="dxf" color="7" fill="1" visible="yes" active="no"/>
-<layer number="51" name="tDocu" color="7" fill="1" visible="yes" active="no"/>
-<layer number="52" name="bDocu" color="7" fill="1" visible="yes" active="no"/>
-<layer number="53" name="tGND_GNDA" color="7" fill="9" visible="yes" active="no"/>
-<layer number="54" name="bGND_GNDA" color="1" fill="9" visible="yes" active="no"/>
-<layer number="56" name="wert" color="7" fill="1" visible="yes" active="no"/>
-<layer number="57" name="tCAD" color="7" fill="1" visible="yes" active="no"/>
-<layer number="58" name="bCAD" color="7" fill="1" visible="yes" active="no"/>
-<layer number="59" name="tCarbon" color="7" fill="1" visible="yes" active="no"/>
-<layer number="60" name="bCarbon" color="7" fill="1" visible="yes" active="no"/>
-<layer number="61" name="stand" color="7" fill="1" visible="yes" active="no"/>
+<layer number="46" name="Milling" color="3" fill="1" visible="no" active="no"/>
+<layer number="47" name="Measures" color="7" fill="1" visible="no" active="no"/>
+<layer number="48" name="Document" color="7" fill="1" visible="no" active="no"/>
+<layer number="49" name="Reference" color="7" fill="1" visible="no" active="no"/>
+<layer number="50" name="dxf" color="7" fill="1" visible="no" active="no"/>
+<layer number="51" name="tDocu" color="7" fill="1" visible="no" active="no"/>
+<layer number="52" name="bDocu" color="7" fill="1" visible="no" active="no"/>
+<layer number="53" name="tGND_GNDA" color="7" fill="9" visible="no" active="no"/>
+<layer number="54" name="bGND_GNDA" color="1" fill="9" visible="no" active="no"/>
+<layer number="56" name="wert" color="7" fill="1" visible="no" active="no"/>
+<layer number="57" name="tCAD" color="7" fill="1" visible="no" active="no"/>
+<layer number="58" name="bCAD" color="7" fill="1" visible="no" active="no"/>
+<layer number="59" name="tCarbon" color="7" fill="1" visible="no" active="no"/>
+<layer number="60" name="bCarbon" color="7" fill="1" visible="no" active="no"/>
+<layer number="61" name="stand" color="7" fill="1" visible="no" active="no"/>
 <layer number="88" name="SimResults" color="9" fill="1" visible="yes" active="yes"/>
 <layer number="89" name="SimProbes" color="9" fill="1" visible="yes" active="yes"/>
@@
 <part name="GND79" library="ds_passive" deviceset="GND" device=""/>
 <part name="GND80" library="ds_passive" deviceset="GND" device=""/>
-<part name="IC23" library="ds_ic_peripherals" deviceset="PI3USB102J" device="XUCEX" package3d_urn="urn:adsk.eagle:package:48463072/1"/>
+<part name="IC23" library="ds_ic_peripherals" deviceset="PI3USB102J" device="XUCEX" package3d_urn="urn:adsk.eagle:package:48463072/1" value="PI3USB102JXUCEX"/>
 <part name="R150" library="ds_passive" deviceset="R" device="0201" package3d_urn="urn:adsk.eagle:package:47403529/2" value="10K"/>
 <part name="GND81" library="ds_passive" deviceset="GND" device=""/>
