File: src/HardwareDesign/ENERGIS/Rev1.0.0/ENERGIS_Rack-PDU_1.0.0.sch (EAGLE design)
At the start: 386 parts, among them IC1 MP2315GJ-Z, IC10 HLW8032, IC11 HLW8032, IC12 HLW8032, IC13 MP150GJ, IC14 HLW8032, IC15 RP2040, IC16 HLW8032, IC17 MCP6001R, IC18 W25Q128JVPIQ, IC19 CAT24C512HU5IGT3, IC2 MP2315S, IC20 W5500, IC21 MIC5504-3.3YM5-TR, IC22 MCP6001R, IC3 ULN2803A, IC4 MCP23017-E/ML, IC5 MP150GJ, IC6 HLW8032, IC7 HLW8032, IC8 HLW8032, IC9 SN74HC151PWR, J10 0R, J2 JP, J7 JP, J8 0R, J9 0R, K1 G2RL-1A-E_DC12, K2 G2RL-1A-E_DC12, K3 G2RL-1A-E_DC12, K4 G2RL-1A-E_DC12, K5 G2RL-1A-E_DC12, K6 G2RL-1A-E_DC12, K7 G2RL-1A-E_DC12, K8 G2RL-1A-E_DC12, P12ON LEDC1608X35N_FLAT-G, P3ON LEDC1608X35N_FLAT-G, P5ON LEDC1608X35N_FLAT-G, SW3 TP, X1 12MHz, X2 25MHz

Commit message: starting with documentation
Parts:
- added C102, C104: 1uF, ds_passive:C-0201
- added R152: 10R, ds_passive:R0201
- added R161: DNI, ds_passive:R0402
- added R162: 10K, ds_passive:R0402
- R1: value 10K -> DNI
Connections:
- new net 5V_EN: IC1.EN, R1.1, R161.2, R162.1
- new net MCP_VIN: C102.1, C63.1, IC17.V+, R152.2
- net +12V: now also R162.2
- net +3V3_MCU: now also C104.1, R152.1; no longer C63.1, IC17.V+
- net BUCK_EN: no longer IC1.EN
- net GND: now also C102.2, C104.2, R161.1; no longer R1.1
Other:
- moved on the sheet: R1

Commit message: update readme
Parts:
- C1, C2: device ds_passive:C-1206 -> ds_capacitors:22UF-25V-1206
- C10, C13, C16: value 100uF -> 100uF 25V; device ds_passive:CPOL -> ds_capacitors:100UF-25V6.3X7.7(DXL)
- C100, C101, C103, C61, C62, C63, C64, C67, C68, C69, C70, C71, C72, C73, C74, C75, C76, C77, C84, C88, C89, C90, C91, C92, C93, C94, C95, C96, C98: value 100nF -> 100nF 25V; device ds_passive:C-0201 -> ds_capacitors:100NF-25V-0201
- C102: value 1uF -> 1uF 16V; device ds_passive:C-0201 -> ds_capacitors:1UF-16V0201
- C104: value 1uF -> 1uF 25V; device ds_passive:C-0201 -> ds_capacitors:1UF-25V0402
- C106, C107, C108, C109, C110, C111, C112, C113: value 1nF -> 1nF 25V; device ds_passive:C-0201 -> ds_capacitors:1NF-25V-0201
- C11, C12: value 33pF -> 33pF 50V; device ds_passive:C0402 -> ds_capacitors:33PF-50V0402
- C14, C15, C17, C18: value 22uF - 10V -> 22uF 25V; device ds_passive:C-1206 -> ds_capacitors:22UF-25V-1206
- C19, C20, C33, C34, C79: value 100nF -> 100nF 25V; device ds_passive:C-0402 -> ds_capacitors:100NF-25V-0402
- C21, C46: value 2.2uF 10V -> 2.2uF 50V; device ds_passive:C-0603 -> ds_capacitors:2.2UF-50V0603
- C22, C52: value 220nF 16V -> 220nF 50V; device ds_passive:C-0805 -> ds_capacitors:220NF-50V0805
- C23, C53: value 100uF 16V -> 100uF 50V; device Wurth_Capacitors_WCAP-PSHP:WCAP-PSHP_6.3X5.8_875115644009 -> ds_capacitors:100UF-50V6.3X7.7(DXL)
- C24, C25, C26, C27, C28, C29, C30, C31, C32, C36, C37, C38, C39, C40, C41, C42, C43, C44, C48, C49, C50, C54, C55, C56: value 33nF -> 33nF 50V; device ds_passive:C-0805 -> ds_capacitors:33NF-50V0805
- C3, C4, C6, C66, C7, C8, C9: value 100nF -> 100nF 25V; device ds_passive:C0402 -> ds_capacitors:100NF-25V-0402
- C35, C47: device Wurth_Capacitors_WCAP-HSAH:WCAP-HSAH_D6.3H7.7P2.2_875585745003 -> ds_capacitors:2.2UF-400V6.3X7.7(DXL)
- C45, C57: device ds_passive:C-0805 -> ds_capacitors:1UF-50V0805
- C5, C51: device ds_passive:C-0603 -> ds_capacitors:1NF-50V-0603
- C58, C59: value 15pF -> 15pF 50V; device ds_passive:C-0201 -> ds_capacitors:15PF-50V0201
- C60: value 1uF -> 1uF 25V; device ds_passive:C-0402 -> ds_capacitors:1UF-25V0402
- C65, C97, C99: value 10uF -> 10uF 50V; device ds_passive:C0805 -> ds_capacitors:10UF-50V-0805
- C78: value 4.7nF -> 4.7nF 50V; device ds_passive:C0402 -> ds_capacitors:4.7NF-50V0402
- C80: value 22nF -> 22nF 50V; device ds_passive:C-0402 -> ds_capacitors:22NF-50V0402
- C81, C82: value 6.8nF -> 6.8nF 50V; device ds_passive:C-0201 -> ds_capacitors:6.8NF-50V0201
- C85: value 4.7uF -> 4.7uF 25V; device ds_passive:C-0402 -> ds_capacitors:4.7UF-25V0402
- C86, C87: value 18pF -> 18pF 50V; device ds_passive:C-0201 -> ds_capacitors:18PF-50V-0201
- DAT: value LEDC1608X35N_FLAT-B -> Blue; device LED:CHIP-FLAT-B_0603-0.35MM -> ds_LED:LED-BLUELED-0603
- IC21: value MIC5504-3.3YM5-TR -> MIC5504-3.3YM5
- J10, J8, J9: value 0R -> 0R 1%; device ds_passive:R0805 -> ds_resistor:0R0805
- L3, L5: value FNR6028S102MT 1mH -> 1mH; device Wurth_Automotive_WE-HEPA:WE-HEPA_6030_78408063006 -> ds_inductor:1MHL-6.6X6.6
- P12ON, P3ON, P5ON, PWR: value LEDC1608X35N_FLAT-G -> Green; device LED:CHIP-FLAT-G_0603-0.35MM -> ds_LED:LED-GREENLED-0603
- R100, R101, R102, R103, R116, R117, R118, R119, R36, R37, R38, R39, R44, R45, R46, R47, R52, R53, R54, R55, R68, R69, R70, R71, R76, R77, R78, R79, R84, R85, R86, R87: value 470K -> 470K 1%; device ds_passive:R0805 -> ds_resistor:470K-1%0805
- R104, R113, R114, R120, R33, R34, R40, R41, R42, R48, R49, R50, R56, R65, R66, R72, R73, R74, R80, R81, R82, R88, R97, R98: device ds_passive:R0805 -> ds_resistor:1K-1%0805
- R105, R107, R60, R61: value 4.99K -> 4.99K 1%; device ds_passive:R0603 -> ds_resistor:4.99K-1%0603
- R106, R62: value 39R 2W -> 39R 1% 2W; device ds_passive:R2512 -> ds_resistor:39R-1%2512
- R108, R96: value 10K -> 10K 1%; device ds_passive:R0805 -> ds_resistor:10K-1%0805
- R109, R129, R145: value 4.7K -> 4.7K 1%; device ds_passive:R0201 -> ds_resistor:4.7K-1%0201
- R11, R13: value 40.2K -> 40.2K 1%; device ds_passive:R0402 -> ds_resistor:40.2K-1%0402
- R110: value 4.99M -> 1M 1%; device ds_passive:R1206 -> ds_resistor:1M-1%1206
- R112, R122, R123, R151: value 1K -> 1K 1%; device ds_passive:R0402 -> ds_resistor:1K-1%0402
- R115, R25, R26, R27, R28, R29, R30, R31, R32, R35, R43, R51, R67, R75, R83, R99: device ds_passive:R2512 -> ds_resistor:0.002R-1%2512
- R12, R6: value 7.5K -> 7.5K 1%; device ds_passive:R0402 -> ds_resistor:7.5K-1%0402
- R121: device ds_passive:R0201 -> ds_resistor:2.2K-1%0201
- R124, R125: value 5.1K -> 5.1K 1%; device ds_passive:R0201 -> ds_resistor:5.1K-1%0201
- R126, R127: value 10K -> 10K 1%; device ds_passive:R0201 -> ds_resistor:10K-1%0201
- R131: value 1M -> 1M 1%; device ds_passive:R0402 -> ds_resistor:1M-1%0402
- R132, R147, R162, R2, R95: value 10K -> 10K 1%; device ds_passive:R0402 -> ds_resistor:10K-1%0402
- R133, R134, R135, R136: value 3.3R -> 3.3R 1%; device ds_passive:R0201 -> ds_resistor:3.3R-1%0201
- R137, R138, R139, R140: value 49.9R -> 49.9R 1%; device ds_passive:R0201 -> ds_resistor:49.9R-1%0201
- R14: value 12.7K -> 12.7K 1%; device ds_passive:R0402 -> ds_resistor:12.7K-1%0402
- R141, R142, R146: value 470R -> 470R 1%; device ds_passive:R0402 -> ds_resistor:470R-1%0402
- R144: value 1M -> 1M 1%; device ds_passive:R0201 -> ds_resistor:1M-1%0201
- R148: value 2.4 K -> 2.4K 1%; device ds_passive:R0402 -> ds_resistor:2.4K-1%0402
- R15, R160: value 27R -> 27R 1%; device ds_passive:R0201 -> ds_resistor:27R-1%0201
- R150: value 8.2K -> 8.2K 1%; device ds_passive:R0402 -> ds_resistor:8.2K-1%0402
- R152: value 10R -> 10R 1%; device ds_passive:R0201 -> ds_resistor:10R-1%0201
- R153, R154, R155, R156, R157, R158, R159, R16, R59: value 1K -> 1K 1%; device ds_passive:R0201 -> ds_resistor:1K-1%0201
- R17, R18, R19, R20, R21, R22, R23, R24: value 330R 1W -> 330R 1% 1W; device ds_passive:R2512 -> ds_resistor:330R-1%-2512
- R3, R5: value 100K -> 100K 1%; device ds_passive:R0402 -> ds_resistor:100K-1%0402
- R4: value 9.09K -> 9.09K 1%; device ds_passive:R0402 -> ds_resistor:9.09K-1%0402
- R57, R91: value 0R -> 0R 1%; device ds_passive:R0402 -> ds_resistor:0R0402
- R7, R9: value 10R -> 10R 1%; device ds_passive:R0402 -> ds_resistor:10R-1%0402
- R8: value 20K -> 20K 1%; device ds_passive:R0402 -> ds_resistor:20K-1%0402
- R94: value 100K -> 10K 1%; device ds_passive:R0402 -> ds_resistor:10K-1%0402
Connections:
- net 12VRAW: now also C10.+, C13.+, C16.+; no longer C10.1, C13.1, C16.1
- net GND: now also C10.-, C13.-, C16.-; no longer C10.2, C13.2, C16.2
Other:
- moved on the sheet: 12VDC, 3VDC, 3VFB, 5VDC, 5VFB, AVDD, C100, C102, C104, C11, C12, C14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

Commit message: update design to final state
Parts:
- removed USBC: USB-TYPE-C-018, Wurth_Connectors_WR-USB:629722000214
- removed Z1: SMAJ15A, 52101-101-REV-A_v16:SUPRESSOR_TVS-UD-SMAJ
- added D16: SMAJ15A, ds_diode:SMAJ15A
- added PROC: Green, ds_LED:LED-GREENLED-0603
- added R163: 1K 1%, ds_resistor:1K-1%0402
- added USB1: USB-TYPE-C-018, ds_con:USB_C-THT
- AC/DC2: value (none) -> IRM-10-15
- BOOT, RESET: value RS032G05A3SM -> B3U-1000P; device BeagleBone_Blue_R3:RS032G05A3SM-SPST-MOMENTARY-SWSMD-1101NE -> ds_passive:B3U-1000P
- D1: device diode:MBRA340T3 -> ds_diode:MBRA340T3G
- D10, D12, D13, D9: device diode:S1M -> ds_diode:1N4007
- D11, D14: value US1J -> US1J-E3/61T; device diode:S1M -> ds_diode:US1J-E3/61T
- D15: device Diodes:SS12 -> ds_diode:SS12
- D2, D3, D4, D5, D6, D7, D8: value MBRA340T3 -> MBRA340T3G; device diode:MBRA340T3 -> ds_diode:MBRA340T3G
- DSP: value AFC11-S20ICC-00 -> AFC11-S20ICC-00
- ESD1: value SP0503BAHTG-ES -> SP0503BAHTG
- ETH1: value SI-60118-F -> J1B1211CCD; device ds_con:RJ45-CAT5 -> ds_con:J1B1211CCD
- IC1: value MP2315GJ-Z -> MP2315GJ-Z
- IC17, IC22: value MCP6001R -> MCP6001RT-I/OT
- IC19: value CAT24C512HU5IGT3 -> CAT24C256HU4IGT3
- IC2: value MP2315S -> MP2315GJ-Z
- IC3: value ULN2803A -> ULN2803AFWG
- IC4: value MCP23017-E/ML -> MCP23017T-E/ML
- K1, K2, K3, K4, K5, K6, K7, K8: value G2RL-1A-E_DC12 -> G2RL-1A-E DC12
- L4: device ds_passive:R0603 -> ds_inductor:BLM18EG221TN1D
- OPT1, OPT2: value ACPL-247 -> ACPL-247-500E
- R130, R149: value 4D03WGJ0332T5E -> 3.3K 1%; device Resistor Array:742C083103JP -> ds_resistor:3.3K-1%_ARRAY0603X4-1206
- R63, R64: value 4x1K 1206 -> 1K 1%; device Resistor Array:742C083103JP -> ds_resistor:1K-1%_ARRAY0603X4-1206
- R89, R90: value 4x1K 1206 -> 10K 1%; device Resistor Array:742C083103JP -> ds_resistor:10K-1%_ARRAY0603X4-1206
- R94: value 10K 1% -> 100K 1%; device ds_resistor:10K-1%0402 -> ds_resistor:100K-1%0402
- REF1: value LM4040BXX -> LM4040B30FTA
- X1: device Wurth_Quartz Crystals & Oscillators_WE-XTAL:WE-XTAL_CFPX-180_830055295 -> ds_passive:CRYSTAL-3225X322512MSB4SI
- X2: device Wurth_Quartz Crystals & Oscillators_WE-XTAL:WE-XTAL_CFPX-180_830059800 -> ds_passive:CRYSTAL-3225X322525MOB4SI
Connections:
- net N$20 renamed LREC1
- net N$25 renamed SRC1
- net N$26 renamed VNI1
- net N$55 renamed FB1
- net N$57 renamed FBIN1
- net N$77 renamed LREC2
- net N$78 renamed SRC2
- net N$79 renamed VNI2
- net N$80 renamed FB2
- net N$81 renamed FBIN2
- removed net USB_SEL: IC15.GPIO27/ADC1
- new net N$17: IC15.GPIO28/ADC2, R163.2
- new net N$19: PROC.A, R163.1
- net +3V3: now also ETH1.GREEN+, ETH1.YELLOW+; no longer ETH1.GA1, ETH1.GA2
- net 12VRAW: now also D16.C; no longer Z1.C
- net CC1: now also USB1.CC1; no longer USBC.CC1
- net CC2: now also USB1.CC2; no longer USBC.CC2
- net GND: now also BOOT.P$2, D16.A, ETH1.GND, PROC.C, RESET.P$1, USB1.GND; no longer BOOT.2, ETH1.SHIELD-P8, RESET.1, USBC.GND, USBC.GND1, USBC.GND2, USBC.GND3, Z1.A
- net N$82: now also ETH1.YELLOW-; no longer ETH1.GK1
- net N$91: now also ETH1.GREEN-; no longer ETH1.GK2
- net RCT: now also ETH1.P5/RCT; no longer ETH1.RCT
- net RUN: now also RESET.P$2; no longer RESET.2
- net SH: now also USB1.SHILED; no longer USBC.SHIELD
- net TCT: now also ETH1.P4/TCT; no longer ETH1.TCT
- net USB2_DP_N: now also USB1.D-; no longer USBC.D-1, USBC.D-2
- net USB2_DP_P: now also USB1.D+; no longer USBC.D+1, USBC.D+2
- net USB_BOOT: now also BOOT.P$1; no longer BOOT.1
- net VBUS: now also USB1.VBUS; no longer USBC.VBUS, USBC.VBUS1, USBC.VBUS2, USBC.VBUS3
Other:
- note removed: "DISPALY SPI"
- note removed: "DSP I2C"
- note removed: "NETWORK SPI"
- note removed: "PUSHBUTTONS"
- note removed: "REL I2C"
- moved on the sheet: AC/DC1, AC/DC2, C10, C13, C24, C25, C26, C27, C28, C29, C30, C31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

Commit message: update readme with 3D render
Other:
- note added: "230VAC-LIVE"
- note added: "230VAC-NEUTRAL"
- note added: "C13 OUTPUT LIVE"
- note added: "C13 OUTPUT NEUTRAL"
- note added: "DRIVER"
- note added: "I-MEAS V-MEAS"
- note added: "IN1 M IN2 U IN3 X ..."
- note added: "MCU RX"
- note added: "OPTO"
- note added: "OUT"
- note added: "RELAY"
- note added: "RELAY1"
- note added: "RELAY2"
- note added: "RELAY3 ..."
- note added: "SEL A/B/C"
- note added: "SELECTOR"
- note added: "TX1 TX2 TX3 ..."

Commit message: update software, bugfix
Parts:
- R93: value 4x10K 1206 -> 10K 1%; device Resistor Array:742C083103JP -> ds_resistor:10K-1%_ARRAY0603X4-1206
- X1: value 12MHz -> ABM8-272-T3 12MHz

Commit message: Baseline commit. Device is functioning as expected, software is working
Parts:
- added CS0, CS1, MISO0, MISO1, MOSI0, MOSI1, REL0, REL1, REL2, REL3, REL4, REL5, REL6, REL7, RX0, RX1, SCL0, SCL1, SCLK0, SCLK1, SDA0, SDA1: TP, ds_passive:TP
- added FAN: (no value), con-amp-quick:M02
- added R164: 10K 1%, ds_resistor:10K-1%0402
- added R165: NC, ds_passive:R0201
- added T1: (no value), ds_active:BSS138
Connections:
- new net FAN_CTRL: IC15.GPIO27/ADC1, R164.1, R165.1, T1.G
- new net N$23: FAN.1, T1.D
- net !W5500_CS: now also CS1.P$1
- net +12V: now also FAN.2
- net +3V3_MCU: now also R165.2
- net GND: now also R164.2, T1.S
- net I2C0_SCL: now also SCL0.P$1
- net I2C0_SDA: now also SDA0.P$1
- net I2C1_SCL: now also SCL1.P$1
- net I2C1_SDA: now also SDA1.P$1
- net LCD_CS: now also CS0.P$1
- net LCD_MISO: now also MISO0.P$1
- net LCD_MOSI: now also MOSI0.P$1
- net LCD_SCLK: now also SCLK0.P$1
- net REL_0: now also REL0.P$1
- net REL_1: now also REL1.P$1
- net REL_2: now also REL2.P$1
- net REL_3: now also REL3.P$1
- net REL_4: now also REL4.P$1
- net REL_5: now also REL5.P$1
- net REL_6: now also REL6.P$1
- net REL_7: now also REL7.P$1
- net UART0_RX: now also RX0.P$1
- net UART0_TX: now also RX1.P$1
- net W5500_MISO: now also MISO1.P$1
- net W5500_MOSI: now also MOSI1.P$1
- net W5500_SCK: now also SCLK1.P$1
Other:
- note added: "FAN"
- moved on the sheet: PROC, R130, R163
