File: src/HardwareDesign/ENERGIS/Rev1.0.0/ENERGIS_DispBrd_Rack-PDU_1.0.3.brd (EAGLE design)
At the start: 124 x 40 mm, 62 parts, among them CON1 FPC40-HD, CON2 AFC11-S20ICC-00, IC1 MCP23017-E/ML, IC2 MCP23017-E/ML, T1 BSS138

Commit message: update DspBoard
Parts:
- added DSP: (no value), ds_con:1X4
Connections:
- net +3V3: now also DSP.2
- net GND: now also DSP.1
- net I2C0_SCL: now also DSP.3
- net I2C0_SDA: now also DSP.4
Routing:
- net I2C0_SCL: track 60.3 -> 76.2 mm, vias 0 -> 2
- net I2C0_SDA: track 64.3 -> 78.4 mm, vias 2 -> 4
- net GND: track 420.4 -> 429.7 mm, vias 67 -> 68
- net +3V3: track 240.5 -> 245.4 mm
- net +5V: track 81.4 -> 82.5 mm
Changed lines of the file:
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@@
 <attribute name="NAME" x="37.42946875" y="34.351221875" size="1.27" layer="26" rot="MR225"/>
+</element>
+<element name="DSP" library="ds_con" package="1X4" package3d_urn="urn:adsk.eagle:package:46684991/2" value="" x="21.07" y="37.77" smashed="yes" rot="MR270">
+<attribute name="NAME" x="15.885" y="41.355" size="1.778" layer="26" rot="MR180"/>
+<attribute name="VALUE" x="28.69" y="39.675" size="1.778" layer="28" rot="MR270"/>
 </element>
 </elements>
@@
 <wire x1="13.2" y1="31.9" x2="13.16" y2="31.86" width="0.4064" layer="16"/>
 <wire x1="13.16" y1="31.86" x2="6.64" y2="31.86" width="0.4064" layer="16"/>
-<wire x1="57.1" y1="42.6" x2="17.3" y2="42.6" width="0.4064" layer="1"/>
+<wire x1="57.1" y1="42.6" x2="19.72" y2="42.6" width="0.4064" layer="1"/>
+<wire x1="19.72" y1="42.6" x2="17.3" y2="42.6" width="0.4064" layer="1"/>
 <wire x1="17.3" y1="42.6" x2="13.5" y2="38.8" width="0.4064" layer="1"/>
 <wire x1="18.896" y1="24.714" x2="15.986" y2="24.714" width="0.4064" layer="1"/>
@@
 <wire x1="54.8687" y1="31.4313" x2="55.3" y2="31" width="0.254" layer="1"/>
 <wire x1="55.3" y1="31" x2="59.222" y2="31" width="0.254" layer="1"/>
+<contactref element="DSP" pad="2"/>
+<wire x1="19.78" y1="42.54" x2="19.72" y2="42.6" width="0.3048" layer="1"/>
+<wire x1="19.8" y1="37.77" x2="19.8" y2="42.52" width="0.3048" layer="1"/>
+<wire x1="19.8" y1="42.52" x2="19.78" y2="42.54" width="0.3048" layer="1"/>
 </signal>
 <signal name="GND">
@@
 <via x="31.26" y="34.75" extent="1-16" drill="0.35"/>
 <via x="32.01" y="35.5" extent="1-16" drill="0.35"/>
+<contactref element="DSP" pad="1"/>
+<wire x1="17.13" y1="37.87" x2="16.55" y2="37.87" width="0.2" layer="16"/>
+<via x="12.54" y="37.87" extent="1-16" drill="0.35"/>
+<wire x1="16.55" y1="37.87" x2="12.54" y2="37.87" width="0.2" layer="16"/>
+<wire x1="12.54" y1="37.87" x2="9.63" y2="37.87" width="0.2" layer="1"/>
+<wire x1="9.63" y1="37.87" x2="8.9" y2="38.6" width="0.2" layer="1"/>
+<wire x1="17.26" y1="37.77" x2="16.65" y2="37.77" width="0.2" layer="16"/>
+<wire x1="16.65" y1="37.77" x2="16.55" y2="37.87" width="0.2" layer="16"/>
 </signal>
 <signal name="LCD_CS">
@@
 <wire x1="53.6583" y1="23.7" x2="52.218840625" y2="22.260540625" width="0.254" layer="1"/>
 <wire x1="52.218840625" y1="22.260540625" x2="51.1914625" y2="22.260540625" width="0.254" layer="1"/>
-<wire x1="6.69" y1="42.24" x2="14.46" y2="42.24" width="0.254" layer="16"/>
-<wire x1="20.5" y1="36.2" x2="20.5" y2="24" width="0.254" layer="16"/>
+<wire x1="19.15" y1="35.83" x2="12.69" y2="35.83" width="0.254" layer="16"/>
+<wire x1="6.69" y1="42.24" x2="9.87" y2="42.24" width="0.254" layer="16"/>
+<wire x1="9.87" y1="42.24" x2="10.61" y2="41.5" width="0.254" layer="16"/>
+<wire x1="10.61" y1="41.5" x2="10.61" y2="37.91" width="0.254" layer="16"/>
+<wire x1="10.61" y1="37.91" x2="12.69" y2="35.83" width="0.254" layer="16"/>
+<wire x1="20.5" y1="34.48" x2="20.5" y2="24" width="0.254" layer="16"/>
 <wire x1="20.5" y1="24" x2="23.1" y2="21.4" width="0.254" layer="16"/>
 <wire x1="47.9" y1="21.4" x2="48" y2="21.5" width="0.254" layer="16"/>
@@
 <wire x1="48" y1="21.5" x2="48.760540625" y2="22.260540625" width="0.254" layer="1"/>
 <wire x1="48.760540625" y1="22.260540625" x2="51.1914625" y2="22.260540625" width="0.254" layer="1"/>
-<wire x1="14.46" y1="42.24" x2="20.5" y2="36.2" width="0.254" layer="16"/>
+<wire x1="19.15" y1="35.83" x2="20.5" y2="34.48" width="0.254" layer="16"/>
 <wire x1="23.1" y1="21.4" x2="47.9" y2="21.4" width="0.254" layer="16"/>
 </signal>
@@
 <contactref element="CON2" pad="6"/>
 <contactref element="IC2" pad="9"/>
-<wire x1="30.80844375" y1="30.969965625" x2="29" y2="29.161521875" width="0.2" layer="16"/>
+<wire x1="30.80844375" y1="30.969965625" x2="29.9892375" y2="30.150759375" width="0.2" layer="16"/>
+<wire x1="29.9892375" y1="30.150759375" x2="29" y2="29.161521875" width="0.2" layer="16"/>
 <wire x1="29" y1="29.161521875" x2="29" y2="24.74774375" width="0.2" layer="16"/>
 <wire x1="29" y1="24.74774375" x2="31.67994375" y2="22.0678" width="0.2" layer="16"/>
@@
 <wire x1="57.326128125" y1="27.573871875" x2="57.3" y2="27.6" width="0.2" layer="16"/>
 <wire x1="64.984615625" y1="26.7905" x2="57.66175625" y2="26.7905" width="0.2" layer="16"/>
+<contactref element="DSP" pad="4"/>
+<via x="24.13" y="35.23" extent="1-16" drill="0.35"/>
+<wire x1="24.13" y1="35.23" x2="23.45" y2="35.23" width="0.2" layer="1"/>
+<wire x1="22.96" y1="34.74" x2="22.96" y2="34.01" width="0.2" layer="1"/>
+<wire x1="22.96" y1="34.01" x2="24.62" y2="32.35" width="0.2" layer="1"/>
+<wire x1="28.69" y1="32.35" x2="29.48" y2="31.56" width="0.2" layer="1"/>
+<wire x1="29.48" y1="31.56" x2="29.48" y2="30.71164375" width="0.2" layer="1"/>
+<wire x1="29.48" y1="30.71164375" x2="29.464178125" y2="30.695821875" width="0.2" layer="1"/>
+<via x="29.464178125" y="30.695821875" extent="1-16" drill="0.35"/>
+<wire x1="29.464178125" y1="30.695821875" x2="29.464178125" y2="30.67581875" width="0.2" layer="16"/>
+<wire x1="29.464178125" y1="30.67581875" x2="29.9892375" y2="30.150759375" width="0.2" layer="16"/>
+<wire x1="23.45" y1="35.23" x2="22.96" y2="34.74" width="0.2" layer="1"/>
+<wire x1="24.62" y1="32.35" x2="28.69" y2="32.35" width="0.2" layer="1"/>
+<wire x1="24.88" y1="37.77" x2="24.88" y2="35.98" width="0.2" layer="16"/>
+<wire x1="24.88" y1="35.98" x2="24.13" y2="35.23" width="0.2" layer="16"/>
 </signal>
 <signal name="I2C0_SCL">
@@
 <contactref element="CON2" pad="7"/>
 <contactref element="IC2" pad="8"/>
-<wire x1="31.268065625" y1="30.51034375" x2="29.4" y2="28.642278125" width="0.2" layer="16"/>
+<wire x1="31.268065625" y1="30.51034375" x2="31.0638625" y2="30.306140625" width="0.2" layer="16"/>
+<wire x1="31.0638625" y1="30.306140625" x2="29.4" y2="28.642278125" width="0.2" layer="16"/>
 <wire x1="52.32438125" y1="22.4583" x2="52.6417" y2="22.77561875" width="0.2" layer="16"/>
 <wire x1="52.6417" y1="22.77561875" x2="52.6417" y2="24.1417" width="0.2" layer="16"/>
@@
 <wire x1="52.6417" y1="24.1417" x2="56.178" y2="27.678" width="0.2" layer="16"/>
 <wire x1="56.178" y1="27.678" x2="56.222" y2="27.678" width="0.2" layer="16"/>
+<contactref element="DSP" pad="3"/>
+<wire x1="22.32" y1="35.69" x2="23.69" y2="34.32" width="0.2" layer="16"/>
+<via x="23.69" y="34.32" extent="1-16" drill="0.35"/>
+<wire x1="23.69" y1="34.32" x2="25.08" y2="32.93" width="0.2" layer="1"/>
+<wire x1="28.95" y1="32.93" x2="31.81" y2="30.07" width="0.2" layer="1"/>
+<wire x1="31.81" y1="30.07" x2="31.78" y2="30.04" width="0.2" layer="1"/>
+<wire x1="31.78" y1="30.04" x2="31.78" y2="29.36" width="0.2" layer="1"/>
+<via x="31.78" y="29.36" extent="1-16" drill="0.35"/>
+<wire x1="31.78" y1="29.36" x2="31.0638625" y2="30.0761375" width="0.2" layer="16"/>
+<wire x1="31.0638625" y1="30.0761375" x2="31.0638625" y2="30.306140625" width="0.2" layer="16"/>
+<wire x1="25.08" y1="32.93" x2="28.95" y2="32.93" width="0.2" layer="1"/>
+<wire x1="22.34" y1="37.77" x2="22.32" y2="37.75" width="0.2" layer="16"/>
+<wire x1="22.32" y1="37.75" x2="22.32" y2="35.69" width="0.2" layer="16"/>
 </signal>
 <signal name="LCD_BL">

Commit message: update documentation
Parts:
- added U$1, U$5: (no value), ds_silkscreen:DMT

Commit message: update software, bugfix
Parts:
- removed S4: TC-6601-5.0-160, Wurth_Switch_WS-TASV:430182043816
- added PWR: TS-1002S-04326C, ds_passive:PUSHBUTTON-6X6
- <, >, O: value TC-6601-5.0-160 -> TS-1002S-04326C; device Wurth_Switch_WS-TASV:430182043816 -> ds_passive:PUSHBUTTON-6X6
- C1, C3: value 10uF -> DNI
- C10, C11, C12, C5, C6, C7, C8, C9: value 100nF -> 100nF 50V; device ds_passive:C0402 -> ds_capacitors:0402
- C2, C4: value 100nF -> DNI
- CH1, CH2, CH3, CH4, CH5, CH6, CH7, CH8: value (none) -> Green; device led:CHIP-LED0805 -> ds_LED:LED-0805
- CON1: value FPC40-HD -> DNI
- CON2: value AFC11-S20ICC-00 -> AFC11-S20ICC-00
- DSP: value (none) -> DNI
- IC1, IC2: value MCP23017-E/ML -> MCP23017T-E/ML
- LED1: value (none) -> GREEN; device led:LED3MM -> ds_LED:LED3MM
- LED2: value XL-2012UBC -> BLUE; device led:LED3MM -> ds_LED:LED3MM
- LED3: value XL-2012SURC -> RED; device led:LED3MM -> ds_LED:LED3MM
- R1, R2, R3: value 56R -> DNI
- R10, R11, R7: value 1K -> 1K 1%; device ds_passive:0402 -> ds_resistor:0402
- R12, R13, R4, R5, R6: value 10K -> 10K 1%; device ds_passive:0402 -> ds_resistor:0402
- R14, R15, R8, R9: value 4D03WGJ0102T5E 1K -> 1K 1%; device Resistor Array:742C083103JP -> ds_resistor:_0603X4-1206
- SEL1, SEL2, SEL3, SEL4, SEL5, SEL6, SEL7, SEL8: value (none) -> Orange; device led:CHIP-LED0805 -> ds_LED:LED-0805
- moved U$5 72.1 mm to (107.6, 27.7)
- moved U$2 42.9 mm to (123.2, 28.7)
- moved R4 38.3 mm to (21.4, 26.8), turned to 90 degrees
- moved C1 35.7 mm to (21.3, 30.5), turned to 270 degrees
- moved T1 35.4 mm to (23.9, 26.7), turned to 90 degrees
- moved R3 34.2 mm to (22.5, 30.5), turned to 90 degrees
- moved R2 32.6 mm to (23.8, 30.5), turned to 90 degrees
- moved R1 31.1 mm to (25.0, 30.5), turned to 270 degrees
- moved CON1 21.8 mm to (30.1, 49.6), turned to 270 degrees
- moved C3 19.8 mm to (36.2, 28.1), flipped to the bottom, turned to 90 degrees
- moved U$4 19.2 mm to (8.80, 37.7)
- moved C4 18.3 mm to (37.3, 28.1), flipped to the bottom, turned to 90 degrees
- moved C2 17.0 mm to (38.5, 28.1), flipped to the bottom, turned to 90 degrees
- moved > 11.8 mm to (70.0, 37.9), turned to 0 degrees
- moved O 11.7 mm to (49.9, 37.9), turned to 0 degrees
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Connections:
- net GND: now also <.1, >.1, O.1, PWR.1, PWR.2; no longer <.4, >.4, O.4, S4.2, S4.4
- net KEY_0: now also <.4; no longer <.1
- net KEY_1: now also >.4; no longer >.1
- net KEY_2: now also O.4; no longer O.1
- net KEY_3: now also PWR.3, PWR.4; no longer S4.1, S4.3
- net N$10: now also R14.B1; no longer R14.2
- net N$11: now also R14.A1; no longer R14.1
- net N$12: now also R15.D1; no longer R15.4
- net N$13: now also R15.C1; no longer R15.3
- net N$14: now also R15.B1; no longer R15.2
- net N$15: now also R15.A1; no longer R15.1
- net N$16: now also R14.D2; no longer R14.5
- net N$17: now also R14.C2; no longer R14.6
- net N$18: now also R14.B2; no longer R14.7
- net N$19: now also R14.A2; no longer R14.8
- net N$20: now also R15.D2; no longer R15.5
- net N$21: now also R15.C2; no longer R15.6
- net N$22: now also R15.B2; no longer R15.7
- net N$23: now also R15.A2; no longer R15.8
- net N$50: now also R8.D1; no longer R8.4
- net N$51: now also R8.C1; no longer R8.3
- net N$52: now also R8.B1; no longer R8.2
- net N$53: now also R8.A1; no longer R8.1
- net N$54: now also R9.D1; no longer R9.4
- net N$55: now also R9.C1; no longer R9.3
- net N$56: now also R9.B1; no longer R9.2
- net N$57: now also R9.A1; no longer R9.1
- net N$58: now also R8.D2; no longer R8.5
- net N$59: now also R8.C2; no longer R8.6
- net N$60: now also R8.B2; no longer R8.7
- net N$61: now also R8.A2; no longer R8.8
- net N$62: now also R9.D2; no longer R9.5
- net N$63: now also R9.C2; no longer R9.6
- net N$64: now also R9.B2; no longer R9.7
- net N$65: now also R9.A2; no longer R9.8
- net N$8: now also R14.D1; no longer R14.4
- net N$9: now also R14.C1; no longer R14.3
Routing:
- net GND: track 429.7 -> 123.6 mm, vias 68 -> 37
- net +3V3: track 245.4 -> 199.2 mm, vias 9 -> 11
- net I2C0_SCL: track 76.2 -> 109.6 mm, vias 2 -> 3
- net LCD_BL: track 90.9 -> 60.2 mm, vias 2 -> 0
- net I2C0_SDA: track 78.4 -> 100.5 mm, vias 4 -> 2
- net LCD_RES: track 11.6 -> 29.7 mm
- net LCD_MISO: track 9.03 -> 24.7 mm
- net LCD_MOSI: track 12.2 -> 27.7 mm
- net KEY_1: track 23.2 -> 36.2 mm, vias 1 -> 3
- net LCD_SCLK: track 10.2 -> 23.0 mm
- net LCD_DC: track 13.7 -> 25.3 mm
- net +5V: track 82.5 -> 93.5 mm, vias 4 -> 3
- net N$65: track 17.7 -> 6.81 mm
- net KEY_0: track 46.3 -> 35.8 mm
- net LCD_CS: track 10.7 -> 21.1 mm
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Other:
- board size 124 x 40 mm -> 124 x 28 mm
- board text removed: "4"

Commit message: Baseline commit. Device is functioning as expected, software is working
Parts:
- added CS, MISO, MOSI, SCK, SCL0, SDA0: TP, ds_passive:TP
- renumbered TP1 to 3V3, TP16 to GND, TP2 to 5V, TP3 to BL
Connections:
- net I2C0_SCL: now also SCL0.TP
- net I2C0_SDA: now also SDA0.TP
- net LCD_CS: now also CS.TP
- net LCD_MISO: now also MISO.TP
- net LCD_MOSI: now also MOSI.TP
- net LCD_SCLK: now also SCK.TP
Routing:
- net I2C0_SDA: track 100.5 -> 110.7 mm
- net I2C0_SCL: track 109.6 -> 119.3 mm
- net LCD_MISO: track 24.7 -> 31.0 mm, vias 1 -> 2
- net LCD_MOSI: track 27.7 -> 32.6 mm, vias 1 -> 2
- net LCD_SCLK: track 23.0 -> 27.7 mm, vias 1 -> 2
- net LCD_CS: track 21.1 -> 25.1 mm, vias 1 -> 2
