File: src/HardwareDesign/ENERGIS/Rev1.0.0/ENERGIS_DispBrd_Rack-PDU_1.0.3.sch (EAGLE design)
At the start: 55 parts, among them CON1 FPC40-HD, CON2 FPC20-H, IC1 MCP23017-E/ML, T1 BSS138

Commit message: update schematics
Parts:
- removed S1, S2, S3: TC-6601-5.0-160, Wurth_Switch_WS-TASV:430182043816
- removed TP10, TP11, TP12, TP13, TP14, TP15, TP4, TP5, TP6, TP7, TP8, TP9: TP, ds_passive:TP
- added <, >, O, S4: TC-6601-5.0-160, Wurth_Switch_WS-TASV:430182043816
- added C10, C11, C12: 100nF, ds_passive:C-0402
- added IC2: MCP23017-E/ML, ds_ic_peripherals:MCP23017-E/ML
- added R13: 10K, ds_passive:R0402
- added R14, R15: 4D03WGJ0102T5E 1K, Resistor Array:742C083103JP
- added SEL1, SEL2, SEL3, SEL4, SEL5, SEL6, SEL7, SEL8: (no value), led:LEDCHIP-LED0805
- CON2: value FPC20-H -> AFC11-S20ICC-00; device ds_con:FPC20-H -> ds_con:AFC11-S20ICC-00
- LED1, LED2, LED3: device led:LEDCHIP-LED0805 -> led:LED3MM
- renumbered LED10 to CH7, LED11 to CH8, LED4 to CH1, LED5 to CH2, LED6 to CH3, LED7 to CH4, LED8 to CH5, LED9 to CH6
Connections:
- new net N$10: IC2.IO1.2, R14.2
- new net N$11: IC2.IO1.3, R14.1
- new net N$12: IC2.IO1.4, R15.4
- new net N$13: IC2.IO1.5, R15.3
- new net N$14: IC2.IO1.6, R15.2
- new net N$15: IC2.IO1.7, R15.1
- new net N$16: R14.5, SEL1.A
- new net N$17: R14.6, SEL2.A
- new net N$18: R14.7, SEL3.A
- new net N$19: R14.8, SEL4.A
- new net N$20: R15.5, SEL5.A
- new net N$21: R15.6, SEL6.A
- new net N$22: R15.7, SEL7.A
- new net N$23: R15.8, SEL8.A
- new net N$8: IC2.IO1.0, R14.4
- new net N$9: IC2.IO1.1, R14.3
- net +3V3: now also C11.1, C12.1, IC2.A0, IC2.A1, IC2.VDD, R13.1
- net GND: now also <.2, <.4, >.2, >.4, C10.2, C11.2, C12.2, IC2.A2, IC2.VSS, O.2, O.4, S4.2, S4.4, SEL1.C, SEL2.C, SEL3.C, SEL4.C, SEL5.C, SEL6.C, SEL7.C, SEL8.C; no longer S1.2, S1.4, S2.2, S2.4, S3.2, S3.4
- net I2C0_SCL: now also IC2.SCL; no longer TP15.P$1
- net I2C0_SDA: now also IC2.SDA; no longer TP14.P$1
- net KEY_0: now also <.1, <.3; no longer S1.1, S1.3, TP9.P$1
- net KEY_1: now also >.1, >.3; no longer S2.1, S2.3, TP10.P$1
- net KEY_2: now also O.1, O.3; no longer S3.1, S3.3, TP11.P$1
- net KEY_3: now also C10.1, R13.2, S4.1, S4.3
- net LCD_CS: no longer TP5.P$1
- net LCD_DC: no longer TP4.P$1
- net LCD_MISO: no longer TP7.P$1
- net LCD_MOSI: no longer TP8.P$1
- net LCD_RES: no longer TP13.P$1
- net LCD_SCLK: no longer TP6.P$1
- net MCP_LCD_RST: now also IC2.!RESET; no longer TP12.P$1
Other:
- moved on the sheet: C7, C8, C9, R12, R5, R6, TP1, TP16, TP2, TP3

Commit message: update DspBoard
Parts:
- added DSP: (no value), ds_con:CON-1X4
Connections:
- net +3V3: now also DSP.P$2
- net GND: now also DSP.P$1
- net I2C0_SCL: now also DSP.P$3
- net I2C0_SDA: now also DSP.P$4

Commit message: update software, bugfix
Parts:
- removed S4: TC-6601-5.0-160, Wurth_Switch_WS-TASV:430182043816
- added PWR: TS-1002S-04326C, ds_passive:SWITCH6X6-SHORT
- <, >, O: value TC-6601-5.0-160 -> TS-1002S-04326C; device Wurth_Switch_WS-TASV:430182043816 -> ds_passive:SWITCH6X6-SHORT
- C1, C3: value 10uF -> DNI
- C10, C11, C12, C5, C6, C7, C8, C9: value 100nF -> 100nF 50V; device ds_passive:C-0402 -> ds_capacitors:100NF-50V-0402
- C2, C4: value 100nF -> DNI
- CH1, CH2, CH3, CH4, CH5, CH6, CH7, CH8: value (none) -> Green; device led:LEDCHIP-LED0805 -> ds_LED:LED-GREENLED-0805
- CON1: value FPC40-HD -> DNI
- CON2: value AFC11-S20ICC-00 -> AFC11-S20ICC-00
- DSP: value (none) -> DNI
- IC1, IC2: value MCP23017-E/ML -> MCP23017T-E/ML
- LED1: value (none) -> GREEN; device led:LED3MM -> ds_LED:LED-GREEN3MM-CLEAR
- LED2: value XL-2012UBC -> BLUE; device led:LED3MM -> ds_LED:LED-BLUE3MM-CLEAR
- LED3: value XL-2012SURC -> RED; device led:LED3MM -> ds_LED:LED-RED3MM-CLEAR
- R1, R2, R3: value 56R -> DNI
- R10, R11, R7: value 1K -> 1K 1%; device ds_passive:R0402 -> ds_resistor:1K-1%0402
- R12, R13, R4, R5, R6: value 10K -> 10K 1%; device ds_passive:R0402 -> ds_resistor:10K-1%0402
- R14, R15, R8, R9: value 4D03WGJ0102T5E 1K -> 1K 1%; device Resistor Array:742C083103JP -> ds_resistor:1K-1%_ARRAY0603X4-1206
- SEL1, SEL2, SEL3, SEL4, SEL5, SEL6, SEL7, SEL8: value (none) -> Orange; device led:LEDCHIP-LED0805 -> ds_LED:LED-ORANGELED-0805
Connections:
- net GND: now also <.P$1, >.P$1, O.P$1, PWR.P$1; no longer <.2, <.4, >.2, >.4, O.2, O.4, S4.2, S4.4
- net KEY_0: now also <.P$2; no longer <.1, <.3
- net KEY_1: now also >.P$2; no longer >.1, >.3
- net KEY_2: now also O.P$2; no longer O.1, O.3
- net KEY_3: now also PWR.P$2; no longer S4.1, S4.3
Other:
- moved on the sheet: C12, C6

Commit message: Baseline commit. Device is functioning as expected, software is working
Parts:
- added CS, MISO, MOSI, SCK, SCL0, SDA0: TP, ds_passive:TP
- renumbered TP1 to 3V3, TP16 to GND, TP2 to 5V, TP3 to BL
Connections:
- net I2C0_SCL: now also SCL0.P$1
- net I2C0_SDA: now also SDA0.P$1
- net LCD_CS: now also CS.P$1
- net LCD_MISO: now also MISO.P$1
- net LCD_MOSI: now also MOSI.P$1
- net LCD_SCLK: now also SCK.P$1
