File: src/Hardware-Design/ENERGIS/Rev1.0.1/ENERGIS_Rack-PDU_1.0.1.sch (EAGLE design)
At the start: 419 parts, among them IC1 MP2315GJ-Z, IC10 HLW8032, IC11 HLW8032, IC12 HLW8032, IC13 MP150GJ, IC14 HLW8032, IC15 RP2040, IC16 HLW8032, IC17 MCP6001RT-I/OT, IC18 W25Q128JVPIQ, IC19 CAT24C256HU4IGT3, IC2 MP2315GJ-Z, IC20 W5500, IC21 MIC5504-3.3YM5, IC22 MCP6001RT-I/OT, IC3 ULN2803AFWG, IC4 MCP23017T-E/ML, IC5 MP150GJ, IC6 HLW8032, IC7 HLW8032, IC8 HLW8032, IC9 SN74HC151PWR, J10 0R 1%, J2 JP, J7 JP, J8 0R 1%, J9 0R 1%, K1 G2RL-1A-E DC12, K2 G2RL-1A-E DC12, K3 G2RL-1A-E DC12, K4 G2RL-1A-E DC12, K5 G2RL-1A-E DC12, K6 G2RL-1A-E DC12, K7 G2RL-1A-E DC12, K8 G2RL-1A-E DC12, P12ON Green, P3ON Green, P5ON Green, SW3 TP, X1 ABM8-272-T3 12MHz, X2 25MHz

Commit message: Add software ESD protection to button control and port expanders. Design sheet metal shielding around electronics. Add ethernet test
Parts:
- added D17, D18: RCLAMP0582BQTCT, ds_diode:RCLAMP0582BQTCT
- added RN1, RN2: 100K 1%, ds_resistor:100K-1%_ARRAY0603X4-1206
- R17, R18, R19, R20, R21, R22, R23, R24: value 330R 1% 1W -> 0R 1%; device ds_resistor:330R-1%-2512 -> ds_resistor:0R2512
Connections:
- net GND: now also D17.3, D18.3, RN1A.1, RN1B.1, RN1C.1, RN1D.1, RN2A.1, RN2B.1, RN2C.1, RN2D.1
- net I2C0_SCL: now also D17.1
- net I2C0_SDA: now also D17.2
- net I2C1_SCL: now also D18.1
- net I2C1_SDA: now also D18.2
- net REL_0: now also RN1A.2
- net REL_1: now also RN1B.2
- net REL_2: now also RN1C.2
- net REL_3: now also RN1D.2
- net REL_4: now also RN2A.2
- net REL_5: now also RN2B.2
- net REL_6: now also RN2C.2
- net REL_7: now also RN2D.2
Other:
- moved on the sheet: C19, C20, RX0, RX1, SCL0, SCL1, SDA0, SDA1
