File: src/Hardware-Design/ENERGIS/Rev1.1.0/ENERGIS_DispBrd_Rack-PDU_1.1.0.brd (EAGLE design)
At the start: 124 x 28 mm, 80 parts, among them CON1 DNI, CON2 AFC11-S20ICC-00, IC1 MCP23017T-E/ML, IC2 MCP23017T-E/ML, T1 BSS138

Commit message: adapt design to NextPCB dru
Parts:
- removed U$2, U$3, U$4: (no value), holes:3,2
- added H1, H2, H3: MOUNT-PAD-ROUND3.2, holes:3,2-PAD
- added U$10: (no value), SparkFun-Aesthetics:NO_PB_LOGO_0.120
- added U$6, U$7: (no value), ds_silkscreen:NEXTPCB_SMALL
- added U$8: (no value), logo:CE-4MM
- added U$9: (no value), SparkFun-Aesthetics:ROHS_LOGO_0.18_IN
- 3V3, 5V, BL, CS, GND, MISO, MOSI, SCK, SCL0, SDA0: value TP -> TP-ROUND; device ds_passive:TP -> ds_passive:TP-ROUND
- moved U$5 18.7 mm to (106.8, 46.4)
- moved SDA0 11.1 mm to (14.1, 33.6), turned to 270 degrees
- moved SCL0 10.8 mm to (14.0, 36.0), turned to 90 degrees
- moved R4 9.13 mm to (29.6, 30.6)
- moved T1 5.27 mm to (27.4, 30.7), turned to 0 degrees
- moved R11 3.83 mm to (95.6, 46.8)
- moved R7 3.54 mm to (95.7, 31.0)
- moved R10 3.49 mm to (95.6, 38.8)
- moved R8 3.13 mm to (73.4, 41.9), turned to 315 degrees
- moved R14 2.64 mm to (28.0, 42.3), turned to 315 degrees
- moved R9 1.79 mm to (80.0, 42.8), turned to 45 degrees
- moved U$1 1.62 mm to (111.8, 45.7)
- moved R15 1.19 mm to (33.9, 43.3), turned to 45 degrees
- moved CS 0.80 mm to (47.7, 28.2)
- moved BL 0.80 mm to (6.77, 32.2)
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Connections:
- net GND: now also H1.B3,2, H2.B3,2, H3.B3,2
Routing:
- net GND: track 169.3 -> 118.6 mm, vias 40 -> 238
- net I2C0_SCL: track 119.1 -> 83.5 mm, vias 3 -> 4
- net I2C0_SDA: track 111.3 -> 85.8 mm, vias 2 -> 4
- net N$28: track 0.00 -> 25.2 mm
- net N$27: track 0.00 -> 23.6 mm
- net LCD_MOSI: track 32.6 -> 41.6 mm, vias 2 -> 4
- net N$1: track 16.6 -> 23.6 mm
- net N$6: track 16.6 -> 23.6 mm
- net N$18: track 3.51 -> 10.2 mm, vias 1 -> 2
- net MCP_LCD_RST: track 54.5 -> 60.9 mm
- net N$19: track 12.1 -> 18.5 mm, vias 1 -> 2
- net KEY_0: track 40.7 -> 46.5 mm, vias 3 -> 2
- net N$65: track 6.81 -> 12.5 mm, vias 1 -> 2
- net LCD_MISO: track 31.0 -> 36.5 mm, vias 2 -> 3
- net N$24: track 14.2 -> 19.7 mm, vias 0 -> 2
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- added copper zone on layer 15, net GND
- added copper zone on layer 2, net GND
Other:
- board text added: "3"
- board text added: "4"

Commit message: update version to 1.1.0
Parts:
- moved C2 0.48 mm to (38.5, 28.6)
- moved C4 0.45 mm to (37.3, 28.6)
- moved C3 0.45 mm to (36.1, 28.6)
Routing:
- net GND: track 118.6 -> 120.5 mm
- net LCD_DC: track 26.6 -> 27.5 mm
- net +3V3: track 205.3 -> 206.0 mm
- net LCD_MOSI: track 41.6 -> 42.1 mm

Commit message: update Readme
Parts:
- 3V3, 5V, BL, CS, GND, MISO, MOSI, SCK, SCL0, SDA0: value TP-ROUND -> DNI
- C10, C11, C12, C5, C6, C7, C8, C9: value 100nF 50V -> 100nF 25V
- D5: device ds_diode:SOT-523 -> ds_diode:SC75
- H1, H2, H3: value MOUNT-PAD-ROUND3.2 -> DNI
- R4: value 10K 1% -> DNI
- T1: value BSS138 -> DNI; device transistor-fet:SOT23 -> ds_active:SOT23
- U$1, U$10, U$5, U$6, U$7, U$8, U$9: value (none) -> DNI
Routing:
- net GND: track 120.5 -> 121.1 mm
