File: src/Hardware-Design/ENERGIS/Rev1.1.0/ENERGIS_DispBrd_Rack-PDU_1.1.0.sch (EAGLE design)
At the start: 75 parts, among them CON1 DNI, CON2 AFC11-S20ICC-00, IC1 MCP23017T-E/ML, IC2 MCP23017T-E/ML, T1 BSS138

Commit message: adapt design to NextPCB dru
Parts:
- added H1, H2, H3: MOUNT-PAD-ROUND3.2, holes:MOUNT-PAD-ROUND3.2
- 3V3, 5V, BL, CS, GND, MISO, MOSI, SCK, SCL0, SDA0: value TP -> TP-ROUND; device ds_passive:TP -> ds_passive:TP-ROUND
Connections:
- net GND: now also H1.MOUNT, H2.MOUNT, H3.MOUNT
Other:
- note added: "I2C DISPLAY"
- note removed: "Rev 2.0"

Commit message: update Readme
Parts:
- 3V3, 5V, BL, CS, GND, MISO, MOSI, SCK, SCL0, SDA0: value TP-ROUND -> DNI
- C10, C11, C12, C5, C6, C7, C8, C9: value 100nF 50V -> 100nF 25V; device ds_capacitors:100NF-50V-0402 -> ds_capacitors:100NF-25V-0402
- D5: device ds_diode:RCLAMP0582BQTCT -> ds_diode:RCLAMP0582BQTCT-
- H1, H2, H3: value MOUNT-PAD-ROUND3.2 -> DNI
- R4: value 10K 1% -> DNI
- T1: value BSS138 -> DNI; device transistor-fet:BSS138 -> ds_active:BSS138
Other:
- note added: "10K"
- note added: "BSS138"
