File: src/Hardware-Design/ENERGIS/Rev1.1.0/ENERGIS_Rack-PDU_1.1.0.brd (EAGLE design)
At the start: 210 x 108 mm, 442 parts, among them IC1 MP2315GJ-Z, IC10 HLW8032, IC11 HLW8032, IC12 HLW8032, IC13 MP150GJ, IC14 HLW8032, IC15 RP2040, IC16 HLW8032, IC17 MCP6001RT-I/OT, IC18 W25Q128JVPIQ, IC19 CAT24C256HU4IGT3, IC2 MP2315GJ-Z, IC20 W5500, IC21 MIC5504-3.3YM5, IC22 MCP6001RT-I/OT, IC3 ULN2803AFWG, IC4 MCP23017T-E/ML, IC5 MP150GJ, IC6 HLW8032, IC7 HLW8032, IC8 HLW8032, IC9 CD74ACT151M96, J10 0R 1%, J2 DNI, J7 DNI, J8 0R 1%, J9 0R 1%, K1 G2RL-1A-E DC12, K2 G2RL-1A-E DC12, K3 G2RL-1A-E DC12, K4 G2RL-1A-E DC12, K5 G2RL-1A-E DC12, K6 G2RL-1A-E DC12, K7 G2RL-1A-E DC12, K8 G2RL-1A-E DC12, P12ON Green, P3ON Green, P5ON Green, SW3 TESTPOINT, T1 BSS138, X1 ABM8-272-T3 12MHz, X2 25MHz

Commit message: update Gerbers
Parts:
- added J1: DNI, Wurth_Connectors_WR-FSH:696101000002
- 12VDC, 3VDC, 3VFB, 5V-NI1, 5V-NI2, 5VDC, 5VFB, ADC12, AVDD, CS, CS1, DVDD, FB1, FB2, GND, GND-3, GND-5, IOVDD, L-REC1, L-REC2, MI, MISO1, MO, MOSI1, REL0, REL1, REL2, REL3, REL4, REL5, REL6, REL7, RX0, RX1, SC, SCL0, SCL1, SCLK1, SDA0, SDA1, SW, SW3, VBUS, VCC, VCC2, VREF: value TESTPOINT -> DNI
- K1, K2, K3, K4, K5, K6, K7, K8: value G2RL-1A-E DC12 -> G2RL-1A-E_DC12
- X1: value ABM8-272-T3 12MHz -> 12MHz
- moved U$2 74.5 mm to (58.0, 5.97)
- moved AC_L 38.2 mm to (4.85, 89.3)
- moved AC_N 24.8 mm to (4.86, 77.3)
- moved L-REC1 6.66 mm to (24.5, 41.5)
Connections:
- new net AC_L_F: AC_L.B3,0, J1.1
- net AC_L: now also J1.2; no longer AC_L.B3,0
Routing:
- net AGND: track 353.1 -> 379.4 mm
- net AC_L_F: track 0.00 -> 21.8 mm
- net AC_L: track 108.8 -> 112.9 mm
- net LREC1: track 24.3 -> 22.7 mm
- added copper zone on layer 15, net AC_L_F
- added copper zone on layer 16, net AC_L_F
