File: src/Hardware-Design/ENERGIS/Rev1.1.0/ENERGIS_Rack-PDU_1.1.0.brd (EAGLE design)
At the start: 210 x 108 mm, 443 parts, among them IC1 MP2315GJ-Z, IC10 HLW8032, IC11 HLW8032, IC12 HLW8032, IC13 MP150GJ, IC14 HLW8032, IC15 RP2040, IC16 HLW8032, IC17 MCP6001RT-I/OT, IC18 W25Q128JVPIQ, IC19 CAT24C256HU4IGT3, IC2 MP2315GJ-Z, IC20 W5500, IC21 DNI, IC22 MCP6001RT-I/OT, IC3 ULN2803AFWG, IC4 MCP23017T-E/ML, IC5 MP150GJ, IC6 HLW8032, IC7 HLW8032, IC8 HLW8032, IC9 SN74HC151PWR, J10 0R 1%, J2 JP, J7 JP, J8 0R 1%, J9 0R 1%, K1 G2RL-1A-E DC12, K2 G2RL-1A-E DC12, K3 G2RL-1A-E DC12, K4 G2RL-1A-E DC12, K5 G2RL-1A-E DC12, K6 G2RL-1A-E DC12, K7 G2RL-1A-E DC12, K8 G2RL-1A-E DC12, P12ON Green, P3ON Green, P5ON DNI, SW3 DNI, T1 BSS138, X1 12MHz, X2 25MHz

Commit message: major pre-release update on project files and documentation
Parts:
- added C105: 100nF 25V, ds_capacitors:0201
- added IC23: DNI, ds_ic_peripherals:SC70-5
- added R172: DNI, ds_passive:0402
- AC_L, AC_N: value MOUNT-PAD-ROUND3.0 -> FASTON-1217861-1; device holes:3,0-PAD -> ds_con:1217861-1
- C1, C14, C17: value DNI -> 22uF 25V
- C100, C3, C6, C8, C98: value DNI -> 100nF 25V
- C11: value DNI -> 33pF 50V
- C83: value C1206C102KGRACTM -> (none); device ds_passive:C1206 -> ds_capacitors:1206
- C97, C99: value DNI -> 10uF 50V
- FAN, GDRC, RGTG, U$1, U$10, U$11, U$12, U$13, U$14, U$15, U$2, U$3, U$4, U$5, U$6, U$7: value (none) -> DNI
- IC9: value SN74HC151PWR -> CD74ACT151M96
- J2, J7: value JP -> DNI
- L1: device ds_passive:SRR5228A -> ds_inductor:SRR5228A
- L2: value 4.2uH -> 4.7uH; device ds_passive:SRR5228A -> ds_inductor:SRR5228A
- L_OUT1, L_OUT2, L_OUT3, L_OUT4, L_OUT5, L_OUT6, L_OUT7, L_OUT8, N_OUT1, N_OUT2, N_OUT3, N_OUT4, N_OUT5, N_OUT6, N_OUT7, N_OUT8: value MOUNT-PAD-ROUND2.8 -> FASTON-1217861-1; device holes:2,8-PAD -> ds_con:1217861-1
- R10: value 33K -> 33K 1%; device ds_passive:0402 -> ds_resistor:0402
- R11: value DNI -> 40.2K 1%
- R12: value DNI -> 7.5K 1%
- R128, R165: value NC -> DNI
- R143: device ds_passive:R0201 -> ds_resistor:0201
- R148: value DNI -> 2.4K 1%
- R162: value DNI -> 10K 1%
- R170: value DNI -> 0R 1%
- R3: value DNI -> 100K 1%
- R4: value DNI -> 9.09K 1%
- R7: value DNI -> 10R 1%
- R8: value DNI -> 20K 1%
- moved U$15 44.2 mm to (98.9, 38.2)
- moved 3VDC 11.0 mm to (92.5, 4.74), flipped to the bottom
- moved GND-3 9.92 mm to (85.7, 11.9), flipped to the bottom
- moved GND 6.92 mm to (122.8, 12.9), flipped to the bottom
- moved 12VDC 4.40 mm to (124.0, 19.7), flipped to the bottom
- moved GND-5 3.91 mm to (123.1, 6.79), flipped to the bottom
- moved AC_L 3.88 mm to (13.7, 48.8), turned to 90 degrees
- moved AC_N 3.71 mm to (4.57, 48.8), turned to 90 degrees
- moved IOVDD 3.17 mm to (162.5, 8.71), flipped to the bottom
- moved L_OUT3 3.05 mm to (74.8, 90.2), turned to 180 degrees
- moved L_OUT1 3.03 mm to (27.8, 90.0), turned to 180 degrees
- moved U$2 2.89 mm to (3.67, 60.9)
- moved L_OUT7 2.81 mm to (171.8, 89.6), turned to 180 degrees
- moved L_OUT8 2.73 mm to (196.2, 89.5), turned to 180 degrees
- moved VREF 2.70 mm to (141.3, 19.0), flipped to the bottom
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- renumbered BOOT to BT, RESET to RES, RX1 to TX0
Connections:
- new net 3V3_EN: IC2.6, R171.1, R172.1, R2.2
- new net ADC_TEMP: IC15.39, IC23.3
- net +3V3: now also C105.1, IC23.4
- net AC_L: now also AC_L.1, AC_L.2; no longer AC_L.B3,0
- net AGND: now also AC_N.1, AC_N.2; no longer AC_N.B3,0
- net BUCK_EN: now also R172.2; no longer IC2.6, R171.1, R2.2
- net FAN_CTRL: now also IC15.34; no longer IC15.39
- net GND: now also C105.2, IC23.2
- net LCD_RES: no longer IC15.34
- net N_OUT1: now also N_OUT1.1, N_OUT1.2; no longer N_OUT1.B2,8
- net N_OUT2: now also N_OUT2.1, N_OUT2.2; no longer N_OUT2.B2,8
- net N_OUT3: now also N_OUT3.1, N_OUT3.2; no longer N_OUT3.B2,8
- net N_OUT4: now also N_OUT4.1, N_OUT4.2; no longer N_OUT4.B2,8
- net N_OUT5: now also N_OUT5.1, N_OUT5.2; no longer N_OUT5.B2,8
- net N_OUT6: now also N_OUT6.1, N_OUT6.2; no longer N_OUT6.B2,8
- net N_OUT7: now also N_OUT7.1, N_OUT7.2; no longer N_OUT7.B2,8
- net N_OUT8: now also N_OUT8.1, N_OUT8.2; no longer N_OUT8.B2,8
- net OUT_1: now also L_OUT1.1, L_OUT1.2; no longer L_OUT1.B2,8
- net OUT_2: now also L_OUT2.1, L_OUT2.2; no longer L_OUT2.B2,8
- net OUT_3: now also L_OUT3.1, L_OUT3.2; no longer L_OUT3.B2,8
- net OUT_4: now also L_OUT4.1, L_OUT4.2; no longer L_OUT4.B2,8
- net OUT_5: now also L_OUT5.1, L_OUT5.2; no longer L_OUT5.B2,8
- net OUT_6: now also L_OUT6.1, L_OUT6.2; no longer L_OUT6.B2,8
- net OUT_7: now also L_OUT7.1, L_OUT7.2; no longer L_OUT7.B2,8
- net OUT_8: now also L_OUT8.1, L_OUT8.2; no longer L_OUT8.B2,8
Routing:
- net SH: track 78.4 -> 136.8 mm
- net LCD_RES: track 52.4 -> 15.5 mm, vias 3 -> 2
- net AGND: track 351.5 -> 380.2 mm, vias 286 -> 277
- net 3V3_EN: track 0.00 -> 14.6 mm, vias 0 -> 2
- net ADC_TEMP: track 0.00 -> 11.7 mm, vias 0 -> 2
- net +3V3: track 100.3 -> 109.5 mm, vias 30 -> 32
- net 3VFB: track 4.25 -> 11.4 mm, vias 0 -> 1
- net N_OUT8: track 0.00 -> 6.77 mm, vias 16 -> 10
- net BUCK_EN: track 102.3 -> 96.2 mm, vias 6 -> 5
- net N_OUT2: track 3.61 -> 9.27 mm, vias 16 -> 11
- net 5VFB: track 2.33 -> 7.03 mm, vias 0 -> 1
- net FAN_CTRL: track 44.7 -> 40.5 mm
- net N_OUT4: track 3.72 -> 7.87 mm, vias 16 -> 12
- net N_OUT5: track 3.45 -> 7.53 mm, vias 16 -> 11
- net N_OUT7: track 3.49 -> 7.46 mm, vias 16 -> 12
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Other:
- outline, holes or cut-outs redrawn
- board text added: "EBP"
- board text added: "PE"
- board text added: "Place Label Here"

Commit message: update documentation
Parts:
- added 3V3A, ADCUSB, ADC_TEMP, BOOT, FCTL, MCPVIN, RST, UTX: DNI, ds_passive:TP-ROUND
- added DNI: 0R 1%, ds_resistor:0402
- C83: value (none) -> 1nF 2kV
- IC1: value MP2315GJ-Z -> DNI
- L2: value 4.7uH -> 4.7uH 3.5A
- R170: value 0R 1% -> DNI
- moved REL7 0.80 mm to (137.0, 36.4)
- moved VREF 0.60 mm to (141.3, 18.4)
- moved REL0 0.60 mm to (153.2, 36.4)
- moved REL6 0.60 mm to (139.3, 36.4)
- moved REL1 0.40 mm to (150.8, 36.4)
- moved REL5 0.40 mm to (141.6, 36.4)
- moved RX0 0.40 mm to (158.6, 40.1)
- moved TX0 0.40 mm to (158.7, 36.7)
- moved REL4 0.20 mm to (143.9, 36.4)
- moved REL2 0.20 mm to (148.5, 36.4)
Connections:
- net +3V3_A: now also 3V3A.TP
- net ADC_TEMP: now also ADC_TEMP.TP
- net ADC_V_USB: now also ADCUSB.TP
- net AVDD: now also DNI.1
- net FAN_CTRL: now also FCTL.TP
- net MCP_VIN: now also DNI.2, MCPVIN.TP
- net RUN: now also RST.TP
- net TX_OUTSEL: now also UTX.TP
- net USB_BOOT: now also BOOT.TP
Routing:
- net MCP_VIN: track 2.78 -> 7.59 mm, vias 0 -> 1
- net RUN: track 52.3 -> 56.5 mm
- net TX_OUTSEL: track 4.33 -> 6.98 mm, vias 0 -> 1
- net USB_BOOT: track 1.92 -> 4.14 mm, vias 0 -> 1
- net AVDD: track 34.4 -> 36.2 mm
- net REL_7: track 26.2 -> 27.0 mm
- net VREF: track 9.72 -> 9.12 mm
- net REL_6: track 22.5 -> 23.1 mm
- net REL_0: track 22.3 -> 22.9 mm

Commit message: correct BOM
Parts:
- IC21: value DNI -> MIC5504-3.3YM5
- IC23: value DNI -> MCP9700AT-E/LT
- IC9: value CD74ACT151M96 -> SN74HC151PWR
Changed lines of the file:
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@@
 <attribute name="VALUE" x="194.341409375" y="50.374409375" size="0.66234375" layer="27" rot="R90"/>
 </element>
-<element name="IC9" library="ds_ic_logic" package="TSSOP16" package3d_urn="urn:adsk.eagle:package:16485/2" value="CD74ACT151M96" x="170.3664" y="33.7262" smashed="yes" rot="R180">
+<element name="IC9" library="ds_ic_logic" package="TSSOP16" package3d_urn="urn:adsk.eagle:package:16485/2" value="SN74HC151PWR" x="170.3664" y="33.7262" smashed="yes" rot="R180">
 <attribute name="DATASHEET" value="https://www.ti.com/lit/ds/symlink/sn74hc151.pdf?ts=1749408396579&amp;ref_url=https%253A%252F%252Fwww.google.com%252F" x="170.3664" y="33.7262" size="1.778" layer="27" rot="R180" display="off"/>
-<attribute name="DESCRIPTION" value="24mA 4.5V~5.5V 24mA SOIC-16 Signal Switches, Multiplexers, Decoders ROHS " x="170.3664" y="33.7262" size="1.778" layer="27" rot="R180" display="off"/>
+<attribute name="DESCRIPTION" value="-40℃~+85℃ 25ns@6V,50pF 2V~6V 7.8mA 7.8mA 80uA Single Supply TSSOP-16 Signal Switches, Multiplexers, Decoders ROHS" x="170.3664" y="33.7262" size="1.778" layer="27" rot="R180" display="off"/>
 <attribute name="HQ_PART" value="IC0244620" x="170.3664" y="33.7262" size="1.778" layer="27" rot="R180" display="off"/>
-<attribute name="LCSC_PART" value="C2674746" x="170.3664" y="33.7262" size="1.778" layer="27" rot="R180" display="off"/>
-<attribute name="MANUFACTURER" value="Nexperia" x="170.3664" y="33.7262" size="1.778" layer="27" rot="R180" display="off"/>
-<attribute name="MPN" value="74HC151PW-Q100,118 " x="170.3664" y="33.7262" size="1.778" layer="27" rot="R180" display="off"/>
+<attribute name="LCSC_PART" value="C2653837" x="170.3664" y="33.7262" size="1.778" layer="27" rot="R180" display="off"/>
+<attribute name="MANUFACTURER" value="Texas Instruments" x="170.3664" y="33.7262" size="1.778" layer="27" rot="R180" display="off"/>
+<attribute name="MPN" value="SN74HC151PWR" x="170.3664" y="33.7262" size="1.778" layer="27" rot="R180" display="off"/>
 <attribute name="NAME" x="173.472" y="36.809" size="0.8128" layer="25" ratio="10" rot="R270"/>
 <attribute name="ROHS" value="YES" x="170.3664" y="33.7262" size="1.778" layer="27" rot="R180" display="off"/>
-<attribute name="VALUE" value="CD74ACT151M96" x="170.3664" y="33.7262" size="1.778" layer="27" rot="R180" display="off"/>
+<attribute name="VALUE" value="SN74HC151PWR" x="170.3664" y="33.7262" size="1.778" layer="27" rot="R180" display="off"/>
 <attribute name="VALUE" x="166.4802" y="35.809" size="1.016" layer="27" ratio="10" rot="R270"/>
 </element>
@@
 <attribute name="VALUE" x="190.101" y="24.6036" size="1.016" layer="27" rot="R90"/>
 </element>
-<element name="IC21" library="ds_ic_vreg" package="SOT23-5" package3d_urn="urn:adsk.eagle:package:25419215/2" value="DNI" x="178.6242" y="17.1666" smashed="yes">
+<element name="IC21" library="ds_ic_vreg" package="SOT23-5" package3d_urn="urn:adsk.eagle:package:25419215/2" value="MIC5504-3.3YM5 " x="178.6242" y="17.1666" smashed="yes">
 <attribute name="DATASHEET" value="https://ww1.microchip.com/downloads/en/DeviceDoc/MIC5501-02-03-04-300mA-Single-Output-LDO-in-Small-Packages-DS20006006B.pdf" x="178.6242" y="17.1666" size="1.778" layer="27" display="off"/>
 <attribute name="DESCRIPTION" value="SOT-23-5 Voltage Regulators - Linear, Low Drop Out (LDO) Regulators ROHS " x="178.6242" y="17.1666" size="1.778" layer="27" display="off"/>
@@
 <attribute name="VALUE" x="81.665" y="6.385" size="1.016" layer="27" rot="R270"/>
 </element>
-<element name="IC23" library="ds_ic_peripherals" package="SC70-5" package3d_urn="urn:adsk.eagle:package:49052119/1" value="DNI" x="164.41" y="4.1" smashed="yes" rot="R90">
+<element name="IC23" library="ds_ic_peripherals" package="SC70-5" package3d_urn="urn:adsk.eagle:package:49052119/1" value="MCP9700AT-E/LT " x="164.41" y="4.1" smashed="yes" rot="R90">
 <attribute name="DATASHEET" value="https://ww1.microchip.com/downloads/aemDocuments/documents/MSLD/ProductDocuments/DataSheets/MCP970X-Family-Data-Sheet-DS20001942.pdf" x="164.41" y="4.1" size="1.778" layer="27" rot="R90" display="off"/>
 <attribute name="DESCRIPTION" value="-40℃~+125℃ 2.3V~5.5V ±2℃ SC-70-5 Temperature Sensors ROHS" x="164.41" y="4.1" size="1.778" layer="27" rot="R90" display="off"/>
