File: src/Hardware-Design/ENERGIS/Rev1.1.0/ENERGIS_Main-Board-1.1.0.brd (EAGLE design)
At the start: 210 x 108 mm, 455 parts, among them IC1 DNI, IC10 HLW8032, IC11 HLW8032, IC12 HLW8032, IC13 MP150GJ, IC14 HLW8032, IC15 RP2040, IC16 HLW8032, IC17 MCP6001RT-I/OT, IC18 W25Q128JVPIQ, IC19 CAT24C256HU4IGT3, IC2 MP2315GJ-Z, IC20 W5500, IC21 MIC5504-3.3YM5, IC22 MCP6001RT-I/OT, IC23 MCP9700AT-E/LT, IC3 ULN2803AFWG, IC4 MCP23017T-E/ML, IC5 MP150GJ, IC6 HLW8032, IC7 HLW8032, IC8 HLW8032, IC9 SN74HC151PWR, J10 0R 1%, J2 DNI, J7 DNI, J8 0R 1%, J9 0R 1%, K1 G2RL-1A-E DC12, K2 G2RL-1A-E DC12, K3 G2RL-1A-E DC12, K4 G2RL-1A-E DC12, K5 G2RL-1A-E DC12, K6 G2RL-1A-E DC12, K7 G2RL-1A-E DC12, K8 G2RL-1A-E DC12, P12ON Green, P3ON Green, P5ON DNI, SW3 DNI, T1 BSS138, X1 12MHz, X2 25MHz

Commit message: update readme
Parts:
- AC/DC2: value IRM-10-15 -> IRM-15-12
- R130, R166, R167, R168: value 3.3K 1% -> 1.2K 1%
- R147: value 10K 1% -> 1K 1%
- R149: value 3.3K 1% -> DNI
- R171: value 10K 1% -> 33K 1%
Changed lines of the file:
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@@
 <attribute name="NAME" x="41.3706" y="13.771" size="1.27" layer="25" ratio="10" rot="R270"/>
 </element>
-<element name="AC/DC2" library="ds_trafo" package="IRM_15_12" package3d_urn="urn:adsk.eagle:package:47260462/2" value="IRM-10-15 " x="87.2676" y="33.0386" smashed="yes">
+<element name="AC/DC2" library="ds_trafo" package="IRM_15_12" package3d_urn="urn:adsk.eagle:package:47260462/2" value="IRM-15-12 " x="87.2676" y="33.0386" smashed="yes">
 <attribute name="DATASHEET" value="https://www.meanwell.com/Upload/PDF/IRM-15/IRM-15-SPEC.PDF" x="87.2676" y="33.0386" size="1.778" layer="27" display="off"/>
 <attribute name="DESCRIPTION" value="15W AC-DC PCB-Mount Green Power Module" x="87.2676" y="33.0386" size="1.778" layer="27" display="off"/>
@@
 <attribute name="VALUE" x="180.497" y="18.4314" size="1.27" layer="27" rot="R90"/>
 </element>
-<element name="R147" library="ds_resistor" package="0402" package3d_urn="urn:adsk.eagle:package:46683744/3" value="10K 1%" x="147.106" y="3.173" smashed="yes" rot="R90">
+<element name="R147" library="ds_resistor" package="0402" package3d_urn="urn:adsk.eagle:package:46683744/3" value="1K 1%" x="147.106" y="3.173" smashed="yes" rot="R90">
 <attribute name="DESCRIPTION" value="62.5mW Thick Film Resistors 50V ±100ppm/℃ ±1% 10kΩ 0402 Chip Resistor - Surface Mount ROHS" x="147.106" y="3.173" size="1.778" layer="27" rot="R90" display="off"/>
 <attribute name="HQ_PART" value="RE0207399" x="147.106" y="3.173" size="1.778" layer="27" rot="R90" display="off"/>
@@
 <attribute name="VALUE" x="149.011" y="2.538" size="1.016" layer="27" rot="R90"/>
 </element>
-<element name="R149" library="ds_resistor" package="_0603X4-1206" package3d_urn="urn:adsk.eagle:package:49287421/2" value="3.3K 1%" x="125.0276" y="10.1948" smashed="yes" rot="R270">
+<element name="R149" library="ds_resistor" package="_0603X4-1206" package3d_urn="urn:adsk.eagle:package:49287421/2" value="DNI" x="125.0276" y="10.1948" smashed="yes" rot="R270">
 <attribute name="DESCRIPTION" value="4 ±1% 3.3kΩ 62.5mW ±200ppm/℃ 0603x4 Resistor Networks, Arrays ROHS " x="125.0276" y="10.1948" size="1.778" layer="27" rot="R270" display="off"/>
 <attribute name="HQ_PART" value="RE0093863" x="125.0276" y="10.1948" size="1.778" layer="27" rot="R270" display="off"/>
@@
 <attribute name="VALUE" value="DNI" x="121.99" y="15.88" size="1.778" layer="28" rot="MR180" display="off"/>
 </element>
-<element name="R130" library="ds_resistor" package="0402" package3d_urn="urn:adsk.eagle:package:46683744/3" value="3.3K 1%" x="137.58" y="9.11" smashed="yes" rot="R270">
+<element name="R130" library="ds_resistor" package="0402" package3d_urn="urn:adsk.eagle:package:46683744/3" value="1.2K 1%" x="137.58" y="9.11" smashed="yes" rot="R270">
 <attribute name="DESCRIPTION" value="62.5mW Thick Film Resistors 50V ±100ppm/℃ ±1% 3.3kΩ 0402 Chip Resistor - Surface Mount ROHS" x="137.58" y="9.11" size="1.778" layer="27" rot="R270" display="off"/>
 <attribute name="HQ_PART" value="RE0189064" x="137.58" y="9.11" size="1.778" layer="27" rot="R270" display="off"/>
@@
 <attribute name="VALUE" x="135.675" y="9.745" size="1.016" layer="27" rot="R270"/>
 </element>
-<element name="R166" library="ds_resistor" package="0402" package3d_urn="urn:adsk.eagle:package:46683744/3" value="3.3K 1%" x="139.3" y="9.1" smashed="yes" rot="R270">
+<element name="R166" library="ds_resistor" package="0402" package3d_urn="urn:adsk.eagle:package:46683744/3" value="1.2K 1%" x="139.3" y="9.1" smashed="yes" rot="R270">
 <attribute name="DESCRIPTION" value="62.5mW Thick Film Resistors 50V ±100ppm/℃ ±1% 3.3kΩ 0402 Chip Resistor - Surface Mount ROHS" x="139.3" y="9.1" size="1.778" layer="27" rot="R270" display="off"/>
 <attribute name="HQ_PART" value="RE0189064" x="139.3" y="9.1" size="1.778" layer="27" rot="R270" display="off"/>
@@
 <attribute name="VALUE" x="137.395" y="9.735" size="1.016" layer="27" rot="R270"/>
 </element>
-<element name="R167" library="ds_resistor" package="0402" package3d_urn="urn:adsk.eagle:package:46683744/3" value="3.3K 1%" x="153.26" y="22.29" smashed="yes" rot="R270">
+<element name="R167" library="ds_resistor" package="0402" package3d_urn="urn:adsk.eagle:package:46683744/3" value="1.2K 1%" x="153.26" y="22.29" smashed="yes" rot="R270">
 <attribute name="DESCRIPTION" value="62.5mW Thick Film Resistors 50V ±100ppm/℃ ±1% 3.3kΩ 0402 Chip Resistor - Surface Mount ROHS" x="153.26" y="22.29" size="1.778" layer="27" rot="R270" display="off"/>
 <attribute name="HQ_PART" value="RE0189064" x="153.26" y="22.29" size="1.778" layer="27" rot="R270" display="off"/>
@@
 <attribute name="VALUE" x="151.355" y="22.925" size="1.016" layer="27" rot="R270"/>
 </element>
-<element name="R168" library="ds_resistor" package="0402" package3d_urn="urn:adsk.eagle:package:46683744/3" value="3.3K 1%" x="155.38" y="22.3" smashed="yes" rot="R270">
+<element name="R168" library="ds_resistor" package="0402" package3d_urn="urn:adsk.eagle:package:46683744/3" value="1.2K 1%" x="155.38" y="22.3" smashed="yes" rot="R270">
 <attribute name="DESCRIPTION" value="62.5mW Thick Film Resistors 50V ±100ppm/℃ ±1% 3.3kΩ 0402 Chip Resistor - Surface Mount ROHS" x="155.38" y="22.3" size="1.778" layer="27" rot="R270" display="off"/>
 <attribute name="HQ_PART" value="RE0189064" x="155.38" y="22.3" size="1.778" layer="27" rot="R270" display="off"/>
@@
 <attribute name="VALUE" x="176.44" y="-2.12" size="1.016" layer="28" rot="MR0"/>
 </element>
-<element name="R171" library="ds_resistor" package="0402" package3d_urn="urn:adsk.eagle:package:46683744/3" value="10K 1%" x="83.57" y="5.75" smashed="yes" rot="R270">
-<attribute name="DESCRIPTION" value="62.5mW Thick Film Resistors 50V ±100ppm/℃ ±1% 10kΩ 0402 Chip Resistor - Surface Mount ROHS" x="83.57" y="5.75" size="1.778" layer="27" rot="R270" display="off"/>
-<attribute name="HQ_PART" value="RE0207399" x="83.57" y="5.75" size="1.778" layer="27" rot="R270" display="off"/>
-<attribute name="LCSC_PART" value="C25744" x="83.57" y="5.75" size="1.778" layer="27" rot="R270" display="off"/>
-<attribute name="MANUFACTURER" value="ROHM" x="83.57" y="5.75" size="1.778" layer="27" rot="R270" display="off"/>
-<attribute name="MPN" value="MCR01MZPF1002" x="83.57" y="5.75" size="1.778" layer="27" rot="R270" display="off"/>
+<element name="R171" library="ds_resistor" package="0402" package3d_urn="urn:adsk.eagle:package:46683744/3" value="33K 1%" x="83.57" y="5.75" smashed="yes" rot="R270">
+<attribute name="DESCRIPTION" value="62.5mW Thick Film Resistors 50V ±100ppm/℃ ±1% 33kΩ 0402 Chip Resistor - Surface Mount ROHS" x="83.57" y="5.75" size="1.778" layer="27" rot="R270" display="off"/>
+<attribute name="HQ_PART" value="RE0321838" x="83.57" y="5.75" size="1.778" layer="27" rot="R270" display="off"/>
+<attribute name="LCSC_PART" value="C25779" x="83.57" y="5.75" size="1.778" layer="27" rot="R270" display="off"/>
+<attribute name="MANUFACTURER" value="RALEC" x="83.57" y="5.75" size="1.778" layer="27" rot="R270" display="off"/>
+<attribute name="MPN" value="RTT023302FTH" x="83.57" y="5.75" size="1.778" layer="27" rot="R270" display="off"/>
 <attribute name="PACKAGE" value="0402" x="83.57" y="5.75" size="1.778" layer="27" rot="R270" display="off"/>
 <attribute name="ROHS" value="YES" x="83.57" y="5.75" size="1.778" layer="27" rot="R270" display="off"/>
-<attribute name="VALUE" x="81.665" y="6.385" size="1.016" layer="27" rot="R270"/>
+<attribute name="VALUE" value="33K 1%" x="81.665" y="6.385" size="1.016" layer="27" rot="R270"/>
 </element>
 <element name="IC23" library="ds_ic_peripherals" package="SC70-5" package3d_urn="urn:adsk.eagle:package:49052119/1" value="MCP9700AT-E/LT " x="164.41" y="4.1" smashed="yes" rot="R90">
