File: src/Hardware-Design/ENERGIS/Rev1.1.0/ENERGIS_Main-Board-1.1.0.sch (EAGLE design)
At the start: 442 parts, among them IC1 DNI, IC10 HLW8032, IC11 HLW8032, IC12 HLW8032, IC13 MP150GJ, IC14 HLW8032, IC15 RP2040, IC16 HLW8032, IC17 MCP6001RT-I/OT, IC18 W25Q128JVPIQ, IC19 CAT24C256HU4IGT3, IC2 MP2315GJ-Z, IC20 W5500, IC21 MIC5504-3.3YM5, IC22 MCP6001RT-I/OT, IC23 MCP9700AT-E/LT, IC3 ULN2803AFWG, IC4 MCP23017T-E/ML, IC5 MP150GJ, IC6 HLW8032, IC7 HLW8032, IC8 HLW8032, IC9 SN74HC151PWR, J10 0R 1%, J2 DNI, J7 DNI, J8 0R 1%, J9 0R 1%, K1 G2RL-1A-E DC12, K2 G2RL-1A-E DC12, K3 G2RL-1A-E DC12, K4 G2RL-1A-E DC12, K5 G2RL-1A-E DC12, K6 G2RL-1A-E DC12, K7 G2RL-1A-E DC12, K8 G2RL-1A-E DC12, P12ON Green, P3ON Green, P5ON DNI, SW3 DNI, T1 BSS138, X1 12MHz, X2 25MHz

Commit message: update readme
Parts:
- AC/DC2: value IRM-10-15 -> IRM-15-12
- R130, R166, R167, R168: value 3.3K 1% -> 1.2K 1%
- R147: value 10K 1% -> 1K 1%
- R149: value 3.3K 1% -> DNI
- R171: value 10K 1% -> 33K 1%; device ds_resistor:10K-1%0402 -> ds_resistor:33K-1%0402
Other:
- note added: "ADDRESS ON 0x50"
- note added: "DNI ALL"
