File: src/Hardware-Design/ENERGIS/Rev1.0.0/ENERGIS_Rack-PDU_1.0.0.brd (EAGLE design)
At the start: 210 x 108 mm, 428 parts, among them IC1 MP2315GJ-Z, IC10 HLW8032, IC11 HLW8032, IC12 HLW8032, IC13 MP150GJ, IC14 HLW8032, IC15 RP2040, IC16 HLW8032, IC17 MCP6001RT-I/OT, IC18 W25Q128JVPIQ, IC19 CAT24C256HU4IGT3, IC2 MP2315GJ-Z, IC20 W5500, IC21 MIC5504-3.3YM5, IC22 MCP6001RT-I/OT, IC3 ULN2803AFWG, IC4 MCP23017T-E/ML, IC5 MP150GJ, IC6 HLW8032, IC7 HLW8032, IC8 HLW8032, IC9 SN74HC151PWR, J10 0R 1%, J2 JP, J7 JP, J8 0R 1%, J9 0R 1%, K1 G2RL-1A-E DC12, K2 G2RL-1A-E DC12, K3 G2RL-1A-E DC12, K4 G2RL-1A-E DC12, K5 G2RL-1A-E DC12, K6 G2RL-1A-E DC12, K7 G2RL-1A-E DC12, K8 G2RL-1A-E DC12, P12ON Green, P3ON Green, P5ON Green, SW3 TP, X1 ABM8-272-T3 12MHz, X2 25MHz

Commit message: add mac calculation
Connections:
- net LCD_CS renamed SPI1_CS
- net LCD_MISO renamed SPI1_MISO
- net LCD_MOSI renamed SPI1_MOSI
- net LCD_SCLK renamed SPI1_SCLK
Changed lines of the file:
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@@
 <drawing>
 <settings>
-<setting alwaysvectorfont="yes"/>
+<setting alwaysvectorfont="no"/>
 <setting verticaltext="up"/>
 </settings>
@@
 <wire x1="153.2" y1="15.01118125" x2="150.85781875" y2="12.669" width="0.2032" layer="14"/>
 </signal>
-<signal name="LCD_CS">
+<signal name="SPI1_CS">
 <contactref element="IC15" pad="12"/>
 <contactref element="R149" pad="C2"/>
@@
 <wire x1="128.31" y1="11.49" x2="131.14" y2="8.66" width="0.2032" layer="16"/>
 </signal>
-<signal name="LCD_SCLK">
+<signal name="SPI1_SCLK">
 <contactref element="IC15" pad="13"/>
 <contactref element="DSP" pad="17"/>
@@
 <wire x1="129.22781875" y1="7.991" x2="131.953" y2="7.991" width="0.2032" layer="16"/>
 </signal>
-<signal name="LCD_MISO">
+<signal name="SPI1_MISO">
 <contactref element="IC15" pad="11"/>
 <contactref element="R149" pad="B2"/>
@@
 <wire x1="130.6052" y1="11.7548" x2="132.87" y2="11.7548" width="0.2032" layer="16"/>
 </signal>
-<signal name="LCD_MOSI">
+<signal name="SPI1_MOSI">
 <contactref element="IC15" pad="14"/>
 <contactref element="DSP" pad="16"/>
