File: src/Hardware-Design/ENERGIS/Rev1.0.0/ENERGIS_Rack-PDU_1.0.0.sch (EAGLE design)
At the start: 419 parts, among them IC1 MP2315GJ-Z, IC10 HLW8032, IC11 HLW8032, IC12 HLW8032, IC13 MP150GJ, IC14 HLW8032, IC15 RP2040, IC16 HLW8032, IC17 MCP6001RT-I/OT, IC18 W25Q128JVPIQ, IC19 CAT24C256HU4IGT3, IC2 MP2315GJ-Z, IC20 W5500, IC21 MIC5504-3.3YM5, IC22 MCP6001RT-I/OT, IC3 ULN2803AFWG, IC4 MCP23017T-E/ML, IC5 MP150GJ, IC6 HLW8032, IC7 HLW8032, IC8 HLW8032, IC9 SN74HC151PWR, J10 0R 1%, J2 JP, J7 JP, J8 0R 1%, J9 0R 1%, K1 G2RL-1A-E DC12, K2 G2RL-1A-E DC12, K3 G2RL-1A-E DC12, K4 G2RL-1A-E DC12, K5 G2RL-1A-E DC12, K6 G2RL-1A-E DC12, K7 G2RL-1A-E DC12, K8 G2RL-1A-E DC12, P12ON Green, P3ON Green, P5ON Green, SW3 TP, X1 ABM8-272-T3 12MHz, X2 25MHz

Commit message: add mac calculation
Connections:
- net LCD_CS renamed SPI1_CS
- net LCD_MISO renamed SPI1_MISO
- net LCD_MOSI renamed SPI1_MOSI
- net LCD_SCLK renamed SPI1_SCLK
Changed lines of the file:
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@@
 </segment>
 </net>
-<net name="LCD_CS" class="0">
+<net name="SPI1_CS" class="0">
 <segment>
 <pinref part="IC15" gate="G$1" pin="GPIO9"/>
@@
 </segment>
 </net>
-<net name="LCD_SCLK" class="0">
+<net name="SPI1_SCLK" class="0">
 <segment>
 <pinref part="IC15" gate="G$1" pin="GPIO10"/>
@@
 </segment>
 </net>
-<net name="LCD_MISO" class="0">
+<net name="SPI1_MISO" class="0">
 <segment>
 <pinref part="IC15" gate="G$1" pin="GPIO8"/>
@@
 </segment>
 </net>
-<net name="LCD_MOSI" class="0">
+<net name="SPI1_MOSI" class="0">
 <segment>
 <pinref part="IC15" gate="G$1" pin="GPIO11"/>
@@
 </segment>
 </net>
-<net name="LCD_CS" class="0">
+<net name="SPI1_CS" class="0">
 <segment>
 <wire x1="327.66" y1="58.42" x2="289.56" y2="58.42" width="0.1524" layer="91"/>
@@
 </segment>
 </net>
-<net name="LCD_MOSI" class="0">
+<net name="SPI1_MOSI" class="0">
 <segment>
 <wire x1="289.56" y1="66.04" x2="327.66" y2="66.04" width="0.1524" layer="91"/>
@@
 </segment>
 </net>
-<net name="LCD_MISO" class="0">
+<net name="SPI1_MISO" class="0">
 <segment>
 <wire x1="327.66" y1="68.58" x2="289.56" y2="68.58" width="0.1524" layer="91"/>
@@
 </segment>
 </net>
-<net name="LCD_SCLK" class="0">
+<net name="SPI1_SCLK" class="0">
 <segment>
 <wire x1="327.66" y1="63.5" x2="289.56" y2="63.5" width="0.1524" layer="91"/>

Commit message: update documentation
Parts:
- removed CS0, CS1, MISO0, MISO1, MOSI0, MOSI1, REL0, REL1, REL2, REL3, REL4, REL5, REL6, REL7, RX0, RX1, SCL0, SCL1, SCLK0, SCLK1, SDA0, SDA1: TP, ds_passive:TP
- removed FAN: (no value), con-amp-quick:M02
- removed R164: 10K 1%, ds_resistor:10K-1%0402
- removed R165: NC, ds_passive:R0201
- removed T1: (no value), ds_active:BSS138
- R93: value 10K 1% -> 4x10K 1206; device ds_resistor:10K-1%_ARRAY0603X4-1206 -> Resistor Array:742C083103JP
- X1: value ABM8-272-T3 12MHz -> 12MHz
Connections:
- removed net FAN_CTRL: IC15.GPIO27/ADC1, R164.1, R165.1, T1.G
- removed net N$23: FAN.1, T1.D
- removed net SPI1_CS: CS0.P$1, DSP.19, IC15.GPIO9, R149.6
- removed net SPI1_MISO: DSP.15, IC15.GPIO8, MISO0.P$1, R149.7
- removed net SPI1_MOSI: DSP.16, IC15.GPIO11, MOSI0.P$1
- removed net SPI1_SCLK: DSP.17, IC15.GPIO10, SCLK0.P$1
- new net LCD_CS: DSP.19, IC15.GPIO9, R149.6
- new net LCD_MISO: DSP.15, IC15.GPIO8, R149.7
- new net LCD_MOSI: DSP.16, IC15.GPIO11
- new net LCD_SCLK: DSP.17, IC15.GPIO10
- net !W5500_CS: no longer CS1.P$1
- net +12V: no longer FAN.2
- net +3V3_MCU: no longer R165.2
- net GND: no longer R164.2, T1.S
- net I2C0_SCL: no longer SCL0.P$1
- net I2C0_SDA: no longer SDA0.P$1
- net I2C1_SCL: no longer SCL1.P$1
- net I2C1_SDA: no longer SDA1.P$1
- net REL_0: no longer REL0.P$1
- net REL_1: no longer REL1.P$1
- net REL_2: no longer REL2.P$1
- net REL_3: no longer REL3.P$1
- net REL_4: no longer REL4.P$1
- net REL_5: no longer REL5.P$1
- net REL_6: no longer REL6.P$1
- net REL_7: no longer REL7.P$1
- net UART0_RX: no longer RX0.P$1
- net UART0_TX: no longer RX1.P$1
- net W5500_MISO: no longer MISO1.P$1
- net W5500_MOSI: no longer MOSI1.P$1
- net W5500_SCK: no longer SCLK1.P$1
Other:
- note removed: "230VAC-LIVE"
- note removed: "230VAC-NEUTRAL"
- note removed: "C13 OUTPUT LIVE"
- note removed: "C13 OUTPUT NEUTRAL"
- note removed: "DRIVER"
- note removed: "FAN"
- note removed: "I-MEAS V-MEAS"
- note removed: "IN1 M IN2 U IN3 X ..."
- note removed: "MCU RX"
- note removed: "OPTO"
- note removed: "OUT"
- note removed: "RELAY"
- note removed: "RELAY1"
- note removed: "RELAY2"
- note removed: "RELAY3 ..."
- note removed: "SEL A/B/C"
- note removed: "SELECTOR"
- note removed: "TX1 TX2 TX3 ..."
