File: src/Hardware-Design/ENERGIS/Rev1.0.0/ENERGIS_Rack-PDU_1.0.1.sch (EAGLE design)
At the start: 430 parts, among them IC1 MP2315GJ-Z, IC10 HLW8032, IC11 HLW8032, IC12 HLW8032, IC13 MP150GJ, IC14 HLW8032, IC15 RP2040, IC16 HLW8032, IC17 MCP6001RT-I/OT, IC18 W25Q128JVPIQ, IC19 CAT24C256HU4IGT3, IC2 MP2315GJ-Z, IC20 W5500, IC21 DNI, IC22 MCP6001RT-I/OT, IC3 ULN2803AFWG, IC4 MCP23017T-E/ML, IC5 MP150GJ, IC6 HLW8032, IC7 HLW8032, IC8 HLW8032, IC9 SN74HC151PWR, J10 0R 1%, J2 JP, J7 JP, J8 0R 1%, J9 0R 1%, K1 G2RL-1A-E DC12, K2 G2RL-1A-E DC12, K3 G2RL-1A-E DC12, K4 G2RL-1A-E DC12, K5 G2RL-1A-E DC12, K6 G2RL-1A-E DC12, K7 G2RL-1A-E DC12, K8 G2RL-1A-E DC12, P12ON Green, P3ON Green, P5ON DNI, SW3 DNI, T1 BSS138, X1 12MHz, X2 25MHz

Commit message: update documentation
Parts:
- removed ADC12, CS, FB1, FB2, MI, MO, SC, VCC, VCC2: DNI, ds_passive:TP-ROUND
- removed D17, D18: RCLAMP0582BQTCT, ds_diode:RCLAMP0582BQTCT-
- removed GDRC: (no value), ds_con:CON-1X4
- removed R166, R167, R168: 3.3K 1%, ds_resistor:3.3K-1%0402
- removed R169: 0R 1%, ds_resistor:0R1206
- removed R170: DNI, ds_resistor:0R1206
- removed R171: 10K 1%, ds_resistor:10K-1%0402
- removed RN1, RN2: 100K 1%, ds_resistor:100K-1%_ARRAY0603X4-1206
- added CS0, FB-NI1, FB-NI2, MISO0, MOSI0, SCLK0, VNI1, VNI2: TP, ds_passive:TP
- added GDGC: (no value), ds_con:CON-1X4
- 12VDC, 3VDC, 3VFB, 5V-NI1, 5V-NI2, 5VDC, 5VFB, AVDD, CS1, DVDD, GND, GND-3, GND-5, IOVDD, L-REC1, L-REC2, MISO1, MOSI1, REL0, REL1, REL2, REL3, REL4, REL5, REL6, REL7, RX0, RX1, SCL0, SCL1, SCLK1, SDA0, SDA1, SW, SW3, VBUS, VREF: value DNI -> TP; device ds_passive:TP-ROUND -> ds_passive:TP
- C1, C14, C17: value DNI -> 22uF 25V
- C100, C3, C6, C8, C98: value DNI -> 100nF 25V
- C11: value DNI -> 33pF 50V
- C97, C99: value DNI -> 10uF 50V
- D15: value DNI -> SS12
- IC21: value DNI -> MIC5504-3.3YM5
- L1: value DNI -> 4.9uH
- P5ON: value DNI -> Green
- R11: value DNI -> 40.2K 1%
- R12: value DNI -> 7.5K 1%
- R130: device ds_resistor:3.3K-1%0402 -> ds_resistor:3.3K-1%_ARRAY0603X4-1206
- R148: value DNI -> 2.4K 1%
- R162: value DNI -> 10K 1%
- R17, R18, R19, R20, R21, R22, R23, R24: value 0R 1% -> 330R 1% 1W; device ds_resistor:0R2512 -> ds_resistor:330R-1%-2512
- R3: value DNI -> 100K 1%
- R4: value DNI -> 9.09K 1%
- R7: value DNI -> 10R 1%
- R8: value DNI -> 20K 1%
- REF1: value LM4040x30 -> LM4040B30FTA
- T1: value BSS138 -> (none)
- X1: value 12MHz -> ABM8-272-T3 12MHz
Connections:
- removed net LCD_CS: CS.P$1, DSP.19, IC15.GPIO9, R149.6
- removed net LCD_MISO: DSP.15, IC15.GPIO8, MI.P$1, R149.7
- removed net LCD_MOSI: DSP.16, IC15.GPIO11, MO.P$1
- removed net LCD_SCLK: DSP.17, IC15.GPIO10, SC.P$1
- removed net USB_VBUS: R121.1, R126.1, R170.1, USB1.VBUS
- new net SPI1_CS: CS0.P$1, DSP.19, IC15.GPIO9, R149.6
- new net SPI1_MISO: DSP.15, IC15.GPIO8, MISO0.P$1, R149.7
- new net SPI1_MOSI: DSP.16, IC15.GPIO11, MOSI0.P$1
- new net SPI1_SCLK: DSP.17, IC15.GPIO10, SCLK0.P$1
- net +12V: no longer R171.2
- net +12V_MEA: no longer ADC12.P$1
- net +3V3: no longer R169.1
- net +3V3_MCU: now also R130.5, R130.6, R130.7, R130.8; no longer R130.1, R166.1, R167.1, R168.1, R169.2
- net BUCK_EN: no longer R171.1
- net FB1: now also FB-NI1.P$1; no longer FB1.P$1
- net FB2: now also FB-NI2.P$1; no longer FB2.P$1
- net GND: now also GDGC.P$4; no longer D17.3, D18.3, GDRC.P$4, RN1A.1, RN1B.1, RN1C.1, RN1D.1, RN2A.1, RN2B.1, RN2C.1, RN2D.1
- net I2C0_SCL: now also R130.1; no longer D17.1, R130.2
- net I2C0_SDA: now also R130.2; no longer D17.2, R166.2
- net I2C1_SCL: now also R130.3; no longer D18.2, R167.2
- net I2C1_SDA: now also R130.4; no longer D18.1, R168.2
- net REL_0: no longer RN1A.2
- net REL_1: no longer RN1B.2
- net REL_2: no longer RN1C.2
- net REL_3: no longer RN1D.2
- net REL_4: no longer RN2A.2
- net REL_5: no longer RN2B.2
- net REL_6: no longer RN2C.2
- net REL_7: no longer RN2D.2
- net RUN: now also GDGC.P$2; no longer GDRC.P$2
- net SWCLK: now also GDGC.P$1; no longer GDRC.P$1
- net SWDIO: now also GDGC.P$3; no longer GDRC.P$3
- net TX_MUX5: now also OPT2.16; no longer OPT2.10
- net TX_MUX6: now also OPT2.14; no longer OPT2.12
- net TX_MUX7: now also OPT2.12; no longer OPT2.14
- net TX_MUX8: now also OPT2.10; no longer OPT2.16
- net VBUS: now also R121.1, R126.1, USB1.VBUS; no longer R170.2
- net VNI1: now also VNI1.P$1; no longer VCC.P$1
- net VNI2: now also VNI2.P$1; no longer VCC2.P$1
Other:
- note added: "5V AC-MEASUREMENT"
- note added: "DEBUG"
- note added: "FAN"
- note added: "Rev 1.0.0"
- note removed: "12VDC"
- note removed: "230VAC"
- note removed: "5V NON-ISOLATED"
- note removed: "DEBUG CONNECTOR"
- note removed: "Design Note — 12 V supply (Mean Well IRM-10 series), universal 110 V/230 V AC This schematic uses the Mean Well IRM-10 encapsulated AC-DC module (e.g., IRM-10-12) to produce 12 VDC. The IRM-10 series is specified for a wide input range of 85–305 VAC (47–440 Hz) and 120–430 VDC, meaning it operates from both ~115 VAC and ~230 VAC mains with no selector or changes to the circuit. Safety approvals (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"
- note removed: "Design Note — 5 V / 200 mA non-isolated supply (MP150), universal 110 V/230 V AC This design uses MPS MP150 in high-side buck to generate 5 V/200 mA directly from rectified mains. MP150 integrates a 500 V MOSFET (Drain-to-Source rating 500 V), covering the ~325 VDC peak from 230 VAC and ~155 VDC from 115 VAC, so the circuit from 85–265 VAC (“universal input”)."
- note removed: "ENABLE/DISABLE"
- note removed: "FAN CONNECTOR"
- note removed: "MCU"
- note removed: "PERIPHERALS"
- note removed: "USB-C 5VDC"
